File: picdev/picdev/PIC18F26K83.sch (KiCad schematic (older format))
At the start: 16 parts, among them J3 Programming Header, U5 MCP2562, U6 PIC18F26K83

Commit message: Schematic review changes
- swap signals on RC4, RA5 (pic16f)
- add oscillator to 26k83
- break out usb connector
- break out some unused 26k83 pins

Also:
- break out can bus
- add missing decoupling caps
Parts:
- added C10, C9: 26pF, symbol device:C
- added C7: 0.1uF, symbol device:C
- added C8: 10uF, symbol device:C
- added J6: Conn_01x04_Female, symbol Connector:Conn_01x04_Female
- added Y1: Crystal, symbol device:Crystal
Connections:
- net labels added: OSC1, OSC2
- wire segments 47 -> 68
- no-connect marks 1 -> 9
Other:
- moved on the sheet: TP5
Changed lines of the file:
@@
 L power:+5V #PWR026
 U 1 1 5B96EA42
-P 4350 3800
-F 0 "#PWR026" H 4350 3650 50  0001 C CNN
-F 1 "+5V" H 4365 3973 50  0000 C CNN
-F 2 "" H 4350 3800 50  0001 C CNN
-F 3 "" H 4350 3800 50  0001 C CNN
-	1    4350 3800
-	1    0    0    -1
-$EndComp
-Wire Wire Line
-	4350 3800 4350 4000
+P 4350 3500
+F 0 "#PWR026" H 4350 3350 50  0001 C CNN
+F 1 "+5V" H 4365 3673 50  0000 C CNN
+F 2 "" H 4350 3500 50  0001 C CNN
+F 3 "" H 4350 3500 50  0001 C CNN
+	1    4350 3500
+	1    0    0    -1
+$EndComp
 Wire Wire Line
 	4350 4000 4200 4000
@@
 L Connector:TestPoint TP5
 U 1 1 5B973A0D
-P 2100 4800
-F 0 "TP5" H 2158 4920 50  0000 L CNN
-F 1 "TestPoint" H 2158 4829 50  0000 L CNN
-F 2 "" H 2300 4800 50  0001 C CNN
-F 3 "~" H 2300 4800 50  0001 C CNN
-	1    2100 4800
-	1    0    0    -1
+P 1900 5100
+F 0 "TP5" H 2200 5100 50  0000 R CNN
+F 1 "TestPoint" H 2300 5200 50  0000 R CNN
+F 2 "" H 2100 5100 50  0001 C CNN
+F 3 "~" H 2100 5100 50  0001 C CNN
+	1    1900 5100
+	-1   0    0    1
 $EndComp
 $Comp
@@
 $EndComp
 Wire Wire Line
-	1800 4900 2100 4900
-Wire Wire Line
 	1800 5000 2100 5000
-Wire Wire Line
-	2100 4800 2100 4900
-Connection ~ 2100 4900
-Wire Wire Line
-	2100 4900 2750 4900
 Wire Wire Line
 	2100 5100 2100 5000
@@
 Wire Wire Line
 	10100 4700 9650 4700
+$Comp
+L device:C C8
+U 1 1 5B9B3193
+P 8500 5050
+F 0 "C8" H 8615 5096 50  0000 L CNN
+F 1 "10uF" H 8615 5005 50  0000 L CNN
+F 2 "" H 8538 4900 50  0001 C CNN
+F 3 "~" H 8500 5050 50  0001 C CNN
+	1    8500 5050
+	1    0    0    -1
+$EndComp
+$Comp
+L power:GND #PWR036
+U 1 1 5B9B3244
+P 8500 5200
+F 0 "#PWR036" H 8500 4950 50  0001 C CNN
+F 1 "GND" H 8505 5027 50  0000 C CNN
+F 2 "" H 8500 5200 50  0001 C CNN
+F 3 "" H 8500 5200 50  0001 C CNN
+	1    8500 5200
+	1    0    0    -1
+$EndComp
+Wire Wire Line
+	8500 4900 8500 4600
+Connection ~ 8500 4600
+$Comp
+L device:C C7
+U 1 1 5B9B40F8
+P 4550 3650
+F 0 "C7" V 4298 3650 50  0000 C CNN
+F 1 "0.1uF" V 4389 3650 50  0000 C CNN
+F 2 "" H 4588 3500 50  0001 C CNN
+F 3 "~" H 4550 3650 50  0001 C CNN
+	1    4550 3650
+	0    1    1    0
+$EndComp
+$Comp
+L power:GND #PWR035
+U 1 1 5B9B41BF
+P 4700 3650
+F 0 "#PWR035" H 4700 3400 50  0001 C CNN
+F 1 "GND" H 4705 3477 50  0000 C CNN
+F 2 "" H 4700 3650 50  0001 C CNN
+F 3 "" H 4700 3650 50  0001 C CNN
+	1    4700 3650
+	1    0    0    -1
+$EndComp
+Wire Wire Line
+	4350 3500 4350 3650
+Wire Wire Line
+	4400 3650 4350 3650
+Connection ~ 4350 3650
+Wire Wire Line
+	4350 3650 4350 4000
+Wire Wire Line
+	1800 4900 1900 4900
+Wire Wire Line
+	1900 5100 1900 4900
+Connection ~ 1900 4900
+Wire Wire Line
+	1900 4900 2750 4900
+Text Label 2550 4700 2    50   ~ 0
+OSC1
+Text Label 2550 4800 2    50   ~ 0
+OSC2
+Wire Wire Line
+	2550 4700 2750 4700
+Wire Wire Line
+	2550 4800 2750 4800
+$Comp
+L device:Crystal Y1
+U 1 1 5B9BE86F
+P 3600 6500
+F 0 "Y1" V 3554 6631 50  0000 L CNN
+F 1 "Crystal" V 3645 6631 50  0000 L CNN
+F 2 "" H 3600 6500 50  0001 C CNN
+F 3 "~" H 3600 6500 50  0001 C CNN
+	1    3600 6500
+	0    1    1    0
+$EndComp
+$Comp
+L device:C C9
+U 1 1 5B9BEA08
+P 3150 6250
+F 0 "C9" V 2898 6250 50  0000 C CNN
+F 1 "26pF" V 2989 6250 50  0000 C CNN
+F 2 "" H 3188 6100 50  0001 C CNN
+F 3 "~" H 3150 6250 50  0001 C CNN
+	1    3150 6250
+	0    1    1    0
+$EndComp
+$Comp
+L device:C C10
+U 1 1 5B9BEAA4
+P 3150 6750
+F 0 "C10" V 2898 6750 50  0000 C CNN
+F 1 "26pF" V 2989 6750 50  0000 C CNN
+F 2 "" H 3188 6600 50  0001 C CNN
+F 3 "~" H 3150 6750 50  0001 C CNN
+	1    3150 6750
+	0    1    1    0
+$EndComp
+Wire Wire Line
+	3300 6250 3600 6250
+Wire Wire Line
+	3600 6250 3600 6350
+Wire Wire Line
+	3300 6750 3600 6750
+Wire Wire Line
+	3600 6750 3600 6650
+Text Label 3950 6250 0    50   ~ 0
+OSC1
+Text Label 3950 6750 0    50   ~ 0
+OSC2
+Wire Wire Line
+	3950 6250 3600 6250
+Connection ~ 3600 6250
+Wire Wire Line
+	3950 6750 3600 6750
+Connection ~ 3600 6750
+Wire Wire Line
+	3000 6250 2850 6250
+Wire Wire Line
+	2850 6250 2850 6500
+Wire Wire Line
+	2850 6750 3000 6750
+$Comp
+L power:GND #PWR037
+U 1 1 5B9C3A58
+P 2650 6550
+F 0 "#PWR037" H 2650 6300 50  0001 C CNN
+F 1 "GND" H 2655 6377 50  0000 C CNN
+F 2 "" H 2650 6550 50  0001 C CNN
+F 3 "" H 2650 6550 50  0001 C CNN
+	1    2650 6550
+	1    0    0    -1
+$EndComp
+Wire Wire Line
+	2650 6550 2650 6500
+Wire Wire Line
+	2650 6500 2850 6500
+Connection ~ 2850 6500
+Wire Wire Line
+	2850 6500 2850 6750
+$Comp
+L Connector:Conn_01x04_Female J6
+U 1 1 5B9D02A5
+P 1450 4200
+F 0 "J6" H 1344 4485 50  0000 C CNN
+F 1 "Conn_01x04_Female" H 1344 4394 50  0000 C CNN
+F 2 "" H 1450 4200 50  0001 C CNN
+F 3 "~" H 1450 4200 50  0001 C CNN
+	1    1450 4200
+	-1   0    0    -1
+$EndComp
+Wire Wire Line
+	1650 4100 2750 4100
+Wire Wire Line
+	1650 4200 2750 4200
+Wire Wire Line
+	1650 4300 2750 4300
+Wire Wire Line
+	1650 4400 2750 4400
+NoConn ~ 2750 4500
+NoConn ~ 2750 4600
+NoConn ~ 2750 5100
+NoConn ~ 2750 5200
+NoConn ~ 2750 5300
+NoConn ~ 4200 4900
+NoConn ~ 4200 5000
+NoConn ~ 4200 5100
 $EndSCHEMATC

Commit message: Picdev pcb first draft
Parts:
- C10, C7, C9: footprint (none) -> Capacitors_SMD:C_0805_HandSoldering
- C8: footprint (none) -> Capacitor_THT:CP_Radial_D5.0mm_P2.50mm
- D3, D4, D5, D6, D7: footprint (none) -> LED_SMD:LED_1206_3216Metric
- J3: footprint (none) -> Pin_Headers:Pin_Header_Straight_1x05_Pitch2.54mm
- J6: footprint (none) -> Pin_Headers:Pin_Header_Straight_1x04_Pitch2.54mm
- R10, R11, R6, R7, R8, R9: footprint (none) -> Resistors_SMD:R_0805_HandSoldering
- TP5, TP6: footprint (none) -> TestPoint:TestPoint_Pad_D2.0mm
- U5: footprint (none) -> Housings_DIP:DIP-8_W7.62mm
- U6: footprint (none) -> Housings_DIP:DIP-28_W7.62mm
- Y1: footprint (none) -> Crystal:Crystal_HC49-4H_Vertical
Changed lines of the file:
@@
 EESchema Schematic File Version 4
+LIBS:picdev-cache
 EELAYER 26 0
 EELAYER END
@@
 F 0 "U6" H 3475 5565 50  0000 C CNN
 F 1 "PIC18F26K83" H 3475 5474 50  0000 C CNN
-F 2 "" H 3950 4650 50  0001 C CNN
+F 2 "Housings_DIP:DIP-28_W7.62mm" H 3950 4650 50  0001 C CNN
 F 3 "" H 3950 4650 50  0001 C CNN
 	1    3500 4650
@@
 F 0 "U5" H 9175 4765 50  0000 C CNN
 F 1 "MCP2562" H 9175 4674 50  0000 C CNN
-F 2 "" H 9200 4500 50  0001 C CNN
+F 2 "Housings_DIP:DIP-8_W7.62mm" H 9200 4500 50  0001 C CNN
 F 3 "" H 9200 4500 50  0001 C CNN
 	1    9200 4500
@@
 F 0 "J3" H 3350 1650 50  0000 C CNN
 F 1 "Programming Header" H 3000 1750 50  0000 C CNN
-F 2 "" H 3000 2100 50  0001 C CNN
+F 2 "Pin_Headers:Pin_Header_Straight_1x05_Pitch2.54mm" H 3000 2100 50  0001 C CNN
 F 3 "~" H 3000 2100 50  0001 C CNN
 	1    3000 2100
@@
 F 0 "R6" H 2620 3696 50  0000 L CNN
 F 1 "1OK" H 2620 3605 50  0000 L CNN
-F 2 "" V 2480 3650 50  0001 C CNN
+F 2 "Resistors_SMD:R_0805_HandSoldering" V 2480 3650 50  0001 C CNN
 F 3 "~" H 2550 3650 50  0001 C CNN
 	1    2550 3650
@@
 F 0 "D3" V 5238 3733 50  0000 R CNN
 F 1 "LED" V 5147 3733 50  0000 R CNN
-F 2 "" H 5200 3850 50  0001 C CNN
+F 2 "LED_SMD:LED_1206_3216Metric" H 5200 3850 50  0001 C CNN
 F 3 "~" H 5200 3850 50  0001 C CNN
 	1    5200 3850
@@
 F 0 "R7" H 5270 4196 50  0000 L CNN
 F 1 "330R" H 5270 4105 50  0000 L CNN
-F 2 "" V 5130 4150 50  0001 C CNN
+F 2 "Resistors_SMD:R_0805_HandSoldering" V 5130 4150 50  0001 C CNN
 F 3 "~" H 5200 4150 50  0001 C CNN
 	1    5200 4150
@@
 F 0 "D4" V 5588 3733 50  0000 R CNN
 F 1 "LED" V 5497 3733 50  0000 R CNN
-F 2 "" H 5550 3850 50  0001 C CNN
+F 2 "LED_SMD:LED_1206_3216Metric" H 5550 3850 50  0001 C CNN
 F 3 "~" H 5550 3850 50  0001 C CNN
 	1    5550 3850
@@
 F 0 "R8" H 5620 4196 50  0000 L CNN
 F 1 "330R" H 5620 4105 50  0000 L CNN
-F 2 "" V 5480 4150 50  0001 C CNN
+F 2 "Resistors_SMD:R_0805_HandSoldering" V 5480 4150 50  0001 C CNN
 F 3 "~" H 5550 4150 50  0001 C CNN
 	1    5550 4150
@@
 F 0 "D5" V 5938 3733 50  0000 R CNN
 F 1 "LED" V 5847 3733 50  0000 R CNN
-F 2 "" H 5900 3850 50  0001 C CNN
+F 2 "LED_SMD:LED_1206_3216Metric" H 5900 3850 50  0001 C CNN
 F 3 "~" H 5900 3850 50  0001 C CNN
 	1    5900 3850
@@
 F 0 "R9" H 5970 4196 50  0000 L CNN
 F 1 "330R" H 5970 4105 50  0000 L CNN
-F 2 "" V 5830 4150 50  0001 C CNN
+F 2 "Resistors_SMD:R_0805_HandSoldering" V 5830 4150 50  0001 C CNN
 F 3 "~" H 5900 4150 50  0001 C CNN
 	1    5900 4150
@@
 F 0 "D6" V 6288 3733 50  0000 R CNN
 F 1 "LED" V 6197 3733 50  0000 R CNN
-F 2 "" H 6250 3850 50  0001 C CNN
+F 2 "LED_SMD:LED_1206_3216Metric" H 6250 3850 50  0001 C CNN
 F 3 "~" H 6250 3850 50  0001 C CNN
 	1    6250 3850
@@
 F 0 "R10" H 6320 4196 50  0000 L CNN
 F 1 "330R" H 6320 4105 50  0000 L CNN
-F 2 "" V 6180 4150 50  0001 C CNN
+F 2 "Resistors_SMD:R_0805_HandSoldering" V 6180 4150 50  0001 C CNN
 F 3 "~" H 6250 4150 50  0001 C CNN
 	1    6250 4150
@@
 F 0 "D7" V 6638 3733 50  0000 R CNN
 F 1 "LED" V 6547 3733 50  0000 R CNN
-F 2 "" H 6600 3850 50  0001 C CNN
+F 2 "LED_SMD:LED_1206_3216Metric" H 6600 3850 50  0001 C CNN
 F 3 "~" H 6600 3850 50  0001 C CNN
 	1    6600 3850
@@
 F 0 "R11" H 6670 4196 50  0000 L CNN
 F 1 "330R" H 6670 4105 50  0000 L CNN
-F 2 "" V 6530 4150 50  0001 C CNN
+F 2 "Resistors_SMD:R_0805_HandSoldering" V 6530 4150 50  0001 C CNN
 F 3 "~" H 6600 4150 50  0001 C CNN
 	1    6600 4150
@@
 F 0 "TP5" H 2200 5100 50  0000 R CNN
 F 1 "TestPoint" H 2300 5200 50  0000 R CNN
-F 2 "" H 2100 5100 50  0001 C CNN
+F 2 "TestPoint:TestPoint_Pad_D2.0mm" H 2100 5100 50  0001 C CNN
 F 3 "~" H 2100 5100 50  0001 C CNN
 	1    1900 5100
@@
 F 0 "TP6" H 2042 5127 50  0000 R CNN
 F 1 "TestPoint" H 2042 5218 50  0000 R CNN
-F 2 "" H 2300 5100 50  0001 C CNN
+F 2 "TestPoint:TestPoint_Pad_D2.0mm" H 2300 5100 50  0001 C CNN
 F 3 "~" H 2300 5100 50  0001 C CNN
 	1    2100 5100
@@
 F 0 "C8" H 8615 5096 50  0000 L CNN
 F 1 "10uF" H 8615 5005 50  0000 L CNN
-F 2 "" H 8538 4900 50  0001 C CNN
+F 2 "Capacitor_THT:CP_Radial_D5.0mm_P2.50mm" H 8538 4900 50  0001 C CNN
 F 3 "~" H 8500 5050 50  0001 C CNN
 	1    8500 5050
@@
 F 0 "C7" V 4298 3650 50  0000 C CNN
 F 1 "0.1uF" V 4389 3650 50  0000 C CNN
-F 2 "" H 4588 3500 50  0001 C CNN
+F 2 "Capacitors_SMD:C_0805_HandSoldering" H 4588 3500 50  0001 C CNN
 F 3 "~" H 4550 3650 50  0001 C CNN
 	1    4550 3650
@@
 F 0 "Y1" V 3554 6631 50  0000 L CNN
 F 1 "Crystal" V 3645 6631 50  0000 L CNN
-F 2 "" H 3600 6500 50  0001 C CNN
+F 2 "Crystal:Crystal_HC49-4H_Vertical" H 3600 6500 50  0001 C CNN
 F 3 "~" H 3600 6500 50  0001 C CNN
 	1    3600 6500
@@
 F 0 "C9" V 2898 6250 50  0000 C CNN
 F 1 "26pF" V 2989 6250 50  0000 C CNN
-F 2 "" H 3188 6100 50  0001 C CNN
+F 2 "Capacitors_SMD:C_0805_HandSoldering" H 3188 6100 50  0001 C CNN
 F 3 "~" H 3150 6250 50  0001 C CNN
 	1    3150 6250
@@
 F 0 "C10" V 2898 6750 50  0000 C CNN
 F 1 "26pF" V 2989 6750 50  0000 C CNN
-F 2 "" H 3188 6600 50  0001 C CNN
+F 2 "Capacitors_SMD:C_0805_HandSoldering" H 3188 6600 50  0001 C CNN
 F 3 "~" H 3150 6750 50  0001 C CNN
 	1    3150 6750
@@
 F 0 "J6" H 1344 4485 50  0000 C CNN
 F 1 "Conn_01x04_Female" H 1344 4394 50  0000 C CNN
-F 2 "" H 1450 4200 50  0001 C CNN
+F 2 "Pin_Headers:Pin_Header_Straight_1x04_Pitch2.54mm" H 1450 4200 50  0001 C CNN
 F 3 "~" H 1450 4200 50  0001 C CNN
 	1    1450 4200

Commit message: Review changes
- change test point footprint
- generate gerbers
Parts:
- TP5, TP6: footprint TestPoint:TestPoint_Pad_D2.0mm -> TestPoint:TestPoint_THTPad_D2.0mm_Drill1.0mm
Changed lines of the file:
@@
 F 0 "TP5" H 2200 5100 50  0000 R CNN
 F 1 "TestPoint" H 2300 5200 50  0000 R CNN
-F 2 "TestPoint:TestPoint_Pad_D2.0mm" H 2100 5100 50  0001 C CNN
+F 2 "TestPoint:TestPoint_THTPad_D2.0mm_Drill1.0mm" H 2100 5100 50  0001 C CNN
 F 3 "~" H 2100 5100 50  0001 C CNN
 	1    1900 5100
@@
 F 0 "TP6" H 2042 5127 50  0000 R CNN
 F 1 "TestPoint" H 2042 5218 50  0000 R CNN
-F 2 "TestPoint:TestPoint_Pad_D2.0mm" H 2300 5100 50  0001 C CNN
+F 2 "TestPoint:TestPoint_THTPad_D2.0mm_Drill1.0mm" H 2300 5100 50  0001 C CNN
 F 3 "~" H 2300 5100 50  0001 C CNN
 	1    2100 5100
