File: rocketlog/rocketlog/logger_power.sch (KiCad schematic (older format))
At the start: 18 parts

Commit message: Rocketlog - Review Changes
Changes in this commit:
    - change capacitor on SD card power rail to 4.7uF. Not sure of proper value,
    but decoupling definitely is necessary (SD cards draw a lot of current).
    - Remove the SMPS, run the board off 5V CAN rail (3v3 LDO is still there)
    - Replace 4pin CAN connector with standard pinout 5pin connector
    - Put current sense amplifier on 5V rail instead of VBATT rail
    - Annotate the schematic (sorry)
    - change MCLR to ~MCLR
    - add polyfuse on 5V CAN bus rail
    - remove US style resistors, all resistors now EU metric apologist style
    - Set R_Sense and current gain values, full scale at 266mA (is this good?)
Parts:
- removed C? (x5): C, symbol Device:C
- removed D?: D_Zener, symbol Device:D_Zener
- removed J?: BUS_CONN, symbol Connector:Conn_01x04_Female
- removed L?: L, symbol Device:L
- removed R? (x3): R, symbol Device:R
- removed U?: TPS5405TR, symbol canhw:TPS5405TR
- added F1: Polyfuse, symbol Device:Polyfuse
- added J4: BUS CONN, symbol Connector:Conn_01x05_Female
- R5: renamed from R?; value R_sense -> 62mOhm
- gave numbers to parts that had none: 5
Connections:
- net labels removed: +BATT
- wire segments 53 -> 27
- no-connect marks 0 -> 1
Other:
- note added: "200V/V"
- note added: "62mR * I * 200v/v = 3.3V\nImax = 266mA"
- moved on the sheet: C10, C8, C9, R5, U3, U4

Commit message: Logger: Initial ballpark layout for logger, to see how big it should be
Some footprints are not final ones - CAN connector is wrong, crystal
is wrong, current sense resistor is probably wrong, SD card holder is
wrong. These are just ballpark estimates so that we can get an idea of
the order of magnitude of the size of the final board.
Parts:
- C10, C8, C9: footprint (none) -> Capacitor_SMD:C_0805_2012Metric_Pad1.15x1.40mm_HandSolder
- F1: footprint (none) -> Fuse:Fuse_1206_3216Metric_Pad1.42x1.75mm_HandSolder
- J4: footprint (none) -> Connector_Harwin:Harwin_LTek-Male_2x03_P2.00mm_Vertical_StrainRelief
- R5: footprint (none) -> Resistor_SMD:R_0805_2012Metric_Pad1.15x1.40mm_HandSolder
- U4: footprint (none) -> Package_TO_SOT_SMD:SOT-23-5_HandSoldering
Changed lines of the file:
@@
 F 0 "U4" H 4850 3528 50  0000 C CNN
 F 1 "INA180" H 4850 3437 50  0000 C CNN
-F 2 "" H 4900 4000 50  0001 C CNN
+F 2 "Package_TO_SOT_SMD:SOT-23-5_HandSoldering" H 4900 4000 50  0001 C CNN
 F 3 "" H 4900 4000 50  0001 C CNN
 	1    4900 4000
@@
 F 0 "R5" V 3943 3050 50  0000 C CNN
 F 1 "62mOhm" V 4034 3050 50  0000 C CNN
-F 2 "" V 4080 3050 50  0001 C CNN
+F 2 "Resistor_SMD:R_0805_2012Metric_Pad1.15x1.40mm_HandSolder" V 4080 3050 50  0001 C CNN
 F 3 "~" H 4150 3050 50  0001 C CNN
 	1    4150 3050
@@
 F 0 "C8" V 4748 3450 50  0000 C CNN
 F 1 "0.1u" V 4839 3450 50  0000 C CNN
-F 2 "" H 5038 3300 50  0001 C CNN
+F 2 "Capacitor_SMD:C_0805_2012Metric_Pad1.15x1.40mm_HandSolder" H 5038 3300 50  0001 C CNN
 F 3 "~" H 5000 3450 50  0001 C CNN
 	1    5000 3450
@@
 F 0 "C10" H 6935 3954 50  0000 R CNN
 F 1 "4.7u" H 6935 4045 50  0000 R CNN
-F 2 "" H 7088 3850 50  0001 C CNN
+F 2 "Capacitor_SMD:C_0805_2012Metric_Pad1.15x1.40mm_HandSolder" H 7088 3850 50  0001 C CNN
 F 3 "~" H 7050 4000 50  0001 C CNN
 	1    7050 4000
@@
 F 0 "C9" H 8285 3904 50  0000 R CNN
 F 1 "4.7u" H 8285 3995 50  0000 R CNN
-F 2 "" H 8438 3800 50  0001 C CNN
+F 2 "Capacitor_SMD:C_0805_2012Metric_Pad1.15x1.40mm_HandSolder" H 8438 3800 50  0001 C CNN
 F 3 "~" H 8400 3950 50  0001 C CNN
 	1    8400 3950
@@
 F 0 "J4" H 2644 2725 50  0000 C CNN
 F 1 "BUS CONN" H 2644 2816 50  0000 C CNN
-F 2 "" H 2750 3150 50  0001 C CNN
+F 2 "Connector_Harwin:Harwin_LTek-Male_2x03_P2.00mm_Vertical_StrainRelief" H 2750 3150 50  0001 C CNN
 F 3 "~" H 2750 3150 50  0001 C CNN
 	1    2750 3150
@@
 F 0 "F1" V 3125 3050 50  0000 C CNN
 F 1 "Polyfuse" V 3216 3050 50  0000 C CNN
-F 2 "" H 3400 2850 50  0001 L CNN
+F 2 "Fuse:Fuse_1206_3216Metric_Pad1.42x1.75mm_HandSolder" H 3400 2850 50  0001 L CNN
 F 3 "~" H 3350 3050 50  0001 C CNN
 	1    3350 3050

Commit message: Logger: route traces - got 95% of the way there
Required remapping a bunch of SD card pins. Only things that I
couldn't manage to route onto a 4cm by 6cm single sided board was the
current sense line, and a couple of ground pour islands. It should be
doable with maybe one or two jumpers. I want to try rotating the
microcontroller 90 degrees CCW, that should make the current sense
line easier, as well as some of the SD card stuff.
Parts:
- J4: footprint Connector_Harwin:Harwin_LTek-Male_2x03_P2.00mm_Vertical_StrainRelief -> canhw_footprints:connector_Harwin_M80-4120642-ND
Changed lines of the file:
@@
 F 0 "J4" H 2644 2725 50  0000 C CNN
 F 1 "BUS CONN" H 2644 2816 50  0000 C CNN
-F 2 "Connector_Harwin:Harwin_LTek-Male_2x03_P2.00mm_Vertical_StrainRelief" H 2750 3150 50  0001 C CNN
+F 2 "canhw_footprints:connector_Harwin_M80-4120642-ND" H 2750 3150 50  0001 C CNN
 F 3 "~" H 2750 3150 50  0001 C CNN
 	1    2750 3150

Commit message: Logger Board PCB Review 1 changes
Changes in this commit:
        - Move C2 further from U1
        - Space out F1, R5, U4 and C8
        - Silkscreen rearrangements to make it pretty
        - Replace J1 (SMT programming header) with a 90 degree connector
        - Replace U3 with hand soldering footprints
        - Turn mounting holes into plated holes
        - Remove daisy chaining through pads. I hope I got all of them, please check
        - Get rid of the power trace running through the SD card housing....
        - Move SD card holders down, so the SD cards don't overhand the board
        - Add rocketry logo to front silkscreen for that sweet sweet brand value
Parts:
- U3: footprint Package_TO_SOT_SMD:SOT-23-5 -> Package_TO_SOT_SMD:SOT-23-5_HandSoldering
Changed lines of the file:
@@
 F 0 "U3" H 7800 4192 50  0000 C CNN
 F 1 "AP2114H-3.3" H 7800 4101 50  0000 C CNN
-F 2 "Package_TO_SOT_SMD:SOT-23-5" H 7800 4175 50  0001 C CNN
+F 2 "Package_TO_SOT_SMD:SOT-23-5_HandSoldering" H 7800 4175 50  0001 C CNN
 F 3 "https://www.diodes.com/assets/Datasheets/AP2112.pdf" H 7800 3950 50  0001 C CNN
 	1    7800 3850

Commit message: Logger Board: Update CAN connector to use 90 degree SMD, not vertical SMD
Parts:
- J4: footprint canhw_footprints:connector_Harwin_M80-4120642-ND -> canhw_footprints:connector_Harwin_M80-5420642
Changed lines of the file:
@@
 F 0 "J4" H 2644 2725 50  0000 C CNN
 F 1 "BUS CONN" H 2644 2816 50  0000 C CNN
-F 2 "canhw_footprints:connector_Harwin_M80-4120642-ND" H 2750 3150 50  0001 C CNN
+F 2 "canhw_footprints:connector_Harwin_M80-5420642" H 2750 3150 50  0001 C CNN
 F 3 "~" H 2750 3150 50  0001 C CNN
 	1    2750 3150
