File: rocketlog/rocketlog/rocketlog.sch (KiCad schematic (older format))
At the start: 15 parts

Commit message: Rocketlog - Review Changes
Changes in this commit:
    - change capacitor on SD card power rail to 4.7uF. Not sure of proper value,
    but decoupling definitely is necessary (SD cards draw a lot of current).
    - Remove the SMPS, run the board off 5V CAN rail (3v3 LDO is still there)
    - Replace 4pin CAN connector with standard pinout 5pin connector
    - Put current sense amplifier on 5V rail instead of VBATT rail
    - Annotate the schematic (sorry)
    - change MCLR to ~MCLR
    - add polyfuse on 5V CAN bus rail
    - remove US style resistors, all resistors now EU metric apologist style
    - Set R_Sense and current gain values, full scale at 266mA (is this good?)
Parts:
- removed R? (x2): 330, symbol Device:R_US
- added R3, R4: 330, symbol Device:R
- gave numbers to parts that had none: 13
Connections:
- net labels added: ~MCLR
- net labels removed: MCLR
Changed lines of the file:
@@
 $Descr A4 11693 8268
 encoding utf-8
-Sheet 1 5
+Sheet 1 4
 Title ""
 Date ""
@@
 $EndDescr
 $Comp
-L canhw:DSPIC33EP512GP502 U?
+L canhw:DSPIC33EP512GP502 U1
 U 1 1 5B9D0DB3
 P 5800 3950
-F 0 "U?" H 7150 2750 50  0000 C CNN
+F 0 "U1" H 7150 2750 50  0000 C CNN
 F 1 "DSPIC33EP512GP502" H 6700 2950 50  0000 C CNN
 F 2 "Package_DIP:DIP-28_W7.62mm" H 5800 3950 50  0001 C CNN
@@
 $EndComp
 $Comp
-L Device:R R?
+L Device:R R1
 U 1 1 5B9D0F02
 P 3700 3000
-F 0 "R?" H 3770 3046 50  0000 L CNN
+F 0 "R1" H 3770 3046 50  0000 L CNN
 F 1 "10K" H 3770 2955 50  0000 L CNN
 F 2 "" V 3630 3000 50  0001 C CNN
@@
 $EndComp
 $Comp
-L power:+3.3V #PWR?
+L power:+3.3V #PWR07
 U 1 1 5B9D0FA1
 P 3700 2750
-F 0 "#PWR?" H 3700 2600 50  0001 C CNN
+F 0 "#PWR07" H 3700 2600 50  0001 C CNN
 F 1 "+3.3V" H 3715 2923 50  0000 C CNN
 F 2 "" H 3700 2750 50  0001 C CNN
@@
 	3700 3250 3700 3150
 Text Label 3450 3250 2    50   ~ 0
-MCLR
+~MCLR
 Wire Wire Line
 	3450 3250 3700 3250
 $Comp
-L Device:C C?
+L Device:C C1
 U 1 1 5B9D1079
 P 5450 2500
-F 0 "C?" V 5198 2500 50  0000 C CNN
+F 0 "C1" V 5198 2500 50  0000 C CNN
 F 1 "0.1u" V 5289 2500 50  0000 C CNN
 F 2 "" H 5488 2350 50  0001 C CNN
@@
 $EndComp
 $Comp
-L Device:C C?
+L Device:C C2
 U 1 1 5B9D10DB
 P 6150 2500
-F 0 "C?" V 5898 2500 50  0000 C CNN
+F 0 "C2" V 5898 2500 50  0000 C CNN
 F 1 "0.1u" V 5989 2500 50  0000 C CNN
 F 2 "" H 6188 2350 50  0001 C CNN
@@
 	5900 2500 5950 2500
 $Comp
-L power:GND #PWR?
+L power:GND #PWR05
 U 1 1 5B9D11ED
 P 5200 2550
-F 0 "#PWR?" H 5200 2300 50  0001 C CNN
+F 0 "#PWR05" H 5200 2300 50  0001 C CNN
 F 1 "GND" H 5205 2377 50  0000 C CNN
 F 2 "" H 5200 2550 50  0001 C CNN
@@
 	5200 2500 5300 2500
 $Comp
-L power:GND #PWR?
+L power:GND #PWR06
 U 1 1 5B9D1253
 P 6400 2550
-F 0 "#PWR?" H 6400 2300 50  0001 C CNN
+F 0 "#PWR06" H 6400 2300 50  0001 C CNN
 F 1 "GND" H 6405 2377 50  0000 C CNN
 F 2 "" H 6400 2550 50  0001 C CNN
@@
 	6400 2500 6300 2500
 $Comp
-L power:+3.3V #PWR?
+L power:+3.3V #PWR03
 U 1 1 5B9D131A
 P 5650 2300
-F 0 "#PWR?" H 5650 2150 50  0001 C CNN
+F 0 "#PWR03" H 5650 2150 50  0001 C CNN
 F 1 "+3.3V" H 5665 2473 50  0000 C CNN
 F 2 "" H 5650 2300 50  0001 C CNN
@@
 $EndComp
 $Comp
-L power:+3.3V #PWR?
+L power:+3.3V #PWR04
 U 1 1 5B9D14F7
 P 5950 2300
-F 0 "#PWR?" H 5950 2150 50  0001 C CNN
+F 0 "#PWR04" H 5950 2150 50  0001 C CNN
 F 1 "+3.3V" H 5965 2473 50  0000 C CNN
 F 2 "" H 5950 2300 50  0001 C CNN
@@
 	5950 2500 6000 2500
 $Comp
-L Device:C C?
+L Device:C C3
 U 1 1 5B9D1690
 P 3950 3800
-F 0 "C?" H 4065 3846 50  0000 L CNN
+F 0 "C3" H 4065 3846 50  0000 L CNN
 F 1 "10u" H 4065 3755 50  0000 L CNN
 F 2 "" H 3988 3650 50  0001 C CNN
@@
 $EndComp
 $Comp
-L power:GND #PWR?
+L power:GND #PWR09
 U 1 1 5B9D1753
 P 3950 4000
-F 0 "#PWR?" H 3950 3750 50  0001 C CNN
+F 0 "#PWR09" H 3950 3750 50  0001 C CNN
 F 1 "GND" H 3955 3827 50  0000 C CNN
 F 2 "" H 3950 4000 50  0001 C CNN
@@
 	3950 3650 4200 3650
 $Comp
-L Device:R R?
+L Device:R R2
 U 1 1 5B9D1F66
 P 3950 3250
-F 0 "R?" V 3800 3250 50  0000 C BNN
+F 0 "R2" V 3800 3250 50  0000 C BNN
 F 1 "470" V 3850 3250 50  0000 C CNN
 F 2 "" V 3880 3250 50  0001 C CNN
@@
 	4100 3250 4200 3250
 $Comp
-L power:GND #PWR?
+L power:GND #PWR011
 U 1 1 5B9D2607
 P 5700 5250
-F 0 "#PWR?" H 5700 5000 50  0001 C CNN
+F 0 "#PWR011" H 5700 5000 50  0001 C CNN
 F 1 "GND" H 5705 5077 50  0000 C CNN
 F 2 "" H 5700 5250 50  0001 C CNN
@@
 $EndComp
 $Comp
-L power:GND #PWR?
+L power:GND #PWR012
 U 1 1 5B9D2625
 P 5900 5250
-F 0 "#PWR?" H 5900 5000 50  0001 C CNN
+F 0 "#PWR012" H 5900 5000 50  0001 C CNN
 F 1 "GND" H 5905 5077 50  0000 C CNN
 F 2 "" H 5900 5250 50  0001 C CNN
@@
 $EndComp
 $Comp
-L Device:Crystal Y?
+L Device:Crystal Y1
 U 1 1 5B9D28E5
 P 2750 5350
-F 0 "Y?" V 2650 5500 50  0000 L CNN
+F 0 "Y1" V 2650 5500 50  0000 L CNN
 F 1 "Crystal" V 2750 5500 50  0000 L CNN
 F 2 "" H 2750 5350 50  0001 C CNN
@@
 $EndComp
 $Comp
-L Device:C_Small C?
+L Device:C_Small C4
 U 1 1 5B9D2A77
 P 2500 5200
-F 0 "C?" V 2271 5200 50  0000 C CNN
+F 0 "C4" V 2271 5200 50  0000 C CNN
 F 1 "C_Small" V 2362 5200 50  0000 C CNN
 F 2 "" H 2500 5200 50  0001 C CNN
@@
 $EndComp
 $Comp
-L Device:C_Small C?
+L Device:C_Small C5
 U 1 1 5B9D2ABA
 P 2500 5500
-F 0 "C?" V 2700 5500 50  0000 C CNN
+F 0 "C5" V 2700 5500 50  0000 C CNN
 F 1 "C_Small" V 2600 5500 50  0000 C CNN
 F 2 "" H 2500 5500 50  0001 C CNN
@@
 	2300 5200 2400 5200
 $Comp
-L power:GND #PWR?
+L power:GND #PWR013
 U 1 1 5B9D31BD
 P 2150 5400
-F 0 "#PWR?" H 2150 5150 50  0001 C CNN
+F 0 "#PWR013" H 2150 5150 50  0001 C CNN
 F 1 "GND" H 2155 5227 50  0000 C CNN
 F 2 "" H 2150 5400 50  0001 C CNN
@@
 Connection ~ 2750 5200
 $Comp
-L Device:LED_Small D?
+L Device:LED_Small D2
 U 1 1 5B9F454C
 P 9850 4800
-F 0 "D?" V 9896 4732 50  0000 R CNN
+F 0 "D2" V 9896 4732 50  0000 R CNN
 F 1 "DEBUG2" V 9805 4732 50  0000 R CNN
 F 2 "" V 9850 4800 50  0001 C CNN
@@
 $EndComp
 $Comp
-L Device:LED_Small D?
+L Device:LED_Small D1
 U 1 1 5B9F46EE
 P 3100 4200
-F 0 "D?" V 3150 4350 50  0000 R CNN
+F 0 "D1" V 3150 4350 50  0000 R CNN
 F 1 "DEBUG1" V 3050 4550 50  0000 R CNN
 F 2 "" V 3100 4200 50  0001 C CNN
@@
 Text Label 4200 4650 2    50   ~ 0
 OSC2
-$Comp
-L Device:R_US R?
-U 1 1 5B9F90E6
-P 3100 3950
-F 0 "R?" H 2950 4000 50  0000 L CNN
-F 1 "330" H 2850 3900 50  0000 L CNN
-F 2 "" V 3140 3940 50  0001 C CNN
-F 3 "~" H 3100 3950 50  0001 C CNN
-	1    3100 3950
-	1    0    0    -1
-$EndComp
-$Comp
-L Device:R_US R?
-U 1 1 5B9F918A
-P 9850 4550
-F 0 "R?" H 9918 4596 50  0000 L CNN
-F 1 "330" H 9918 4505 50  0000 L CNN
-F 2 "" V 9890 4540 50  0001 C CNN
-F 3 "~" H 9850 4550 50  0001 C CNN
-	1    9850 4550
-	1    0    0    -1
-$EndComp
 Wire Wire Line
 	3100 4300 3100 4450
@@
 	3100 4450 4200 4450
 $Comp
-L power:+5V #PWR?
+L power:+5V #PWR08
 U 1 1 5B9FF5DB
 P 3100 3800
-F 0 "#PWR?" H 3100 3650 50  0001 C CNN
+F 0 "#PWR08" H 3100 3650 50  0001 C CNN
 F 1 "+5V" H 3115 3973 50  0000 C CNN
 F 2 "" H 3100 3800 50  0001 C CNN
@@
 $EndComp
 $Comp
-L power:+5V #PWR?
+L power:+5V #PWR010
 U 1 1 5B9FF607
 P 9850 4400
-F 0 "#PWR?" H 9850 4250 50  0001 C CNN
+F 0 "#PWR010" H 9850 4250 50  0001 C CNN
 F 1 "+5V" H 9865 4573 50  0000 C CNN
 F 2 "" H 9850 4400 50  0001 C CNN
@@
 $EndSheet
 $Comp
-L canhw:MCP2562 U?
+L canhw:MCP2562 U2
 U 1 1 5B9EA850
 P 8800 5700
-F 0 "U?" H 8775 5965 50  0000 C CNN
+F 0 "U2" H 8775 5965 50  0000 C CNN
 F 1 "MCP2562" H 8775 5874 50  0000 C CNN
 F 2 "" H 8800 5700 50  0001 C CNN
@@
 $EndComp
 $Comp
-L power:+5V #PWR?
+L power:+5V #PWR015
 U 1 1 5B9EA857
 P 8200 5550
-F 0 "#PWR?" H 8200 5400 50  0001 C CNN
+F 0 "#PWR015" H 8200 5400 50  0001 C CNN
 F 1 "+5V" H 8215 5723 50  0000 C CNN
 F 2 "" H 8200 5550 50  0001 C CNN
@@
 $EndComp
 $Comp
-L power:+3.3V #PWR?
+L power:+3.3V #PWR014
 U 1 1 5B9EA85D
 P 7950 5550
-F 0 "#PWR?" H 7950 5400 50  0001 C CNN
+F 0 "#PWR014" H 7950 5400 50  0001 C CNN
 F 1 "+3.3V" H 7965 5723 50  0000 C CNN
 F 2 "" H 7950 5550 50  0001 C CNN
@@
 	8200 5700 8300 5700
 $Comp
-L power:GND #PWR?
+L power:GND #PWR016
 U 1 1 5B9EA867
 P 9400 6150
-F 0 "#PWR?" H 9400 5900 50  0001 C CNN
+F 0 "#PWR016" H 9400 5900 50  0001 C CNN
 F 1 "GND" H 9405 5977 50  0000 C CNN
 F 2 "" H 9400 6150 50  0001 C CNN
@@
 ICSPCLK
 $Comp
-L Connector:Conn_01x05_Female J?
+L Connector:Conn_01x05_Female J1
 U 1 1 5B9ED738
 P 9950 1550
-F 0 "J?" H 9977 1576 50  0000 L CNN
+F 0 "J1" H 9977 1576 50  0000 L CNN
 F 1 "Conn_01x05_Female" H 9977 1485 50  0000 L CNN
 F 2 "" H 9950 1550 50  0001 C CNN
@@
 $EndComp
 Text Label 9750 1350 2    50   ~ 0
-MCLR
-$Comp
-L power:+3.3V #PWR?
+~MCLR
+$Comp
+L power:+3.3V #PWR01
 U 1 1 5B9ED8C4
 P 9350 1350
-F 0 "#PWR?" H 9350 1200 50  0001 C CNN
+F 0 "#PWR01" H 9350 1200 50  0001 C CNN
 F 1 "+3.3V" H 9365 1523 50  0000 C CNN
 F 2 "" H 9350 1350 50  0001 C CNN
@@
 ICSPCLK
 $Comp
-L power:GND #PWR?
+L power:GND #PWR02
 U 1 1 5B9EEE79
 P 9350 1800
-F 0 "#PWR?" H 9350 1550 50  0001 C CNN
+F 0 "#PWR02" H 9350 1550 50  0001 C CNN
 F 1 "GND" H 9355 1627 50  0000 C CNN
 F 2 "" H 9350 1800 50  0001 C CNN
@@
 Wire Wire Line
 	9350 1550 9750 1550
+$Comp
+L Device:R R3
+U 1 1 5BAC6D7D
+P 3100 3950
+F 0 "R3" H 3170 3996 50  0000 L CNN
+F 1 "330" H 3170 3905 50  0000 L CNN
+F 2 "" V 3030 3950 50  0001 C CNN
+F 3 "~" H 3100 3950 50  0001 C CNN
+	1    3100 3950
+	1    0    0    -1
+$EndComp
+$Comp
+L Device:R R4
+U 1 1 5BAC6DFE
+P 9850 4550
+F 0 "R4" H 9920 4596 50  0000 L CNN
+F 1 "330" H 9920 4505 50  0000 L CNN
+F 2 "" V 9780 4550 50  0001 C CNN
+F 3 "~" H 9850 4550 50  0001 C CNN
+	1    9850 4550
+	1    0    0    -1
+$EndComp
 $EndSCHEMATC

Commit message: Logger: Initial ballpark layout for logger, to see how big it should be
Some footprints are not final ones - CAN connector is wrong, crystal
is wrong, current sense resistor is probably wrong, SD card holder is
wrong. These are just ballpark estimates so that we can get an idea of
the order of magnitude of the size of the final board.
Parts:
- C1, C2, C3, C4, C5: footprint (none) -> Capacitor_SMD:C_0805_2012Metric_Pad1.15x1.40mm_HandSolder
- D1, D2: footprint (none) -> LED_SMD:LED_1206_3216Metric_Pad1.42x1.75mm_HandSolder
- J1: footprint (none) -> Connector_PinHeader_2.54mm:PinHeader_1x05_P2.54mm_Vertical_SMD_Pin1Right
- R1, R2, R3, R4: footprint (none) -> Resistor_SMD:R_0805_2012Metric_Pad1.15x1.40mm_HandSolder
- U1: footprint Package_DIP:DIP-28_W7.62mm -> Package_SO:SOIC-28W_7.5x17.9mm_P1.27mm
- U2: footprint (none) -> Package_SO:SOIC-8_3.9x4.9mm_P1.27mm
- Y1: footprint (none) -> Crystal:Crystal_SMD_0603-2Pin_6.0x3.5mm_HandSoldering
Changed lines of the file:
@@
 F 0 "U1" H 7150 2750 50  0000 C CNN
 F 1 "DSPIC33EP512GP502" H 6700 2950 50  0000 C CNN
-F 2 "Package_DIP:DIP-28_W7.62mm" H 5800 3950 50  0001 C CNN
+F 2 "Package_SO:SOIC-28W_7.5x17.9mm_P1.27mm" H 5800 3950 50  0001 C CNN
 F 3 "http://ww1.microchip.com/downloads/en/DeviceDoc/70000657H.pdf" H 5800 3950 50  0001 C CNN
 	1    5800 3950
@@
 F 0 "R1" H 3770 3046 50  0000 L CNN
 F 1 "10K" H 3770 2955 50  0000 L CNN
-F 2 "" V 3630 3000 50  0001 C CNN
+F 2 "Resistor_SMD:R_0805_2012Metric_Pad1.15x1.40mm_HandSolder" V 3630 3000 50  0001 C CNN
 F 3 "~" H 3700 3000 50  0001 C CNN
 	1    3700 3000
@@
 F 0 "C1" V 5198 2500 50  0000 C CNN
 F 1 "0.1u" V 5289 2500 50  0000 C CNN
-F 2 "" H 5488 2350 50  0001 C CNN
+F 2 "Capacitor_SMD:C_0805_2012Metric_Pad1.15x1.40mm_HandSolder" H 5488 2350 50  0001 C CNN
 F 3 "~" H 5450 2500 50  0001 C CNN
 	1    5450 2500
@@
 F 0 "C2" V 5898 2500 50  0000 C CNN
 F 1 "0.1u" V 5989 2500 50  0000 C CNN
-F 2 "" H 6188 2350 50  0001 C CNN
+F 2 "Capacitor_SMD:C_0805_2012Metric_Pad1.15x1.40mm_HandSolder" H 6188 2350 50  0001 C CNN
 F 3 "~" H 6150 2500 50  0001 C CNN
 	1    6150 2500
@@
 F 0 "C3" H 4065 3846 50  0000 L CNN
 F 1 "10u" H 4065 3755 50  0000 L CNN
-F 2 "" H 3988 3650 50  0001 C CNN
+F 2 "Capacitor_SMD:C_0805_2012Metric_Pad1.15x1.40mm_HandSolder" H 3988 3650 50  0001 C CNN
 F 3 "~" H 3950 3800 50  0001 C CNN
 	1    3950 3800
@@
 F 0 "R2" V 3800 3250 50  0000 C BNN
 F 1 "470" V 3850 3250 50  0000 C CNN
-F 2 "" V 3880 3250 50  0001 C CNN
+F 2 "Resistor_SMD:R_0805_2012Metric_Pad1.15x1.40mm_HandSolder" V 3880 3250 50  0001 C CNN
 F 3 "~" H 3950 3250 50  0001 C CNN
 	1    3950 3250
@@
 F 0 "Y1" V 2650 5500 50  0000 L CNN
 F 1 "Crystal" V 2750 5500 50  0000 L CNN
-F 2 "" H 2750 5350 50  0001 C CNN
+F 2 "Crystal:Crystal_SMD_0603-2Pin_6.0x3.5mm_HandSoldering" H 2750 5350 50  0001 C CNN
 F 3 "~" H 2750 5350 50  0001 C CNN
 	1    2750 5350
@@
 F 0 "C4" V 2271 5200 50  0000 C CNN
 F 1 "C_Small" V 2362 5200 50  0000 C CNN
-F 2 "" H 2500 5200 50  0001 C CNN
+F 2 "Capacitor_SMD:C_0805_2012Metric_Pad1.15x1.40mm_HandSolder" H 2500 5200 50  0001 C CNN
 F 3 "~" H 2500 5200 50  0001 C CNN
 	1    2500 5200
@@
 F 0 "C5" V 2700 5500 50  0000 C CNN
 F 1 "C_Small" V 2600 5500 50  0000 C CNN
-F 2 "" H 2500 5500 50  0001 C CNN
+F 2 "Capacitor_SMD:C_0805_2012Metric_Pad1.15x1.40mm_HandSolder" H 2500 5500 50  0001 C CNN
 F 3 "~" H 2500 5500 50  0001 C CNN
 	1    2500 5500
@@
 F 0 "D2" V 9896 4732 50  0000 R CNN
 F 1 "DEBUG2" V 9805 4732 50  0000 R CNN
-F 2 "" V 9850 4800 50  0001 C CNN
+F 2 "LED_SMD:LED_1206_3216Metric_Pad1.42x1.75mm_HandSolder" V 9850 4800 50  0001 C CNN
 F 3 "~" V 9850 4800 50  0001 C CNN
 	1    9850 4800
@@
 F 0 "D1" V 3150 4350 50  0000 R CNN
 F 1 "DEBUG1" V 3050 4550 50  0000 R CNN
-F 2 "" V 3100 4200 50  0001 C CNN
+F 2 "LED_SMD:LED_1206_3216Metric_Pad1.42x1.75mm_HandSolder" V 3100 4200 50  0001 C CNN
 F 3 "~" V 3100 4200 50  0001 C CNN
 	1    3100 4200
@@
 F 0 "U2" H 8775 5965 50  0000 C CNN
 F 1 "MCP2562" H 8775 5874 50  0000 C CNN
-F 2 "" H 8800 5700 50  0001 C CNN
+F 2 "Package_SO:SOIC-8_3.9x4.9mm_P1.27mm" H 8800 5700 50  0001 C CNN
 F 3 "" H 8800 5700 50  0001 C CNN
 	1    8800 5700
@@
 F 0 "J1" H 9977 1576 50  0000 L CNN
 F 1 "Conn_01x05_Female" H 9977 1485 50  0000 L CNN
-F 2 "" H 9950 1550 50  0001 C CNN
+F 2 "Connector_PinHeader_2.54mm:PinHeader_1x05_P2.54mm_Vertical_SMD_Pin1Right" H 9950 1550 50  0001 C CNN
 F 3 "~" H 9950 1550 50  0001 C CNN
 	1    9950 1550
@@
 F 0 "R3" H 3170 3996 50  0000 L CNN
 F 1 "330" H 3170 3905 50  0000 L CNN
-F 2 "" V 3030 3950 50  0001 C CNN
+F 2 "Resistor_SMD:R_0805_2012Metric_Pad1.15x1.40mm_HandSolder" V 3030 3950 50  0001 C CNN
 F 3 "~" H 3100 3950 50  0001 C CNN
 	1    3100 3950
@@
 F 0 "R4" H 9920 4596 50  0000 L CNN
 F 1 "330" H 9920 4505 50  0000 L CNN
-F 2 "" V 9780 4550 50  0001 C CNN
+F 2 "Resistor_SMD:R_0805_2012Metric_Pad1.15x1.40mm_HandSolder" V 9780 4550 50  0001 C CNN
 F 3 "~" H 9850 4550 50  0001 C CNN
 	1    9850 4550
