File: sensors/analog_sense.sch (KiCad schematic (older format))
At the start: 11 parts

Commit message: Sensor board review changes
- annotate everything
- fix symbol library mapping
- fix debug header orientation
- add extra decoupling cap to mcu
- add a couple debug leds
- add 15V regulator (tht)
- add sensor comments
Parts:
- C18, C19: renamed from C?; symbol device:C -> Device:C
- R6, R7, R8: renamed from R?; symbol device:R_US -> Device:R_US
- gave numbers to parts that had none: 6
Other:
- note removed: "Lead wires < 10ft.\n3/4 wire not needed.\n(TI App Note)"
Changed lines of the file:
@@
 EESchema Schematic File Version 4
-LIBS:sensors-cache
 EELAYER 26 0
 EELAYER END
@@
 $EndDescr
 $Comp
-L flight_instr:74HC4051D U?
+L flight_instr:74HC4051D U12
 U 1 1 5BB4F094
 P 2650 2050
-F 0 "U?" H 2625 2737 60  0000 C CNN
+F 0 "U12" H 2625 2737 60  0000 C CNN
 F 1 "74HC4051D" H 2625 2631 60  0000 C CNN
 F 2 "" H 2600 2050 60  0001 C CNN
@@
 	1850 1800 2200 1800
 $Comp
-L power:+3V3 #PWR?
+L power:+3V3 #PWR055
 U 1 1 5BB4FD46
 P 2100 1450
-F 0 "#PWR?" H 2100 1300 50  0001 C CNN
+F 0 "#PWR055" H 2100 1300 50  0001 C CNN
 F 1 "+3V3" H 2115 1623 50  0000 C CNN
 F 2 "" H 2100 1450 50  0001 C CNN
@@
 	2100 1650 2200 1650
 $Comp
-L power:GND #PWR?
+L power:GND #PWR058
 U 1 1 5BB4FF10
 P 2100 2600
-F 0 "#PWR?" H 2100 2350 50  0001 C CNN
+F 0 "#PWR058" H 2100 2350 50  0001 C CNN
 F 1 "GND" H 2105 2427 50  0000 C CNN
 F 2 "" H 2100 2600 50  0001 C CNN
@@
 	2650 2700 2650 3050
 $Comp
-L Connector:Conn_01x04_Female J?
+L Connector:Conn_01x04_Female J3
 U 1 1 5BB51AC9
 P 6550 1550
-F 0 "J?" H 6577 1526 50  0000 L CNN
+F 0 "J3" H 6577 1526 50  0000 L CNN
 F 1 "Differential Pressure Conn" H 6577 1435 50  0000 L CNN
 F 2 "" H 6550 1550 50  0001 C CNN
@@
 DIFF_S+
 $Comp
-L power:GND #PWR?
+L power:GND #PWR056
 U 1 1 5BB51E98
 P 7100 1850
-F 0 "#PWR?" H 7100 1600 50  0001 C CNN
+F 0 "#PWR056" H 7100 1600 50  0001 C CNN
 F 1 "GND" H 7105 1677 50  0000 C CNN
 F 2 "" H 7100 1850 50  0001 C CNN
@@
 	7100 1750 6750 1750
 $Comp
-L canhw:INA826 U?
+L canhw:INA826 U11
 U 1 1 5BB51EC4
 P 8800 1550
-F 0 "U?" H 8800 1775 50  0000 C CNN
+F 0 "U11" H 8800 1775 50  0000 C CNN
 F 1 "INA826" H 8800 1684 50  0000 C CNN
 F 2 "" H 8800 1550 50  0001 C CNN
@@
 $EndComp
 $Comp
-L power:GND #PWR?
+L power:GND #PWR057
 U 1 1 5BB52074
 P 9350 1950
-F 0 "#PWR?" H 9350 1700 50  0001 C CNN
+F 0 "#PWR057" H 9350 1700 50  0001 C CNN
 F 1 "GND" H 9355 1777 50  0000 C CNN
 F 2 "" H 9350 1950 50  0001 C CNN
@@
 	9350 1550 9250 1550
 $Comp
-L power:+3V3 #PWR?
+L power:+3V3 #PWR052
 U 1 1 5BB6477C
 P 9350 1150
-F 0 "#PWR?" H 9350 1000 50  0001 C CNN
+F 0 "#PWR052" H 9350 1000 50  0001 C CNN
 F 1 "+3V3" H 9365 1323 50  0000 C CNN
 F 2 "" H 9350 1150 50  0001 C CNN
@@
 	6750 1650 7450 1650
 $Comp
-L device:R_US R?
+L Device:R_US R6
 U 1 1 5BB660AB
 P 8200 1650
-F 0 "R?" V 8200 1250 50  0000 C CNN
+F 0 "R6" V 8200 1250 50  0000 C CNN
 F 1 "R_US" V 8300 1300 50  0000 C CNN
 F 2 "" V 8240 1640 50  0001 C CNN
@@
 	8050 1750 8350 1750
 $Comp
-L power:+10V #PWR?
+L power:+10V #PWR054
 U 1 1 5BB66C0F
 P 7100 1350
-F 0 "#PWR?" H 7100 1200 50  0001 C CNN
+F 0 "#PWR054" H 7100 1200 50  0001 C CNN
 F 1 "+10V" H 7115 1523 50  0000 C CNN
 F 2 "" H 7100 1350 50  0001 C CNN
@@
 Wire Wire Line
 	7100 1450 6750 1450
-Text Notes 9550 1800 0    50   ~ 0
+Text Notes 7550 1500 0    50   ~ 0
 2 mV/V probably
 Text Label 3350 2050 0    50   ~ 0
@@
 	3350 2050 3050 2050
 $Comp
-L Connector:Conn_01x02_Female J?
+L Connector:Conn_01x02_Female J4
 U 1 1 5BB6EB08
 P 6500 3400
-F 0 "J?" H 6394 3585 50  0000 C CNN
+F 0 "J4" H 6394 3585 50  0000 C CNN
 F 1 "RTD Conn" H 6394 3494 50  0000 C CNN
 F 2 "" H 6500 3400 50  0001 C CNN
@@
 $EndComp
 $Comp
-L device:R_US R?
+L Device:R_US R7
 U 1 1 5BB6ECBD
 P 7200 3000
-F 0 "R?" H 7268 3046 50  0000 L CNN
+F 0 "R7" H 7268 3046 50  0000 L CNN
 F 1 "R_US" H 7268 2955 50  0000 L CNN
 F 2 "" V 7240 2990 50  0001 C CNN
@@
 $EndComp
 $Comp
-L power:+3V3 #PWR?
+L power:+3V3 #PWR062
 U 1 1 5BB6EDB6
 P 7200 2850
-F 0 "#PWR?" H 7200 2700 50  0001 C CNN
+F 0 "#PWR062" H 7200 2700 50  0001 C CNN
 F 1 "+3V3" H 7215 3023 50  0000 C CNN
 F 2 "" H 7200 2850 50  0001 C CNN
@@
 	6700 3400 7200 3400
 $Comp
-L power:GND #PWR?
+L power:GND #PWR063
 U 1 1 5BB6F57A
 P 7200 3600
-F 0 "#PWR?" H 7200 3350 50  0001 C CNN
+F 0 "#PWR063" H 7200 3350 50  0001 C CNN
 F 1 "GND" H 7205 3427 50  0000 C CNN
 F 2 "" H 7200 3600 50  0001 C CNN
@@
 	7200 3500 6700 3500
 $Comp
-L canhw:INA826 U?
+L canhw:INA826 U13
 U 1 1 5BB70118
 P 8800 3100
-F 0 "U?" H 8800 3325 50  0000 C CNN
+F 0 "U13" H 8800 3325 50  0000 C CNN
 F 1 "INA826" H 8800 3234 50  0000 C CNN
 F 2 "" H 8800 3100 50  0001 C CNN
@@
 Connection ~ 7200 3400
 $Comp
-L power:GND #PWR?
+L power:GND #PWR060
 U 1 1 5BB711C6
 P 8050 2800
-F 0 "#PWR?" H 8050 2550 50  0001 C CNN
+F 0 "#PWR060" H 8050 2550 50  0001 C CNN
 F 1 "GND" H 8055 2627 50  0000 C CNN
 F 2 "" H 8050 2800 50  0001 C CNN
@@
 	8350 2800 8350 3100
 $Comp
-L device:R_US R?
+L Device:R_US R8
 U 1 1 5BB719C4
 P 8100 3200
-F 0 "R?" V 8150 3550 50  0000 C CNN
+F 0 "R8" V 8150 3550 50  0000 C CNN
 F 1 "R_US" V 8050 3500 50  0000 C CNN
 F 2 "" V 8140 3190 50  0001 C CNN
@@
 todo: check common mode
 $Comp
-L power:GND #PWR?
+L power:GND #PWR064
 U 1 1 5BB72C19
 P 9500 3600
-F 0 "#PWR?" H 9500 3350 50  0001 C CNN
+F 0 "#PWR064" H 9500 3350 50  0001 C CNN
 F 1 "GND" H 9505 3427 50  0000 C CNN
 F 2 "" H 9500 3600 50  0001 C CNN
@@
 	9500 3400 9250 3400
 $Comp
-L power:+3V3 #PWR?
+L power:+3V3 #PWR059
 U 1 1 5BB735AE
 P 9500 2650
-F 0 "#PWR?" H 9500 2500 50  0001 C CNN
+F 0 "#PWR059" H 9500 2500 50  0001 C CNN
 F 1 "+3V3" H 9515 2823 50  0000 C CNN
 F 2 "" H 9500 2650 50  0001 C CNN
@@
 Wire Wire Line
 	9700 3200 9250 3200
-Text Notes 6450 4200 0    50   ~ 0
-Lead wires < 10ft.\n3/4 wire not needed.\n(TI App Note)
-$Comp
-L Connector:Conn_01x03_Female J?
+$Comp
+L Connector:Conn_01x03_Female J5
 U 1 1 5BB76C20
 P 6500 5250
-F 0 "J?" H 6394 5535 50  0000 C CNN
+F 0 "J5" H 6394 5535 50  0000 C CNN
 F 1 "Tank Pressure Conn" H 6394 5444 50  0000 C CNN
 F 2 "" H 6500 5250 50  0001 C CNN
@@
 $EndComp
 $Comp
-L power:+15V #PWR?
+L power:+15V #PWR065
 U 1 1 5BB76D88
 P 7250 4850
-F 0 "#PWR?" H 7250 4700 50  0001 C CNN
+F 0 "#PWR065" H 7250 4700 50  0001 C CNN
 F 1 "+15V" H 7265 5023 50  0000 C CNN
 F 2 "" H 7250 4850 50  0001 C CNN
@@
 	7250 5150 6700 5150
 $Comp
-L power:GND #PWR?
+L power:GND #PWR066
 U 1 1 5BB77B9E
 P 7250 5500
-F 0 "#PWR?" H 7250 5250 50  0001 C CNN
+F 0 "#PWR066" H 7250 5250 50  0001 C CNN
 F 1 "GND" H 7255 5327 50  0000 C CNN
 F 2 "" H 7250 5500 50  0001 C CNN
@@
 	9350 1150 9350 1300
 $Comp
-L device:C C?
+L Device:C C18
 U 1 1 5BB80ADB
 P 9600 1300
-F 0 "C?" V 9348 1300 50  0000 C CNN
+F 0 "C18" V 9348 1300 50  0000 C CNN
 F 1 "0.1uF" V 9439 1300 50  0000 C CNN
 F 2 "" H 9638 1150 50  0001 C CNN
@@
 	9350 1300 9350 1550
 $Comp
-L power:GND #PWR?
+L power:GND #PWR053
 U 1 1 5BB81C6C
 P 9750 1300
-F 0 "#PWR?" H 9750 1050 50  0001 C CNN
+F 0 "#PWR053" H 9750 1050 50  0001 C CNN
 F 1 "GND" H 9755 1127 50  0000 C CNN
 F 2 "" H 9750 1300 50  0001 C CNN
@@
 $EndComp
 $Comp
-L device:C C?
+L Device:C C19
 U 1 1 5BB82F9C
 P 9750 2800
-F 0 "C?" V 9498 2800 50  0000 C CNN
+F 0 "C19" V 9498 2800 50  0000 C CNN
 F 1 "0.1uF" V 9589 2800 50  0000 C CNN
 F 2 "" H 9788 2650 50  0001 C CNN
@@
 	9500 2800 9500 3100
 $Comp
-L power:GND #PWR?
+L power:GND #PWR061
 U 1 1 5BB87902
 P 9900 2800
-F 0 "#PWR?" H 9900 2550 50  0001 C CNN
+F 0 "#PWR061" H 9900 2550 50  0001 C CNN
 F 1 "GND" H 9905 2627 50  0000 C CNN
 F 2 "" H 9900 2800 50  0001 C CNN

Commit message: Assign most footprints
Parts:
- C18, C19: footprint (none) -> Capacitor_SMD:C_0805_2012Metric_Pad1.15x1.40mm_HandSolder
- R6, R7, R8: footprint (none) -> Resistor_SMD:R_0805_2012Metric_Pad1.15x1.40mm_HandSolder
Changed lines of the file:
@@
 F 0 "R6" V 8200 1250 50  0000 C CNN
 F 1 "R_US" V 8300 1300 50  0000 C CNN
-F 2 "" V 8240 1640 50  0001 C CNN
+F 2 "Resistor_SMD:R_0805_2012Metric_Pad1.15x1.40mm_HandSolder" V 8240 1640 50  0001 C CNN
 F 3 "~" H 8200 1650 50  0001 C CNN
 	1    8200 1650
@@
 F 0 "R7" H 7268 3046 50  0000 L CNN
 F 1 "R_US" H 7268 2955 50  0000 L CNN
-F 2 "" V 7240 2990 50  0001 C CNN
+F 2 "Resistor_SMD:R_0805_2012Metric_Pad1.15x1.40mm_HandSolder" V 7240 2990 50  0001 C CNN
 F 3 "~" H 7200 3000 50  0001 C CNN
 	1    7200 3000
@@
 F 0 "R8" V 8150 3550 50  0000 C CNN
 F 1 "R_US" V 8050 3500 50  0000 C CNN
-F 2 "" V 8140 3190 50  0001 C CNN
+F 2 "Resistor_SMD:R_0805_2012Metric_Pad1.15x1.40mm_HandSolder" V 8140 3190 50  0001 C CNN
 F 3 "~" H 8100 3200 50  0001 C CNN
 	1    8100 3200
@@
 F 0 "C18" V 9348 1300 50  0000 C CNN
 F 1 "0.1uF" V 9439 1300 50  0000 C CNN
-F 2 "" H 9638 1150 50  0001 C CNN
+F 2 "Capacitor_SMD:C_0805_2012Metric_Pad1.15x1.40mm_HandSolder" H 9638 1150 50  0001 C CNN
 F 3 "~" H 9600 1300 50  0001 C CNN
 	1    9600 1300
@@
 F 0 "C19" V 9498 2800 50  0000 C CNN
 F 1 "0.1uF" V 9589 2800 50  0000 C CNN
-F 2 "" H 9788 2650 50  0001 C CNN
+F 2 "Capacitor_SMD:C_0805_2012Metric_Pad1.15x1.40mm_HandSolder" H 9788 2650 50  0001 C CNN
 F 3 "~" H 9750 2800 50  0001 C CNN
 	1    9750 2800

Commit message: WIP sensor layout board
Parts:
- removed U13: INA826, symbol canhw:INA826
- added R19: R_US, Resistor_SMD:R_0805_2012Metric_Pad1.15x1.40mm_HandSolder, symbol Device:R_US
- added U13: MCP6001U, TO_SOT_Packages_SMD:SOT-23-5_HandSoldering, symbol Amplifier_Operational:MCP6001U
- J3: footprint (none) -> Connector_JST:JST_PH_S4B-PH-K_1x04_P2.00mm_Horizontal
- J4: footprint (none) -> Connector_JST:JST_PH_S2B-PH-K_1x02_P2.00mm_Horizontal
- J5: footprint (none) -> Connector_JST:JST_PH_S3B-PH-K_1x03_P2.00mm_Horizontal
- U11: footprint (none) -> Housings_SOIC:SO-8_5.3x6.2mm_Pitch1.27mm
- U12: footprint (none) -> Housings_SSOP:SSOP-16_4.4x5.2mm_Pitch0.65mm
Connections:
- wire segments 67 -> 65
Other:
- note removed: "todo: check common mode"
Changed lines of the file:
@@
 $Descr A4 11693 8268
 encoding utf-8
-Sheet 5 9
+Sheet 4 9
 Title ""
 Date ""
@@
 F 0 "U12" H 2625 2737 60  0000 C CNN
 F 1 "74HC4051D" H 2625 2631 60  0000 C CNN
-F 2 "" H 2600 2050 60  0001 C CNN
+F 2 "Housings_SSOP:SSOP-16_4.4x5.2mm_Pitch0.65mm" H 2600 2050 60  0001 C CNN
 F 3 "" H 2600 2050 60  0001 C CNN
 	1    2650 2050
@@
 Text HLabel 1850 3050 0    50   Input ~ 0
 MUX_OUT
-Text Label 3350 1650 0    50   ~ 0
+Text Label 3350 2050 0    50   ~ 0
 RTD
 Text HLabel 3350 2250 2    50   Input ~ 0
@@
 Text HLabel 3350 2150 2    50   Input ~ 0
 CURR_AMP_12V
+Text Label 3350 1850 0    50   ~ 0
+THERM_0
 Text Label 3350 1750 0    50   ~ 0
-THERM_0
-Text Label 3350 1850 0    50   ~ 0
 THERM_1
-Text Label 3350 1950 0    50   ~ 0
+Text Label 3350 1650 0    50   ~ 0
 THERM_2
 Wire Wire Line
@@
 F 0 "J3" H 6577 1526 50  0000 L CNN
 F 1 "Differential Pressure Conn" H 6577 1435 50  0000 L CNN
-F 2 "" H 6550 1550 50  0001 C CNN
+F 2 "Connector_JST:JST_PH_S4B-PH-K_1x04_P2.00mm_Horizontal" H 6550 1550 50  0001 C CNN
 F 3 "~" H 6550 1550 50  0001 C CNN
 	1    6550 1550
@@
 F 0 "U11" H 8800 1775 50  0000 C CNN
 F 1 "INA826" H 8800 1684 50  0000 C CNN
-F 2 "" H 8800 1550 50  0001 C CNN
+F 2 "Housings_SOIC:SO-8_5.3x6.2mm_Pitch1.27mm" H 8800 1550 50  0001 C CNN
 F 3 "" H 8800 1550 50  0001 C CNN
 	1    8800 1550
@@
 Text Notes 7550 1500 0    50   ~ 0
 2 mV/V probably
-Text Label 3350 2050 0    50   ~ 0
+Text Label 3350 1950 0    50   ~ 0
 THERM_3
 Wire Wire Line
@@
 F 0 "J4" H 6394 3585 50  0000 C CNN
 F 1 "RTD Conn" H 6394 3494 50  0000 C CNN
-F 2 "" H 6500 3400 50  0001 C CNN
+F 2 "Connector_JST:JST_PH_S2B-PH-K_1x02_P2.00mm_Horizontal" H 6500 3400 50  0001 C CNN
 F 3 "~" H 6500 3400 50  0001 C CNN
 	1    6500 3400
@@
 Wire Wire Line
 	7200 3500 6700 3500
-$Comp
-L canhw:INA826 U13
-U 1 1 5BB70118
-P 8800 3100
-F 0 "U13" H 8800 3325 50  0000 C CNN
-F 1 "INA826" H 8800 3234 50  0000 C CNN
-F 2 "" H 8800 3100 50  0001 C CNN
-F 3 "" H 8800 3100 50  0001 C CNN
-	1    8800 3100
-	1    0    0    -1
-$EndComp
 Wire Wire Line
 	7200 3400 7200 3150
-Wire Wire Line
-	8350 3400 7200 3400
 Connection ~ 7200 3400
-$Comp
-L power:GND #PWR060
-U 1 1 5BB711C6
-P 8050 2800
-F 0 "#PWR060" H 8050 2550 50  0001 C CNN
-F 1 "GND" H 8055 2627 50  0000 C CNN
-F 2 "" H 8050 2800 50  0001 C CNN
-F 3 "" H 8050 2800 50  0001 C CNN
-	1    8050 2800
-	1    0    0    -1
-$EndComp
-Wire Wire Line
-	8050 2800 8350 2800
-Wire Wire Line
-	8350 2800 8350 3100
-$Comp
-L Device:R_US R8
-U 1 1 5BB719C4
-P 8100 3200
-F 0 "R8" V 8150 3550 50  0000 C CNN
-F 1 "R_US" V 8050 3500 50  0000 C CNN
-F 2 "Resistor_SMD:R_0805_2012Metric_Pad1.15x1.40mm_HandSolder" V 8140 3190 50  0001 C CNN
-F 3 "~" H 8100 3200 50  0001 C CNN
-	1    8100 3200
-	0    -1   -1   0
-$EndComp
-Wire Wire Line
-	8250 3200 8350 3200
-Wire Wire Line
-	7950 3200 7950 3300
-Wire Wire Line
-	7950 3300 8350 3300
-Text Notes 8300 3650 0    50   ~ 0
-todo: check common mode
-$Comp
-L power:GND #PWR064
-U 1 1 5BB72C19
-P 9500 3600
-F 0 "#PWR064" H 9500 3350 50  0001 C CNN
-F 1 "GND" H 9505 3427 50  0000 C CNN
-F 2 "" H 9500 3600 50  0001 C CNN
-F 3 "" H 9500 3600 50  0001 C CNN
-	1    9500 3600
-	1    0    0    -1
-$EndComp
-Wire Wire Line
-	9500 3600 9500 3400
-Wire Wire Line
-	9500 3400 9250 3400
-$Comp
-L power:+3V3 #PWR059
-U 1 1 5BB735AE
-P 9500 2650
-F 0 "#PWR059" H 9500 2500 50  0001 C CNN
-F 1 "+3V3" H 9515 2823 50  0000 C CNN
-F 2 "" H 9500 2650 50  0001 C CNN
-F 3 "" H 9500 2650 50  0001 C CNN
-	1    9500 2650
-	1    0    0    -1
-$EndComp
-Wire Wire Line
-	9500 3100 9250 3100
-Wire Wire Line
-	9250 3300 9500 3300
-Wire Wire Line
-	9500 3300 9500 3400
-Connection ~ 9500 3400
 Text Label 7300 3400 0    50   ~ 0
 RTD_DIVIDER
-Text Label 9700 3200 0    50   ~ 0
+Text Label 9850 2650 0    50   ~ 0
 RTD
-Wire Wire Line
-	9700 3200 9250 3200
 $Comp
 L Connector:Conn_01x03_Female J5
@@
 F 0 "J5" H 6394 5535 50  0000 C CNN
 F 1 "Tank Pressure Conn" H 6394 5444 50  0000 C CNN
-F 2 "" H 6500 5250 50  0001 C CNN
+F 2 "Connector_JST:JST_PH_S3B-PH-K_1x03_P2.00mm_Horizontal" H 6500 5250 50  0001 C CNN
 F 3 "~" H 6500 5250 50  0001 C CNN
 	1    6500 5250
@@
 	1    0    0    -1
 $EndComp
+NoConn ~ 3050 2350
+$Comp
+L Amplifier_Operational:MCP6001U U13
+U 1 1 5BDBD0F2
+P 9100 3300
+F 0 "U13" H 9200 3050 50  0000 C CNN
+F 1 "MCP6001U" H 9350 3150 50  0000 C CNN
+F 2 "TO_SOT_Packages_SMD:SOT-23-5_HandSoldering" H 9100 3300 50  0001 L CNN
+F 3 "http://ww1.microchip.com/downloads/en/DeviceDoc/21733j.pdf" H 9100 3300 50  0001 C CNN
+	1    9100 3300
+	1    0    0    1
+$EndComp
+Wire Wire Line
+	7200 3400 8800 3400
+$Comp
+L Device:R_US R19
+U 1 1 5BDBEBD7
+P 9150 2650
+F 0 "R19" V 8945 2650 50  0000 C CNN
+F 1 "R_US" V 9036 2650 50  0000 C CNN
+F 2 "Resistor_SMD:R_0805_2012Metric_Pad1.15x1.40mm_HandSolder" V 9190 2640 50  0001 C CNN
+F 3 "~" H 9150 2650 50  0001 C CNN
+	1    9150 2650
+	0    1    1    0
+$EndComp
+Wire Wire Line
+	9000 2650 8650 2650
+Wire Wire Line
+	8650 2650 8650 3200
+Wire Wire Line
+	8650 3200 8800 3200
+$Comp
+L Device:R_US R8
+U 1 1 5BDBF96C
+P 8300 2650
+F 0 "R8" V 8095 2650 50  0000 C CNN
+F 1 "R_US" V 8186 2650 50  0000 C CNN
+F 2 "Resistor_SMD:R_0805_2012Metric_Pad1.15x1.40mm_HandSolder" V 8340 2640 50  0001 C CNN
+F 3 "~" H 8300 2650 50  0001 C CNN
+	1    8300 2650
+	0    1    1    0
+$EndComp
+Wire Wire Line
+	8450 2650 8650 2650
+Connection ~ 8650 2650
+$Comp
+L power:GND #PWR059
+U 1 1 5BDC0772
+P 8050 2700
+F 0 "#PWR059" H 8050 2450 50  0001 C CNN
+F 1 "GND" H 8055 2527 50  0000 C CNN
+F 2 "" H 8050 2700 50  0001 C CNN
+F 3 "" H 8050 2700 50  0001 C CNN
+	1    8050 2700
+	1    0    0    -1
+$EndComp
+Wire Wire Line
+	8050 2700 8050 2650
+Wire Wire Line
+	8050 2650 8150 2650
+Wire Wire Line
+	9300 2650 9600 2650
+Wire Wire Line
+	9600 2650 9600 3300
+Wire Wire Line
+	9600 3300 9400 3300
+Wire Wire Line
+	9850 2650 9600 2650
+Connection ~ 9600 2650
+$Comp
+L power:GND #PWR060
+U 1 1 5BDC3797
+P 9000 3000
+F 0 "#PWR060" H 9000 2750 50  0001 C CNN
+F 1 "GND" H 9005 2827 50  0000 C CNN
+F 2 "" H 9000 3000 50  0001 C CNN
+F 3 "" H 9000 3000 50  0001 C CNN
+	1    9000 3000
+	-1   0    0    1
+$EndComp
+$Comp
+L power:+3V3 #PWR061
+U 1 1 5BDC3836
+P 8700 3850
+F 0 "#PWR061" H 8700 3700 50  0001 C CNN
+F 1 "+3V3" H 8715 4023 50  0000 C CNN
+F 2 "" H 8700 3850 50  0001 C CNN
+F 3 "" H 8700 3850 50  0001 C CNN
+	1    8700 3850
+	1    0    0    -1
+$EndComp
 $Comp
 L Device:C C19
-U 1 1 5BB82F9C
-P 9750 2800
-F 0 "C19" V 9498 2800 50  0000 C CNN
-F 1 "0.1uF" V 9589 2800 50  0000 C CNN
-F 2 "Capacitor_SMD:C_0805_2012Metric_Pad1.15x1.40mm_HandSolder" H 9788 2650 50  0001 C CNN
-F 3 "~" H 9750 2800 50  0001 C CNN
-	1    9750 2800
+U 1 1 5BDC43DB
+P 9150 3850
+F 0 "C19" V 8898 3850 50  0000 C CNN
+F 1 "0.1uF" V 8989 3850 50  0000 C CNN
+F 2 "Capacitor_SMD:C_0805_2012Metric_Pad1.15x1.40mm_HandSolder" H 9188 3700 50  0001 C CNN
+F 3 "~" H 9150 3850 50  0001 C CNN
+	1    9150 3850
 	0    1    1    0
 $EndComp
 Wire Wire Line
-	9500 2650 9500 2800
-Wire Wire Line
-	9600 2800 9500 2800
-Connection ~ 9500 2800
-Wire Wire Line
-	9500 2800 9500 3100
-$Comp
-L power:GND #PWR061
-U 1 1 5BB87902
-P 9900 2800
-F 0 "#PWR061" H 9900 2550 50  0001 C CNN
-F 1 "GND" H 9905 2627 50  0000 C CNN
-F 2 "" H 9900 2800 50  0001 C CNN
-F 3 "" H 9900 2800 50  0001 C CNN
-	1    9900 2800
-	1    0    0    -1
-$EndComp
-NoConn ~ 3050 2350
+	9000 3600 9000 3850
+Wire Wire Line
+	8700 3850 9000 3850
+Connection ~ 9000 3850
+$Comp
+L power:GND #PWR064
+U 1 1 5BDC7789
+P 9300 3850
+F 0 "#PWR064" H 9300 3600 50  0001 C CNN
+F 1 "GND" H 9305 3677 50  0000 C CNN
+F 2 "" H 9300 3850 50  0001 C CNN
+F 3 "" H 9300 3850 50  0001 C CNN
+	1    9300 3850
+	1    0    0    -1
+$EndComp
 $EndSCHEMATC
