File: sensors/power.sch (KiCad schematic (older format))
At the start: 16 parts

Commit message: Sensor board review changes
- annotate everything
- fix symbol library mapping
- fix debug header orientation
- add extra decoupling cap to mcu
- add a couple debug leds
- add 15V regulator (tht)
- add sensor comments
Parts:
- removed F?: Polyfuse, symbol device:Polyfuse
- removed R?: ?, symbol device:R_US
- added C1: 4.7uF, symbol Device:C
- added F1: Polyfuse, symbol Device:Polyfuse
- added R1: R_US, symbol Device:R_US
- added U1: SPU01M-15, symbol flight_instr:SPU01M-15
- C2, C3, C4, C5, C6, C7, C8: renamed from C?; symbol device:C -> Device:C
- F2: renamed from F?; symbol device:Polyfuse -> Device:Polyfuse
- R2: renamed from R?; symbol device:R_US -> Device:R_US
- gave numbers to parts that had none: 5
Connections:
- net labels added: +15V
- wire segments 52 -> 57
Other:
- note added: "Can replace this one if\nwe need one that isn’t\nthrough hole."
- note removed: "todo 15v reg"

Commit message: Replace IMU cause Jacob wanted to
New IMU has better magnetometer sensitivity
Parts:
- added C15, C16: 1uF, symbol Device:C
- added U8: MIC5365-1.8, symbol canhw:MIC5365-1.8
Connections:
- net labels added: +1V8
- wire segments 57 -> 70

Commit message: Assign most footprints
Parts:
- C1, C15, C16, C2, C3, C4, C5, C6, C7, C8: footprint (none) -> Capacitor_SMD:C_0805_2012Metric_Pad1.15x1.40mm_HandSolder
- R1, R2: footprint (none) -> Resistor_SMD:R_0805_2012Metric_Pad1.15x1.40mm_HandSolder
Changed lines of the file:
@@
 F 0 "C6" V 4248 4500 50  0000 C CNN
 F 1 "0.1uF" V 4339 4500 50  0000 C CNN
-F 2 "" H 4538 4350 50  0001 C CNN
+F 2 "Capacitor_SMD:C_0805_2012Metric_Pad1.15x1.40mm_HandSolder" H 4538 4350 50  0001 C CNN
 F 3 "~" H 4500 4500 50  0001 C CNN
 	1    4500 4500
@@
 F 0 "R2" V 3245 4000 50  0000 C CNN
 F 1 "?" V 3336 4000 50  0000 C CNN
-F 2 "" V 3490 3990 50  0001 C CNN
+F 2 "Resistor_SMD:R_0805_2012Metric_Pad1.15x1.40mm_HandSolder" V 3490 3990 50  0001 C CNN
 F 3 "~" H 3450 4000 50  0001 C CNN
 	1    3450 4000
@@
 F 0 "C2" V 4248 2350 50  0000 C CNN
 F 1 "0.1uF" V 4339 2350 50  0000 C CNN
-F 2 "" H 4538 2200 50  0001 C CNN
+F 2 "Capacitor_SMD:C_0805_2012Metric_Pad1.15x1.40mm_HandSolder" H 4538 2200 50  0001 C CNN
 F 3 "~" H 4500 2350 50  0001 C CNN
 	1    4500 2350
@@
 F 0 "C8" H 9315 4446 50  0000 L CNN
 F 1 "1uF" H 9315 4355 50  0000 L CNN
-F 2 "" H 9238 4250 50  0001 C CNN
+F 2 "Capacitor_SMD:C_0805_2012Metric_Pad1.15x1.40mm_HandSolder" H 9238 4250 50  0001 C CNN
 F 3 "~" H 9200 4400 50  0001 C CNN
 	1    9200 4400
@@
 F 0 "C7" H 7615 4446 50  0000 L CNN
 F 1 "1uF" H 7615 4355 50  0000 L CNN
-F 2 "" H 7538 4250 50  0001 C CNN
+F 2 "Capacitor_SMD:C_0805_2012Metric_Pad1.15x1.40mm_HandSolder" H 7538 4250 50  0001 C CNN
 F 3 "~" H 7500 4400 50  0001 C CNN
 	1    7500 4400
@@
 F 0 "C3" H 7365 3146 50  0000 L CNN
 F 1 "1uF" H 7365 3055 50  0000 L CNN
-F 2 "" H 7288 2950 50  0001 C CNN
+F 2 "Capacitor_SMD:C_0805_2012Metric_Pad1.15x1.40mm_HandSolder" H 7288 2950 50  0001 C CNN
 F 3 "~" H 7250 3100 50  0001 C CNN
 	1    7250 3100
@@
 F 0 "C5" H 8865 3346 50  0000 L CNN
 F 1 "10nF" H 8865 3255 50  0000 L CNN
-F 2 "" H 8788 3150 50  0001 C CNN
+F 2 "Capacitor_SMD:C_0805_2012Metric_Pad1.15x1.40mm_HandSolder" H 8788 3150 50  0001 C CNN
 F 3 "~" H 8750 3300 50  0001 C CNN
 	1    8750 3300
@@
 F 0 "C4" H 9365 3146 50  0000 L CNN
 F 1 "2.2uF" H 9365 3055 50  0000 L CNN
-F 2 "" H 9288 2950 50  0001 C CNN
+F 2 "Capacitor_SMD:C_0805_2012Metric_Pad1.15x1.40mm_HandSolder" H 9288 2950 50  0001 C CNN
 F 3 "~" H 9250 3100 50  0001 C CNN
 	1    9250 3100
@@
 F 0 "R1" V 3245 1850 50  0000 C CNN
 F 1 "R_US" V 3336 1850 50  0000 C CNN
-F 2 "" V 3490 1840 50  0001 C CNN
+F 2 "Resistor_SMD:R_0805_2012Metric_Pad1.15x1.40mm_HandSolder" V 3490 1840 50  0001 C CNN
 F 3 "~" H 3450 1850 50  0001 C CNN
 	1    3450 1850
@@
 F 0 "C1" H 9365 1846 50  0000 L CNN
 F 1 "4.7uF" H 9365 1755 50  0000 L CNN
-F 2 "" H 9288 1650 50  0001 C CNN
+F 2 "Capacitor_SMD:C_0805_2012Metric_Pad1.15x1.40mm_HandSolder" H 9288 1650 50  0001 C CNN
 F 3 "~" H 9250 1800 50  0001 C CNN
 	1    9250 1800
@@
 F 0 "C16" H 9315 5546 50  0000 L CNN
 F 1 "1uF" H 9315 5455 50  0000 L CNN
-F 2 "" H 9238 5350 50  0001 C CNN
+F 2 "Capacitor_SMD:C_0805_2012Metric_Pad1.15x1.40mm_HandSolder" H 9238 5350 50  0001 C CNN
 F 3 "~" H 9200 5500 50  0001 C CNN
 	1    9200 5500
@@
 F 0 "C15" H 7615 5546 50  0000 L CNN
 F 1 "1uF" H 7615 5455 50  0000 L CNN
-F 2 "" H 7538 5350 50  0001 C CNN
+F 2 "Capacitor_SMD:C_0805_2012Metric_Pad1.15x1.40mm_HandSolder" H 7538 5350 50  0001 C CNN
 F 3 "~" H 7500 5500 50  0001 C CNN
 	1    7500 5500

Commit message: WIP sensor layout board
Parts:
- added TP1, TP2, TP3, TP4: TestPoint, TestPoint:TestPoint_THTPad_D1.0mm_Drill0.5mm, symbol Connector:TestPoint
- F1, F2: footprint (none) -> Fuse:Fuse_1206_3216Metric_Pad1.42x1.75mm_HandSolder
- J1: footprint (none) -> canhw_footprints:connector_Harwin_M80-5000642
- R1, R2: footprint Resistor_SMD:R_0805_2012Metric_Pad1.15x1.40mm_HandSolder -> Resistor_SMD:R_1206_3216Metric_Pad1.42x1.75mm_HandSolder
- U1: footprint (none) -> Flight_Instr:SIP6_Housing
- U2, U3, U4, U5, U8: footprint (none) -> TO_SOT_Packages_SMD:SOT-23-5_HandSoldering
Connections:
- wire segments 70 -> 77
Changed lines of the file:
@@
 F 0 "U4" H 4300 4528 50  0000 C CNN
 F 1 "INA180" H 4300 4437 50  0000 C CNN
-F 2 "" H 4350 5000 50  0001 C CNN
+F 2 "TO_SOT_Packages_SMD:SOT-23-5_HandSoldering" H 4350 5000 50  0001 C CNN
 F 3 "" H 4350 5000 50  0001 C CNN
 	1    4350 5000
@@
 F 0 "J1" H 1544 4485 50  0000 C CNN
 F 1 "Conn_01x05_Female" H 1544 4394 50  0000 C CNN
-F 2 "" H 1650 4100 50  0001 C CNN
+F 2 "canhw_footprints:connector_Harwin_M80-5000642" H 1650 4100 50  0001 C CNN
 F 3 "~" H 1650 4100 50  0001 C CNN
 	1    1650 4100
@@
 F 0 "F2" V 2325 4000 50  0000 C CNN
 F 1 "Polyfuse" V 2416 4000 50  0000 C CNN
-F 2 "" H 2600 3800 50  0001 L CNN
+F 2 "Fuse:Fuse_1206_3216Metric_Pad1.42x1.75mm_HandSolder" H 2600 3800 50  0001 L CNN
 F 3 "~" H 2550 4000 50  0001 C CNN
 	1    2550 4000
@@
 $EndComp
 Wire Wire Line
-	2400 4000 1850 4000
-Wire Wire Line
-	2700 4000 3200 4000
+	2400 4000 2350 4000
 Connection ~ 3200 4000
 $Comp
@@
 F 0 "R2" V 3245 4000 50  0000 C CNN
 F 1 "?" V 3336 4000 50  0000 C CNN
-F 2 "Resistor_SMD:R_0805_2012Metric_Pad1.15x1.40mm_HandSolder" V 3490 3990 50  0001 C CNN
+F 2 "Resistor_SMD:R_1206_3216Metric_Pad1.42x1.75mm_HandSolder" V 3490 3990 50  0001 C CNN
 F 3 "~" H 3450 4000 50  0001 C CNN
 	1    3450 4000
@@
 F 0 "U2" H 4300 2378 50  0000 C CNN
 F 1 "INA180" H 4300 2287 50  0000 C CNN
-F 2 "" H 4350 2850 50  0001 C CNN
+F 2 "TO_SOT_Packages_SMD:SOT-23-5_HandSoldering" H 4350 2850 50  0001 C CNN
 F 3 "" H 4350 2850 50  0001 C CNN
 	1    4350 2850
@@
 Connection ~ 3700 1850
 Wire Wire Line
-	3200 1850 2700 1850
+	3200 1850 2800 1850
 Connection ~ 3200 1850
 Wire Wire Line
@@
 F 0 "U5" H 8375 4475 50  0000 C CNN
 F 1 "MIC5504-3.3" H 8375 4384 50  0000 C CNN
-F 2 "" H 8350 4250 50  0001 C CNN
+F 2 "TO_SOT_Packages_SMD:SOT-23-5_HandSoldering" H 8350 4250 50  0001 C CNN
 F 3 "http://ww1.microchip.com/downloads/en/DeviceDoc/MIC550x-300mA-Single-Output-LDO-in-Small-Packages-DS20006006A.pdf" H 8350 4250 50  0001 C CNN
 	1    8350 4250
@@
 F 0 "U3" H 8200 3215 50  0000 C CNN
 F 1 "LP2985-10" H 8200 3124 50  0000 C CNN
-F 2 "" H 8050 2950 50  0001 C CNN
+F 2 "TO_SOT_Packages_SMD:SOT-23-5_HandSoldering" H 8050 2950 50  0001 C CNN
 F 3 "http://www.ti.com/lit/ds/symlink/lp2985.pdf" H 8050 2950 50  0001 C CNN
 	1    8050 2950
@@
 F 0 "F1" V 2325 1850 50  0000 C CNN
 F 1 "Polyfuse" V 2416 1850 50  0000 C CNN
-F 2 "" H 2600 1650 50  0001 L CNN
+F 2 "Fuse:Fuse_1206_3216Metric_Pad1.42x1.75mm_HandSolder" H 2600 1650 50  0001 L CNN
 F 3 "~" H 2550 1850 50  0001 C CNN
 	1    2550 1850
@@
 F 0 "R1" V 3245 1850 50  0000 C CNN
 F 1 "R_US" V 3336 1850 50  0000 C CNN
-F 2 "Resistor_SMD:R_0805_2012Metric_Pad1.15x1.40mm_HandSolder" V 3490 1840 50  0001 C CNN
+F 2 "Resistor_SMD:R_1206_3216Metric_Pad1.42x1.75mm_HandSolder" V 3490 1840 50  0001 C CNN
 F 3 "~" H 3450 1850 50  0001 C CNN
 	1    3450 1850
@@
 F 0 "U1" H 8175 1937 60  0000 C CNN
 F 1 "SPU01M-15" H 8175 1831 60  0000 C CNN
-F 2 "" H 8100 1650 60  0001 C CNN
+F 2 "Flight_Instr:SIP6_Housing" H 8100 1650 60  0001 C CNN
 F 3 "" H 8100 1650 60  0001 C CNN
 	1    8100 1650
@@
 F 0 "U8" H 8375 5575 50  0000 C CNN
 F 1 "MIC5365-1.8" H 8375 5484 50  0000 C CNN
-F 2 "" H 8450 5350 50  0001 C CNN
+F 2 "TO_SOT_Packages_SMD:SOT-23-5_HandSoldering" H 8450 5350 50  0001 C CNN
 F 3 "" H 8450 5350 50  0001 C CNN
 	1    8400 5350
@@
 	1    0    0    -1
 $EndComp
+$Comp
+L Connector:TestPoint TP1
+U 1 1 5BDC9287
+P 2250 1400
+F 0 "TP1" H 2308 1520 50  0000 L CNN
+F 1 "TestPoint" H 2308 1429 50  0000 L CNN
+F 2 "TestPoint:TestPoint_THTPad_D1.0mm_Drill0.5mm" H 2450 1400 50  0001 C CNN
+F 3 "~" H 2450 1400 50  0001 C CNN
+	1    2250 1400
+	1    0    0    -1
+$EndComp
+Wire Wire Line
+	2250 1400 2250 1850
+Connection ~ 2250 1850
+$Comp
+L Connector:TestPoint TP2
+U 1 1 5BDCA55D
+P 2800 1400
+F 0 "TP2" H 2858 1520 50  0000 L CNN
+F 1 "TestPoint" H 2858 1429 50  0000 L CNN
+F 2 "TestPoint:TestPoint_THTPad_D1.0mm_Drill0.5mm" H 3000 1400 50  0001 C CNN
+F 3 "~" H 3000 1400 50  0001 C CNN
+	1    2800 1400
+	1    0    0    -1
+$EndComp
+Wire Wire Line
+	2800 1400 2800 1850
+Connection ~ 2800 1850
+Wire Wire Line
+	2800 1850 2700 1850
+$Comp
+L Connector:TestPoint TP4
+U 1 1 5BDCB8C1
+P 2900 3650
+F 0 "TP4" H 2958 3770 50  0000 L CNN
+F 1 "TestPoint" H 2958 3679 50  0000 L CNN
+F 2 "TestPoint:TestPoint_THTPad_D1.0mm_Drill0.5mm" H 3100 3650 50  0001 C CNN
+F 3 "~" H 3100 3650 50  0001 C CNN
+	1    2900 3650
+	1    0    0    -1
+$EndComp
+Wire Wire Line
+	2900 3650 2900 4000
+Wire Wire Line
+	2700 4000 2900 4000
+Connection ~ 2900 4000
+Wire Wire Line
+	2900 4000 3200 4000
+$Comp
+L Connector:TestPoint TP3
+U 1 1 5BDCD140
+P 2350 3650
+F 0 "TP3" H 2408 3770 50  0000 L CNN
+F 1 "TestPoint" H 2408 3679 50  0000 L CNN
+F 2 "TestPoint:TestPoint_THTPad_D1.0mm_Drill0.5mm" H 2550 3650 50  0001 C CNN
+F 3 "~" H 2550 3650 50  0001 C CNN
+	1    2350 3650
+	1    0    0    -1
+$EndComp
+Wire Wire Line
+	2350 3650 2350 4000
+Connection ~ 2350 4000
+Wire Wire Line
+	2350 4000 1850 4000
 $EndSCHEMATC
