File: usbdbg/usbdbg/usbdbg.sch (KiCad schematic (older format))
At the start: 20 parts, among them J1 USB_B, J2 Programming Header, J3 Conn_01x04_Female, U1 MCP2562, U2 PIC16F1455, U3 MCP2515

Commit message: Update part footprints for usbdbg, dump footprints onto pcb
Parts:
- C1, C2, C3, C4: footprint (none) -> Capacitor_SMD:C_0805_2012Metric_Pad1.15x1.40mm_HandSolder
- D1, D2: footprint (none) -> LED_SMD:LED_1206_3216Metric_Pad1.42x1.75mm_HandSolder
- J1: footprint Connector_USB:USB_B_Horizontal -> Connector_USB:USB_B_OST_USB-B1HSxx_Horizontal
- J2: footprint Pin_Headers:Pin_Header_Straight_1x05_Pitch2.54mm -> Connector_PinHeader_2.54mm:PinHeader_1x05_P2.54mm_Vertical
- J3: footprint (none) -> Connector_PinHeader_2.54mm:PinHeader_1x04_P2.54mm_Vertical
- R1, R2, R3, R4, R5, R6: footprint (none) -> Resistor_SMD:R_0805_2012Metric_Pad1.15x1.40mm_HandSolder
- U1: footprint Housings_DIP:DIP-8_W7.62mm -> Package_DIP:DIP-8_W7.62mm_LongPads
- U2: footprint Housings_DIP:DIP-14_W7.62mm -> Package_DIP:DIP-14_W7.62mm_LongPads
- U3: footprint Housings_DIP:DIP-18_W7.62mm -> Package_DIP:DIP-18_W7.62mm_LongPads
Changed lines of the file:
@@
 EESchema Schematic File Version 4
+LIBS:usbdbg-cache
 EELAYER 26 0
 EELAYER END
@@
 F 0 "U2" H 3525 4865 50  0000 C CNN
 F 1 "PIC16F1455" H 3525 4774 50  0000 C CNN
-F 2 "Housings_DIP:DIP-14_W7.62mm" H 3300 4550 50  0001 C CNN
+F 2 "Package_DIP:DIP-14_W7.62mm_LongPads" H 3300 4550 50  0001 C CNN
 F 3 "" H 3300 4550 50  0001 C CNN
 	1    3300 4550
@@
 F 0 "J2" H 3400 2000 50  0000 C CNN
 F 1 "Programming Header" H 3050 2100 50  0000 C CNN
-F 2 "Pin_Headers:Pin_Header_Straight_1x05_Pitch2.54mm" H 3050 2450 50  0001 C CNN
+F 2 "Connector_PinHeader_2.54mm:PinHeader_1x05_P2.54mm_Vertical" H 3050 2450 50  0001 C CNN
 F 3 "~" H 3050 2450 50  0001 C CNN
 	1    3050 2450
@@
 F 0 "U1" H 8925 4515 50  0000 C CNN
 F 1 "MCP2562" H 8925 4424 50  0000 C CNN
-F 2 "Housings_DIP:DIP-8_W7.62mm" H 8950 4250 50  0001 C CNN
+F 2 "Package_DIP:DIP-8_W7.62mm_LongPads" H 8950 4250 50  0001 C CNN
 F 3 "" H 8950 4250 50  0001 C CNN
 	1    8950 4250
@@
 F 0 "U3" H 7050 5115 50  0000 C CNN
 F 1 "MCP2515" H 7050 5024 50  0000 C CNN
-F 2 "Housings_DIP:DIP-18_W7.62mm" H 7000 4650 50  0001 C CNN
+F 2 "Package_DIP:DIP-18_W7.62mm_LongPads" H 7000 4650 50  0001 C CNN
 F 3 "" H 7000 4650 50  0001 C CNN
 	1    7050 4650
@@
 F 0 "J1" H 6205 2767 50  0000 C CNN
 F 1 "USB_B" H 6205 2676 50  0000 C CNN
-F 2 "Connector_USB:USB_B_Horizontal" H 6300 2250 50  0001 C CNN
+F 2 "Connector_USB:USB_B_OST_USB-B1HSxx_Horizontal" H 6300 2250 50  0001 C CNN
 F 3 " ~" H 6300 2250 50  0001 C CNN
 	1    6150 2300
@@
 F 0 "R3" H 1381 4204 50  0000 R CNN
 F 1 "330" H 1381 4295 50  0000 R CNN
-F 2 "" V 1380 4250 50  0001 C CNN
+F 2 "Resistor_SMD:R_0805_2012Metric_Pad1.15x1.40mm_HandSolder" V 1380 4250 50  0001 C CNN
 F 3 "~" H 1450 4250 50  0001 C CNN
 	1    1450 4250
@@
 F 0 "R4" H 1920 4296 50  0000 L CNN
 F 1 "330" H 1920 4205 50  0000 L CNN
-F 2 "" V 1780 4250 50  0001 C CNN
+F 2 "Resistor_SMD:R_0805_2012Metric_Pad1.15x1.40mm_HandSolder" V 1780 4250 50  0001 C CNN
 F 3 "~" H 1850 4250 50  0001 C CNN
 	1    1850 4250
@@
 F 0 "D1" V 1488 4628 50  0000 L CNN
 F 1 "LED" V 1397 4628 50  0000 L CNN
-F 2 "" H 1450 4550 50  0001 C CNN
+F 2 "LED_SMD:LED_1206_3216Metric_Pad1.42x1.75mm_HandSolder" H 1450 4550 50  0001 C CNN
 F 3 "~" H 1450 4550 50  0001 C CNN
 	1    1450 4550
@@
 F 0 "D2" V 1888 4433 50  0000 R CNN
 F 1 "LED" V 1797 4433 50  0000 R CNN
-F 2 "" H 1850 4550 50  0001 C CNN
+F 2 "LED_SMD:LED_1206_3216Metric_Pad1.42x1.75mm_HandSolder" H 1850 4550 50  0001 C CNN
 F 3 "~" H 1850 4550 50  0001 C CNN
 	1    1850 4550
@@
 F 0 "R1" V 6393 2100 50  0000 C CNN
 F 1 "0" V 6484 2100 50  0000 C CNN
-F 2 "" V 6530 2100 50  0001 C CNN
+F 2 "Resistor_SMD:R_0805_2012Metric_Pad1.15x1.40mm_HandSolder" V 6530 2100 50  0001 C CNN
 F 3 "~" H 6600 2100 50  0001 C CNN
 	1    6600 2100
@@
 F 0 "C3" H 2765 5446 50  0000 L CNN
 F 1 "0.1u" H 2765 5355 50  0000 L CNN
-F 2 "" H 2688 5250 50  0001 C CNN
+F 2 "Capacitor_SMD:C_0805_2012Metric_Pad1.15x1.40mm_HandSolder" H 2688 5250 50  0001 C CNN
 F 3 "~" H 2650 5400 50  0001 C CNN
 	1    2650 5400
@@
 F 0 "C2" H 4715 5196 50  0000 L CNN
 F 1 "0.1u" H 4715 5105 50  0000 L CNN
-F 2 "" H 4638 5000 50  0001 C CNN
+F 2 "Capacitor_SMD:C_0805_2012Metric_Pad1.15x1.40mm_HandSolder" H 4638 5000 50  0001 C CNN
 F 3 "~" H 4600 5150 50  0001 C CNN
 	1    4600 5150
@@
 F 0 "C4" H 6465 5496 50  0000 L CNN
 F 1 "0.1u" H 6465 5405 50  0000 L CNN
-F 2 "" H 6388 5300 50  0001 C CNN
+F 2 "Capacitor_SMD:C_0805_2012Metric_Pad1.15x1.40mm_HandSolder" H 6388 5300 50  0001 C CNN
 F 3 "~" H 6350 5450 50  0001 C CNN
 	1    6350 5450
@@
 F 0 "C1" H 8415 4846 50  0000 L CNN
 F 1 "10u" H 8415 4755 50  0000 L CNN
-F 2 "" H 8338 4650 50  0001 C CNN
+F 2 "Capacitor_SMD:C_0805_2012Metric_Pad1.15x1.40mm_HandSolder" H 8338 4650 50  0001 C CNN
 F 3 "~" H 8300 4800 50  0001 C CNN
 	1    8300 4800
@@
 F 0 "R5" H 6170 4446 50  0000 L CNN
 F 1 "10k" H 6170 4355 50  0000 L CNN
-F 2 "" V 6030 4400 50  0001 C CNN
+F 2 "Resistor_SMD:R_0805_2012Metric_Pad1.15x1.40mm_HandSolder" V 6030 4400 50  0001 C CNN
 F 3 "~" H 6100 4400 50  0001 C CNN
 	1    6100 4400
@@
 F 0 "R2" H 4420 3996 50  0000 L CNN
 F 1 "10k" H 4420 3905 50  0000 L CNN
-F 2 "" V 4280 3950 50  0001 C CNN
+F 2 "Resistor_SMD:R_0805_2012Metric_Pad1.15x1.40mm_HandSolder" V 4280 3950 50  0001 C CNN
 F 3 "~" H 4350 3950 50  0001 C CNN
 	1    4350 3950
@@
 F 0 "J3" H 10377 4326 50  0000 L CNN
 F 1 "Conn_01x04_Female" H 10377 4235 50  0000 L CNN
-F 2 "" H 10350 4350 50  0001 C CNN
+F 2 "Connector_PinHeader_2.54mm:PinHeader_1x04_P2.54mm_Vertical" H 10350 4350 50  0001 C CNN
 F 3 "~" H 10350 4350 50  0001 C CNN
 	1    10350 4350
@@
 F 0 "R6" H 10070 4846 50  0000 L CNN
 F 1 "0" H 10070 4755 50  0000 L CNN
-F 2 "" V 9930 4800 50  0001 C CNN
+F 2 "Resistor_SMD:R_0805_2012Metric_Pad1.15x1.40mm_HandSolder" V 9930 4800 50  0001 C CNN
 F 3 "~" H 10000 4800 50  0001 C CNN
 	1    10000 4800

Commit message: Minor review fix on USB dog
Remove the bus power connector on the CAN header, it now only contains
ground, CANH and CANL. Also minor silkscreen edits to show which pins
are CANH, CANL, GND, and ~MCLR.
Parts:
- removed J3: Conn_01x04_Female, Connector_PinHeader_2.54mm:PinHeader_1x04_P2.54mm_Vertical, symbol Connector:Conn_01x04_Female
- added J3: CAN_Header, Connector_PinHeader_2.54mm:PinHeader_1x03_P2.54mm_Vertical, symbol Connector:Conn_01x03_Female
Connections:
- no-connect marks 8 -> 7
Changed lines of the file:
@@
-$EndComp
-$Comp
-L Connector:Conn_01x04_Female J3
-U 1 1 5B9F582C
-P 10350 4350
-F 0 "J3" H 10377 4326 50  0000 L CNN
-F 1 "Conn_01x04_Female" H 10377 4235 50  0000 L CNN
-F 2 "Connector_PinHeader_2.54mm:PinHeader_1x04_P2.54mm_Vertical" H 10350 4350 50  0001 C CNN
-F 3 "~" H 10350 4350 50  0001 C CNN
-	1    10350 4350
-	1    0    0    -1
 $EndComp
 $Comp
@@
 Wire Wire Line
 	9400 4350 10150 4350
-NoConn ~ 10150 4250
 $Comp
 L Device:R R6
@@
 Wire Wire Line
 	10000 5000 10000 4950
+$Comp
+L Connector:Conn_01x03_Female J3
+U 1 1 5BA195A3
+P 10350 4450
+F 0 "J3" H 10243 4125 50  0000 C CNN
+F 1 "CAN_Header" H 10243 4216 50  0000 C CNN
+F 2 "Connector_PinHeader_2.54mm:PinHeader_1x03_P2.54mm_Vertical" H 10350 4450 50  0001 C CNN
+F 3 "~" H 10350 4450 50  0001 C CNN
+	1    10350 4450
+	1    0    0    1
+$EndComp
 $EndSCHEMATC

Commit message: USB Debug update - ready for review for production version (not usbdog)
Remove the 0ohm resistors from USB power to 5V rail and from CAN
ground to ground plane. These were unneccessary, a wire does just
fine.

Replace the CAN bus connector with a more standard 5 pin one. The usb
board should use the same connector as every other board, now it
can. There's a new jumper that allows you to power the CAN bus from
the USB board's 5V rail, in case you're doing an integration test or
something and you want to do that.
Parts:
- removed J3: CAN_Header, Connector_PinHeader_2.54mm:PinHeader_1x03_P2.54mm_Vertical, symbol Connector:Conn_01x03_Female
- removed R1, R6: 0, Resistor_SMD:R_0805_2012Metric_Pad1.15x1.40mm_HandSolder, symbol Device:R
- added J?: BUS CONN, symbol Connector:Conn_01x05_Female
- added JP?: Jumper_NC_Dual, symbol Device:Jumper_NC_Dual
Connections:
- wire segments 76 -> 80
- no-connect marks 7 -> 9
Other:
- note added: "12V (NC, this board\ndoesn't need it)"
- note added: "In some situations (namely, integration testing), we want the\nbus to be powered without having the radio board connected.\nBy moving a jumper on these pins, you can power the bus from\nthe USB port of your computer."
Changed lines of the file:
@@
-$EndComp
-$Comp
-L Device:R R1
-U 1 1 5B9F4C9F
-P 6600 2100
-F 0 "R1" V 6393 2100 50  0000 C CNN
-F 1 "0" V 6484 2100 50  0000 C CNN
-F 2 "Resistor_SMD:R_0805_2012Metric_Pad1.15x1.40mm_HandSolder" V 6530 2100 50  0001 C CNN
-F 3 "~" H 6600 2100 50  0001 C CNN
-	1    6600 2100
-	0    1    1    0
 $EndComp
 $Comp
@@
 $EndComp
 Wire Wire Line
-	10000 4650 10000 4550
-Wire Wire Line
-	10000 4550 10150 4550
-Wire Wire Line
 	9400 4450 10150 4450
 Wire Wire Line
 	9400 4350 10150 4350
 $Comp
-L Device:R R6
-U 1 1 5B9FDAB7
-P 10000 4800
-F 0 "R6" H 10070 4846 50  0000 L CNN
-F 1 "0" H 10070 4755 50  0000 L CNN
-F 2 "Resistor_SMD:R_0805_2012Metric_Pad1.15x1.40mm_HandSolder" V 9930 4800 50  0001 C CNN
-F 3 "~" H 10000 4800 50  0001 C CNN
-	1    10000 4800
+L Connector:Conn_01x05_Female J?
+U 1 1 5BAB19E0
+P 10350 4250
+F 0 "J?" H 10378 4276 50  0000 L CNN
+F 1 "BUS CONN" H 10378 4185 50  0000 L CNN
+F 2 "" H 10350 4250 50  0001 C CNN
+F 3 "~" H 10350 4250 50  0001 C CNN
+	1    10350 4250
 	1    0    0    -1
 $EndComp
 Wire Wire Line
-	10000 5000 10000 4950
+	10000 4250 10150 4250
+Wire Wire Line
+	10000 4250 10000 5000
+Text Notes 10400 4100 0    50   ~ 0
+12V (NC, this board\ndoesn't need it)
 $Comp
-L Connector:Conn_01x03_Female J3
-U 1 1 5BA195A3
-P 10350 4450
-F 0 "J3" H 10243 4125 50  0000 C CNN
-F 1 "CAN_Header" H 10243 4216 50  0000 C CNN
-F 2 "Connector_PinHeader_2.54mm:PinHeader_1x03_P2.54mm_Vertical" H 10350 4450 50  0001 C CNN
-F 3 "~" H 10350 4450 50  0001 C CNN
-	1    10350 4450
-	1    0    0    1
+L Device:Jumper_NC_Dual JP?
+U 1 1 5BAB505C
+P 10000 3450
+F 0 "JP?" H 10000 3689 50  0000 C CNN
+F 1 "Jumper_NC_Dual" H 10000 3598 50  0000 C CNN
+F 2 "" H 10000 3450 50  0001 C CNN
+F 3 "~" H 10000 3450 50  0001 C CNN
+	1    10000 3450
+	1    0    0    -1
 $EndComp
+NoConn ~ 10250 3450
+$Comp
+L power:+5V #PWR?
+U 1 1 5BAB81E8
+P 9500 3200
+F 0 "#PWR?" H 9500 3050 50  0001 C CNN
+F 1 "+5V" H 9515 3373 50  0000 C CNN
+F 2 "" H 9500 3200 50  0001 C CNN
+F 3 "" H 9500 3200 50  0001 C CNN
+	1    9500 3200
+	1    0    0    -1
+$EndComp
+Wire Wire Line
+	9750 3450 9500 3450
+Wire Wire Line
+	9500 3450 9500 3200
+Wire Wire Line
+	10150 4150 10000 4150
+Wire Wire Line
+	10000 4150 10000 3550
+NoConn ~ 10150 4050
+Text Notes 8700 2950 0    50   ~ 0
+In some situations (namely, integration testing), we want the\nbus to be powered without having the radio board connected.\nBy moving a jumper on these pins, you can power the bus from\nthe USB port of your computer.
+Wire Wire Line
+	6450 2100 6750 2100
 $EndSCHEMATC

Commit message: USB Debug - annotate schematic
I screwed up. I'd rather fess up to that than force push and have
github bot announce my shame to all the frosh
Parts:
- gave numbers to parts that had none: 2
Changed lines of the file:
@@
 	9400 4350 10150 4350
 $Comp
-L Connector:Conn_01x05_Female J?
+L Connector:Conn_01x05_Female J3
 U 1 1 5BAB19E0
 P 10350 4250
-F 0 "J?" H 10378 4276 50  0000 L CNN
+F 0 "J3" H 10378 4276 50  0000 L CNN
 F 1 "BUS CONN" H 10378 4185 50  0000 L CNN
 F 2 "" H 10350 4250 50  0001 C CNN
@@
 12V (NC, this board\ndoesn't need it)
 $Comp
-L Device:Jumper_NC_Dual JP?
+L Device:Jumper_NC_Dual JP1
 U 1 1 5BAB505C
 P 10000 3450
-F 0 "JP?" H 10000 3689 50  0000 C CNN
+F 0 "JP1" H 10000 3689 50  0000 C CNN
 F 1 "Jumper_NC_Dual" H 10000 3598 50  0000 C CNN
 F 2 "" H 10000 3450 50  0001 C CNN
@@
 NoConn ~ 10250 3450
 $Comp
-L power:+5V #PWR?
+L power:+5V #PWR019
 U 1 1 5BAB81E8
 P 9500 3200
-F 0 "#PWR?" H 9500 3050 50  0001 C CNN
+F 0 "#PWR019" H 9500 3050 50  0001 C CNN
 F 1 "+5V" H 9515 3373 50  0000 C CNN
 F 2 "" H 9500 3200 50  0001 C CNN

Commit message: USB Flea Preview 1
Parts:
- J3: footprint (none) -> canhw_footprints:connector_Harwin_M80-5000642
- JP1: footprint (none) -> Connector_PinHeader_2.54mm:PinHeader_1x03_P2.54mm_Vertical
- U1: footprint Package_DIP:DIP-8_W7.62mm_LongPads -> Package_SO:SOIC-8_3.9x4.9mm_P1.27mm
- U2: footprint Package_DIP:DIP-14_W7.62mm_LongPads -> Package_SO:SOIC-14_3.9x8.7mm_P1.27mm
- U3: footprint Package_DIP:DIP-18_W7.62mm_LongPads -> Package_SO:SOIC-18W_7.5x11.6mm_P1.27mm
Changed lines of the file:
@@
 F 0 "U2" H 3525 4865 50  0000 C CNN
 F 1 "PIC16F1455" H 3525 4774 50  0000 C CNN
-F 2 "Package_DIP:DIP-14_W7.62mm_LongPads" H 3300 4550 50  0001 C CNN
+F 2 "Package_SO:SOIC-14_3.9x8.7mm_P1.27mm" H 3300 4550 50  0001 C CNN
 F 3 "" H 3300 4550 50  0001 C CNN
 	1    3300 4550
@@
 F 3 "~" H 3050 2450 50  0001 C CNN
 	1    3050 2450
-	-1   0    0    1
+	-1   0    0    -1
 $EndComp
 Text Label 3700 2250 0    50   ~ 0
@@
 F 0 "U1" H 8925 4515 50  0000 C CNN
 F 1 "MCP2562" H 8925 4424 50  0000 C CNN
-F 2 "Package_DIP:DIP-8_W7.62mm_LongPads" H 8950 4250 50  0001 C CNN
+F 2 "Package_SO:SOIC-8_3.9x4.9mm_P1.27mm" H 8950 4250 50  0001 C CNN
 F 3 "" H 8950 4250 50  0001 C CNN
 	1    8950 4250
@@
 F 0 "U3" H 7050 5115 50  0000 C CNN
 F 1 "MCP2515" H 7050 5024 50  0000 C CNN
-F 2 "Package_DIP:DIP-18_W7.62mm_LongPads" H 7000 4650 50  0001 C CNN
+F 2 "Package_SO:SOIC-18W_7.5x11.6mm_P1.27mm" H 7000 4650 50  0001 C CNN
 F 3 "" H 7000 4650 50  0001 C CNN
 	1    7050 4650
@@
 F 0 "J3" H 10378 4276 50  0000 L CNN
 F 1 "BUS CONN" H 10378 4185 50  0000 L CNN
-F 2 "" H 10350 4250 50  0001 C CNN
+F 2 "canhw_footprints:connector_Harwin_M80-5000642" H 10350 4250 50  0001 C CNN
 F 3 "~" H 10350 4250 50  0001 C CNN
 	1    10350 4250
@@
 F 0 "JP1" H 10000 3689 50  0000 C CNN
 F 1 "Jumper_NC_Dual" H 10000 3598 50  0000 C CNN
-F 2 "" H 10000 3450 50  0001 C CNN
+F 2 "Connector_PinHeader_2.54mm:PinHeader_1x03_P2.54mm_Vertical" H 10000 3450 50  0001 C CNN
 F 3 "~" H 10000 3450 50  0001 C CNN
 	1    10000 3450

Commit message: commited changes to rebase
Connections:
- net labels added: +3.3V
Changed lines of the file:
@@
 Text Label 2500 4600 2    50   ~ 0
 CLKOUT
-$Comp
-L power:+5V #PWR09
-U 1 1 5B97E564
-P 2650 4250
-F 0 "#PWR09" H 2650 4100 50  0001 C CNN
-F 1 "+5V" H 2665 4423 50  0000 C CNN
-F 2 "" H 2650 4250 50  0001 C CNN
-F 3 "" H 2650 4250 50  0001 C CNN
-	1    2650 4250
-	1    0    0    -1
-$EndComp
 Wire Wire Line
 	2650 4250 2650 4500
@@
 	4350 4500 4650 4500
 $Comp
-L power:+5V #PWR05
-U 1 1 5B9A5A0C
-P 4350 3800
-F 0 "#PWR05" H 4350 3650 50  0001 C CNN
-F 1 "+5V" H 4365 3973 50  0000 C CNN
-F 2 "" H 4350 3800 50  0001 C CNN
-F 3 "" H 4350 3800 50  0001 C CNN
-	1    4350 3800
-	1    0    0    -1
-$EndComp
-$Comp
 L Connector:TestPoint TP1
 U 1 1 5B9A876F
@@
 Wire Wire Line
 	6450 2100 6750 2100
+$Comp
+L power:+3.3V #PWR?
+U 1 1 5BFB7BBC
+P 4350 3800
+F 0 "#PWR?" H 4350 3650 50  0001 C CNN
+F 1 "+3.3V" H 4365 3973 50  0000 C CNN
+F 2 "" H 4350 3800 50  0001 C CNN
+F 3 "" H 4350 3800 50  0001 C CNN
+	1    4350 3800
+	1    0    0    -1
+$EndComp
+$Comp
+L power:+3.3V #PWR?
+U 1 1 5BFB7C7E
+P 2650 4250
+F 0 "#PWR?" H 2650 4100 50  0001 C CNN
+F 1 "+3.3V" H 2665 4423 50  0000 C CNN
+F 2 "" H 2650 4250 50  0001 C CNN
+F 3 "" H 2650 4250 50  0001 C CNN
+	1    2650 4250
+	1    0    0    -1
+$EndComp
 $EndSCHEMATC
