File: gps/mcu.sch (KiCad schematic (older format))
At the start: 18 parts

Commit message: Addressed Alex's comments
Parts:
- removed C? (x2): 1µf, symbol Device:C
- removed U?: MIC5504-3.3, symbol canhw:MIC5504-3.3
- added C10, C11, C12, C13, C8, C9: 10nF, Capacitor_SMD:C_0805_2012Metric_Pad1.15x1.40mm_HandSolder, symbol Device:C
- added U5, U6, U7: SN74LVC2T45, symbol flight_instr:SN74LVC2T45
- C4: renamed from C?; value 0.1µ -> 0.1µF
- gave numbers to parts that had none: 13
Connections:
- wire segments 62 -> 87
- no-connect marks 2 -> 1
Other:
- moved on the sheet: C4, D1, D2, D3, R2, R3, R4, R5

Commit message: Addressed Alex's comments: Fixed Level shifters, specified directions of the signals correctly. Added Pull-up resistors for the level shifters Switched from SPI to UART, fixed nessesary connections Grounded GPS board Fixed misc. errors mentioned
Parts:
- removed C10, C11: 10nF, Capacitor_SMD:C_0805_2012Metric_Pad1.15x1.40mm_HandSolder, symbol Device:C
- removed U6: SN74LVC2T45, symbol flight_instr:SN74LVC2T45
- added R? (x3): 10K, symbol Device:R
Connections:
- net labels added: RX, RX1, TX, TX1
- net labels removed: SCK, SDI, SDO, SS, WAKE_UP
- wire segments 87 -> 85
- no-connect marks 1 -> 3

Commit message: Addressed Alex's issues: Replaced 5V to 3v3 level shifter with 2 voltage dividers Fixed Hierarchical labels for the gps Renamed and clarified some connections
Parts:
- removed C8, C9: 10nF, Capacitor_SMD:C_0805_2012Metric_Pad1.15x1.40mm_HandSolder, symbol Device:C
- removed R? (x2): 10K, symbol Device:R
- removed U5: SN74LVC2T45, symbol flight_instr:SN74LVC2T45
- added R? (x2): 1K, symbol Device:R
- added R?: 2K, symbol Device:R
- added R?: 2, symbol Device:R
- renumbered C4 to C?, C5 to C?, C6 to C?, C7 to C?, C12 to C?, C13 to C?, D1 to D?, D2 to D?, D3 to D?, R2 to R?, R4 to R?, R3 to R?, R5 to R?, U3 to U?, U4 to U?, U7 to U?, Y1 to Y?
Connections:
- net labels added: PIC_RESET_3V3, PIC_RX_3V3, PIC_TX_3V3, RESET_5V, RX_5V, TX_5V
- net labels removed: RESET, RX, RX1, TX, TX1
- wire segments 85 -> 73
Other:
- moved on the sheet: C?, R?

Commit message: Addressed changes: Re-added the 2.2 resistors in series with the 0ohm resistor Accidentally wired the gps-board into self start mode when changing from SPI to UART. Reverted this change. Connected PIC_RX to GPS_TX and PIC_TX with GPS_RX changed resistor value of the voltage dividers from 1k to 10k and 2k to 20k Added anotation to each components
Parts:
- added R11, R7: 10K, symbol Device:R
- added R12, R8: 20K, symbol Device:R
- R10: renamed from R?; value 2 -> 20K
- R13, R9: renamed from R?; value 1K -> 10K
- R14: renamed from R?; value 2K -> 20K
- gave numbers to parts that had none: 19
Connections:
- net labels added: PIC_ON_OFF_3V3, PIC_WAKEUP_3V3, WAKEUP
- wire segments 73 -> 77
Other:
- note removed: "3.3V"
Changed lines of the file:
@@
 $EndDescr
 $Comp
-L canhw:PIC18F26K83 U?
+L canhw:PIC18F26K83 U2
 U 1 1 5BE4A274
 P 2040 3730
-F 0 "U?" H 2015 4645 50  0000 C CNN
+F 0 "U2" H 2015 4645 50  0000 C CNN
 F 1 "PIC18F26K83" H 2015 4554 50  0000 C CNN
 F 2 "" H 2490 3730 50  0001 C CNN
@@
 $EndComp
 $Comp
-L Device:R R?
+L Device:R R2
 U 1 1 5BE4A9BC
 P 1190 2780
-F 0 "R?" H 1260 2826 50  0000 L CNN
+F 0 "R2" H 1260 2826 50  0000 L CNN
 F 1 "10k" H 1260 2735 50  0000 L CNN
 F 2 "Resistor_SMD:R_0805_2012Metric_Pad1.15x1.40mm_HandSolder" V 1120 2780 50  0001 C CNN
@@
 	3390 4280 3390 4380
 $Comp
-L Device:C C?
+L Device:C C4
 U 1 1 5BE4EF57
 P 3090 2980
-F 0 "C?" V 2838 2980 50  0000 C CNN
+F 0 "C4" V 2838 2980 50  0000 C CNN
 F 1 "0.1µF" V 2929 2980 50  0000 C CNN
 F 2 "Capacitor_SMD:C_0805_2012Metric_Pad1.15x1.40mm_HandSolder" H 3128 2830 50  0001 C CNN
@@
 ICSPCLK
 $Comp
-L Device:LED D?
+L Device:LED D1
 U 1 1 5BE50B84
 P 3490 3930
-F 0 "D?" V 3540 4080 50  0000 C CNN
+F 0 "D1" V 3540 4080 50  0000 C CNN
 F 1 "LED" V 3440 4080 50  0000 C CNN
 F 2 "LED_SMD:LED_1206_3216Metric_Pad1.42x1.75mm_HandSolder" H 3490 3930 50  0001 C CNN
@@
 $EndComp
 $Comp
-L Device:R R?
+L Device:R R4
 U 1 1 5BE51A36
 P 3790 4230
-F 0 "R?" H 3860 4276 50  0000 L CNN
+F 0 "R4" H 3860 4276 50  0000 L CNN
 F 1 "330" H 3860 4185 50  0000 L CNN
 F 2 "Resistor_SMD:R_0805_2012Metric_Pad1.15x1.40mm_HandSolder" V 3720 4230 50  0001 C CNN
@@
 $EndComp
 $Comp
-L Device:R R?
+L Device:R R3
 U 1 1 5BE51B21
 P 3490 4230
-F 0 "R?" H 3560 4276 50  0000 L CNN
+F 0 "R3" H 3560 4276 50  0000 L CNN
 F 1 "330" H 3560 4185 50  0000 L CNN
 F 2 "Resistor_SMD:R_0805_2012Metric_Pad1.15x1.40mm_HandSolder" V 3420 4230 50  0001 C CNN
@@
 $EndComp
 $Comp
-L Device:R R?
+L Device:R R5
 U 1 1 5BE51C0F
 P 4090 4230
-F 0 "R?" H 4160 4276 50  0000 L CNN
+F 0 "R5" H 4160 4276 50  0000 L CNN
 F 1 "330" H 4160 4185 50  0000 L CNN
 F 2 "Resistor_SMD:R_0805_2012Metric_Pad1.15x1.40mm_HandSolder" V 4020 4230 50  0001 C CNN
@@
 $EndComp
 $Comp
-L Device:LED D?
+L Device:LED D2
 U 1 1 5BE52C35
 P 3790 3930
-F 0 "D?" V 3840 4080 50  0000 C CNN
+F 0 "D2" V 3840 4080 50  0000 C CNN
 F 1 "LED" V 3740 4080 50  0000 C CNN
 F 2 "LED_SMD:LED_1206_3216Metric_Pad1.42x1.75mm_HandSolder" H 3790 3930 50  0001 C CNN
@@
 	3790 4380 3490 4380
 $Comp
-L Device:LED D?
+L Device:LED D3
 U 1 1 5BE52D20
 P 4090 3930
-F 0 "D?" V 4140 4080 50  0000 C CNN
+F 0 "D3" V 4140 4080 50  0000 C CNN
 F 1 "LED" V 4040 4080 50  0000 C CNN
 F 2 "LED_SMD:LED_1206_3216Metric_Pad1.42x1.75mm_HandSolder" H 4090 3930 50  0001 C CNN
@@
 debug LEDs
 $Comp
-L Connector:Conn_01x05_Female J?
+L Connector:Conn_01x05_Female J2
 U 1 1 5BF9C3B4
 P 2850 1700
-F 0 "J?" H 2744 1275 50  0000 C CNN
+F 0 "J2" H 2744 1275 50  0000 C CNN
 F 1 "Programming Header" H 2744 1366 50  0000 C CNN
 F 2 "" H 2850 1700 50  0001 C CNN
@@
 	2740 4380 3390 4380
 $Comp
-L canhw:MCP2562 U?
+L canhw:MCP2562 U3
 U 1 1 5C009313
 P 2870 5860
-F 0 "U?" H 2845 6125 50  0000 C CNN
+F 0 "U3" H 2845 6125 50  0000 C CNN
 F 1 "MCP2562" H 2845 6034 50  0000 C CNN
 F 2 "" H 2870 5860 50  0001 C CNN
@@
 $EndComp
 $Comp
-L Device:C C?
+L Device:C C9
 U 1 1 5C00F59F
 P 2170 6460
-F 0 "C?" H 2285 6506 50  0000 L CNN
+F 0 "C9" H 2285 6506 50  0000 L CNN
 F 1 "10uF" H 2285 6415 50  0000 L CNN
 F 2 "" H 2208 6310 50  0001 C CNN
@@
 CAN_RX
 $Comp
-L Device:Crystal Y?
+L Device:Crystal Y1
 U 1 1 5C01FE22
 P 6350 5940
-F 0 "Y?" V 6304 6071 50  0000 L CNN
+F 0 "Y1" V 6304 6071 50  0000 L CNN
 F 1 "Crystal" V 6395 6071 50  0000 L CNN
 F 2 "" H 6350 5940 50  0001 C CNN
@@
 Connection ~ 6350 6210
 $Comp
-L Device:C C?
+L Device:C C5
 U 1 1 5C03346C
 P 6000 5670
-F 0 "C?" V 5748 5670 50  0000 C CNN
+F 0 "C5" V 5748 5670 50  0000 C CNN
 F 1 "26pF" V 5839 5670 50  0000 C CNN
 F 2 "" H 6038 5520 50  0001 C CNN
@@
 $EndComp
 $Comp
-L Device:C C?
+L Device:C C6
 U 1 1 5C03711D
 P 6000 6210
-F 0 "C?" V 5748 6210 50  0000 C CNN
+F 0 "C6" V 5748 6210 50  0000 C CNN
 F 1 "26pF" V 5839 6210 50  0000 C CNN
 F 2 "" H 6038 6060 50  0001 C CNN
@@
 Text Label 6640 6210 0    50   ~ 0
 OSC2
-Text Notes 1920 2730 0    50   ~ 0
-3.3V
 $Comp
 L power:+5V #PWR?
@@
 OSC1
 $Comp
-L flight_instr:SN74LVC2T45 U?
+L flight_instr:SN74LVC2T45 U4
 U 1 1 5C0464AE
 P 8440 4610
-F 0 "U?" H 8440 5047 60  0000 C CNN
+F 0 "U4" H 8440 5047 60  0000 C CNN
 F 1 "SN74LVC2T45" H 8440 4941 60  0000 C CNN
 F 2 "" H 8540 4610 60  0001 C CNN
@@
 $EndComp
 $Comp
-L Device:C C?
+L Device:C C7
 U 1 1 5C0464C1
 P 7630 4070
-F 0 "C?" V 7378 4070 50  0000 C CNN
+F 0 "C7" V 7378 4070 50  0000 C CNN
 F 1 "10nF" V 7469 4070 50  0000 C CNN
 F 2 "Capacitor_SMD:C_0805_2012Metric_Pad1.15x1.40mm_HandSolder" H 7668 3920 50  0001 C CNN
@@
 $EndComp
 $Comp
-L Device:C C?
+L Device:C C8
 U 1 1 5C0464E4
 P 9410 4070
-F 0 "C?" V 9158 4070 50  0000 C CNN
+F 0 "C8" V 9158 4070 50  0000 C CNN
 F 1 "10nF" V 9249 4070 50  0000 C CNN
 F 2 "Capacitor_SMD:C_0805_2012Metric_Pad1.15x1.40mm_HandSolder" H 9448 3920 50  0001 C CNN
@@
 NoConn ~ 8890 4660
 $Comp
-L Device:R R?
+L Device:R R6
 U 1 1 5C0A419E
 P 7120 4320
-F 0 "R?" H 7190 4366 50  0000 L CNN
+F 0 "R6" H 7190 4366 50  0000 L CNN
 F 1 "10K" H 7190 4275 50  0000 L CNN
 F 2 "" V 7050 4320 50  0001 C CNN
@@
 	9360 4760 9360 4700
 $Comp
-L Device:R R?
+L Device:R R13
 U 1 1 5C0EE468
 P 9200 2590
-F 0 "R?" H 9270 2636 50  0000 L CNN
-F 1 "1K" H 9270 2545 50  0000 L CNN
+F 0 "R13" H 9270 2636 50  0000 L CNN
+F 1 "10K" H 9270 2545 50  0000 L CNN
 F 2 "" V 9130 2590 50  0001 C CNN
 F 3 "~" H 9200 2590 50  0001 C CNN
@@
 $EndComp
 $Comp
-L Device:R R?
+L Device:R R14
 U 1 1 5C0F19D9
 P 9200 2890
-F 0 "R?" H 9270 2936 50  0000 L CNN
-F 1 "2K" H 9270 2845 50  0000 L CNN
+F 0 "R14" H 9270 2936 50  0000 L CNN
+F 1 "20K" H 9270 2845 50  0000 L CNN
 F 2 "" V 9130 2890 50  0001 C CNN
 F 3 "~" H 9200 2890 50  0001 C CNN
@@
 	9200 2440 8990 2440
 $Comp
-L Device:R R?
+L Device:R R9
 U 1 1 5C1063B4
 P 9210 1570
-F 0 "R?" H 9280 1616 50  0000 L CNN
-F 1 "1K" H 9280 1525 50  0000 L CNN
+F 0 "R9" H 9280 1616 50  0000 L CNN
+F 1 "10K" H 9280 1525 50  0000 L CNN
 F 2 "" V 9140 1570 50  0001 C CNN
 F 3 "~" H 9210 1570 50  0001 C CNN
@@
 $EndComp
 $Comp
-L Device:R R?
+L Device:R R10
 U 1 1 5C1063BB
 P 9210 1870
-F 0 "R?" H 9280 1916 50  0000 L CNN
-F 1 "2" H 9280 1825 50  0000 L CNN
+F 0 "R10" H 9280 1916 50  0000 L CNN
+F 1 "20K" H 9280 1825 50  0000 L CNN
 F 2 "" V 9140 1870 50  0001 C CNN
 F 3 "~" H 9210 1870 50  0001 C CNN
@@
 	8890 4460 9260 4460
 Connection ~ 9260 4070
+$Comp
+L Device:R R7
+U 1 1 5C1DEF5B
+P 7560 1620
+F 0 "R7" H 7630 1666 50  0000 L CNN
+F 1 "10K" H 7630 1575 50  0000 L CNN
+F 2 "" V 7490 1620 50  0001 C CNN
+F 3 "~" H 7560 1620 50  0001 C CNN
+	1    7560 1620
+	1    0    0    -1
+$EndComp
+$Comp
+L Device:R R8
+U 1 1 5C1DEF62
+P 7560 1920
+F 0 "R8" H 7630 1966 50  0000 L CNN
+F 1 "20K" H 7630 1875 50  0000 L CNN
+F 2 "" V 7490 1920 50  0001 C CNN
+F 3 "~" H 7560 1920 50  0001 C CNN
+	1    7560 1920
+	1    0    0    -1
+$EndComp
+$Comp
+L power:GND #PWR?
+U 1 1 5C1DEF69
+P 7560 2070
+F 0 "#PWR?" H 7560 1820 50  0001 C CNN
+F 1 "GND" H 7565 1897 50  0000 C CNN
+F 2 "" H 7560 2070 50  0001 C CNN
+F 3 "" H 7560 2070 50  0001 C CNN
+	1    7560 2070
+	1    0    0    -1
+$EndComp
+Wire Wire Line
+	7560 1770 7800 1770
+Connection ~ 7560 1770
+Text HLabel 7800 1770 2    50   Input ~ 0
+PIC_ON_OFF_3V3
+Text Label 7350 1470 2    50   ~ 0
+ON_OFF
+Wire Wire Line
+	7560 1470 7350 1470
+Text Label 1290 4380 2    50   ~ 0
+WAKEUP
+$Comp
+L Device:R R11
+U 1 1 5C1E36CC
+P 7560 2560
+F 0 "R11" H 7630 2606 50  0000 L CNN
+F 1 "10K" H 7630 2515 50  0000 L CNN
+F 2 "" V 7490 2560 50  0001 C CNN
+F 3 "~" H 7560 2560 50  0001 C CNN
+	1    7560 2560
+	1    0    0    -1
+$EndComp
+$Comp
+L Device:R R12
+U 1 1 5C1E36D3
+P 7560 2860
+F 0 "R12" H 7630 2906 50  0000 L CNN
+F 1 "20K" H 7630 2815 50  0000 L CNN
+F 2 "" V 7490 2860 50  0001 C CNN
+F 3 "~" H 7560 2860 50  0001 C CNN
+	1    7560 2860
+	1    0    0    -1
+$EndComp
+$Comp
+L power:GND #PWR?
+U 1 1 5C1E36DA
+P 7560 3010
+F 0 "#PWR?" H 7560 2760 50  0001 C CNN
+F 1 "GND" H 7565 2837 50  0000 C CNN
+F 2 "" H 7560 3010 50  0001 C CNN
+F 3 "" H 7560 3010 50  0001 C CNN
+	1    7560 3010
+	1    0    0    -1
+$EndComp
+Wire Wire Line
+	7560 2710 7800 2710
+Connection ~ 7560 2710
+Text HLabel 7800 2710 2    50   Input ~ 0
+PIC_WAKEUP_3V3
+Text Label 7350 2410 2    50   ~ 0
+WAKEUP
+Wire Wire Line
+	7560 2410 7350 2410
 $EndSCHEMATC

Commit message: Address final changes: Add 0 ohm resistor in the Enable pin of U4 (the new level shifter) Replace the old voltage divider with a bidirection level shifter Modify library as necessary
Parts:
- removed R13: 10K, symbol Device:R
- removed R14: 20K, symbol Device:R
- removed U4: SN74LVC2T45, symbol flight_instr:SN74LVC2T45
- added R7: 10K, symbol Device:R
- added R8: 0, symbol Device:R
- added U4: NLSX4373_LEVEL_SHIFTER, symbol canhw:NLSX4373DR2GOSCT-ND_LEVEL_SHIFTER
- renumbered R7 to R13, R8 to R14
Connections:
- wire segments 77 -> 71
- no-connect marks 3 -> 1
Other:
- moved on the sheet: C7, C8, R10, R11, R12, R13, R14, R6, R9

Commit message: Address final changes. Colour in Level Shifter, removed extra pull-up resistors and  rename U4
Parts:
- removed R6, R7: 10K, symbol Device:R
- U4: value NLSX4373_LEVEL_SHIFTER -> NLSX4373
Connections:
- wire segments 71 -> 73
Changed lines of the file:
@@
 RESET_5V
-$Comp
-L Device:R R6
-U 1 1 5C0A419E
-P 9390 4560
-F 0 "R6" H 9460 4606 50  0000 L CNN
-F 1 "10K" H 9460 4515 50  0000 L CNN
-F 2 "" V 9320 4560 50  0001 C CNN
-F 3 "~" H 9390 4560 50  0001 C CNN
-	1    9390 4560
-	1    0    0    -1
-$EndComp
 $Comp
 L power:+3V3 #PWR?
@@
 P 8130 4660
 F 0 "U4" H 8130 5075 50  0000 C CNN
-F 1 "NLSX4373_LEVEL_SHIFTER" H 8130 4984 50  0000 C CNN
+F 1 "NLSX4373" H 8130 4984 50  0000 C CNN
 F 2 "" H 8130 4960 50  0001 C CNN
 F 3 "" H 8130 4960 50  0001 C CNN
@@
 	1    0    0    -1
 $EndComp
-$Comp
-L Device:R R7
-U 1 1 5C4BFD33
-P 6960 4460
-F 0 "R7" H 7030 4506 50  0000 L CNN
-F 1 "10K" H 7030 4415 50  0000 L CNN
-F 2 "" V 6890 4460 50  0001 C CNN
-F 3 "~" H 6960 4460 50  0001 C CNN
-	1    6960 4460
-	1    0    0    -1
-$EndComp
-Wire Wire Line
-	6960 4610 7580 4610
-Wire Wire Line
-	6960 4610 6830 4610
-Connection ~ 6960 4610
 $Comp
 L power:+5V #PWR?
@@
 $EndComp
 Wire Wire Line
-	8680 4710 9390 4710
-Connection ~ 9390 4710
-Wire Wire Line
-	9390 4710 9440 4710
-Wire Wire Line
 	8680 4810 10230 4810
 $Comp
@@
 	1    0    0    -1
 $EndComp
+Wire Wire Line
+	6830 4610 6960 4610
+Wire Wire Line
+	8680 4710 9390 4710
+Wire Wire Line
+	9390 4410 9390 4710
+Connection ~ 9390 4710
+Wire Wire Line
+	9390 4710 9440 4710
+Wire Wire Line
+	6960 4310 6960 4610
+Connection ~ 6960 4610
+Wire Wire Line
+	6960 4610 7580 4610
 $EndSCHEMATC

Commit message: Initial draft of GPS PCB layout; fixed GPS_TX connection
Parts:
- C7: renamed from C5; footprint (none) -> Capacitor_SMD:C_0805_2012Metric_Pad1.15x1.40mm_HandSolder
- C8: renamed from C6; footprint (none) -> Capacitor_SMD:C_0805_2012Metric_Pad1.15x1.40mm_HandSolder
- C9: footprint (none) -> Capacitor_SMD:C_0805_2012Metric_Pad1.15x1.40mm_HandSolder
- J2: footprint (none) -> canhw_footprints:PinHeader_5x2.54_SMD_90deg_952-3198-1-ND
- R12: renamed from R8; footprint (none) -> Resistor_SMD:R_0805_2012Metric_Pad1.15x1.40mm_HandSolder
- R2: renamed from R9; footprint (none) -> Resistor_SMD:R_0805_2012Metric_Pad1.15x1.40mm_HandSolder
- R3: renamed from R13; footprint (none) -> Resistor_SMD:R_0805_2012Metric_Pad1.15x1.40mm_HandSolder
- R4: renamed from R11; footprint (none) -> Resistor_SMD:R_0805_2012Metric_Pad1.15x1.40mm_HandSolder
- R5: renamed from R10; footprint (none) -> Resistor_SMD:R_0805_2012Metric_Pad1.15x1.40mm_HandSolder
- R6: renamed from R14; footprint (none) -> Resistor_SMD:R_0805_2012Metric_Pad1.15x1.40mm_HandSolder
- R7: renamed from R12; footprint (none) -> Resistor_SMD:R_0805_2012Metric_Pad1.15x1.40mm_HandSolder
- U3: renamed from U2; footprint (none) -> Package_SO:SOIC-28W_7.5x18.7mm_P1.27mm; symbol canhw:PIC18F26K83 -> gps-rescue:PIC18F26K83-canhw
- U4: footprint (none) -> Package_SO:SOIC-8_3.9x4.9mm_P1.27mm; symbol canhw:NLSX4373DR2GOSCT-ND_LEVEL_SHIFTER -> gps-rescue:NLSX4373DR2GOSCT-ND_LEVEL_SHIFTER-canhw
- U5: renamed from U3; footprint (none) -> Package_SO:SOIC-8_3.9x4.9mm_P1.27mm; symbol canhw:MCP2562 -> gps-rescue:MCP2562-canhw
- Y1: footprint (none) -> Crystal:Crystal_HC49-U_Vertical
- renumbered C8 to C5, C7 to C6, R4 to R10, R5 to R11, R2 to R8, R3 to R9
Connections:
- wire segments 73 -> 71
