File: gps/gps_2.sch (KiCad schematic (older format))
At the start: 38 parts, among them J1 Programming Header, J2 CAN Bus Conn, J3 Aux. bat. conn., U1 M10578-A2, U2 PIC18F26K83, U3 MCP2562, U4 MIC5504-3.3, U5 INA180, U6 SMA_CONN, Y1 Crystal

Commit message: Address Aaron's comments: - Change D1, D2, D3 from 323_handsolering to 1206_handsoldering - Add LED colour silkscreen - Connect islands on GND, 3V3 pours - Move U3 up for cleaner CANH, CANL routing - Change INA180 routing to a 4T setup - Add team logo and board creation info
Parts:
- D1, D2, D3: footprint Diode_SMD:D_SOD-323_HandSoldering -> LED_SMD:LED_1206_3216Metric_Pad1.42x1.75mm_HandSolder
Changed lines of the file:
@@
 F 0 "D3" V 10680 2350 50  0000 C CNN
 F 1 "BLUE" V 10580 2350 50  0000 C CNN
-F 2 "Diode_SMD:D_SOD-323_HandSoldering" H 10630 2200 50  0001 C CNN
+F 2 "LED_SMD:LED_1206_3216Metric_Pad1.42x1.75mm_HandSolder" H 10630 2200 50  0001 C CNN
 F 3 "~" H 10630 2200 50  0001 C CNN
 	1    10630 2200
@@
 F 0 "D2" V 10380 2350 50  0000 C CNN
 F 1 "RED" V 10280 2350 50  0000 C CNN
-F 2 "Diode_SMD:D_SOD-323_HandSoldering" H 10330 2200 50  0001 C CNN
+F 2 "LED_SMD:LED_1206_3216Metric_Pad1.42x1.75mm_HandSolder" H 10330 2200 50  0001 C CNN
 F 3 "~" H 10330 2200 50  0001 C CNN
 	1    10330 2200
@@
 F 0 "D1" V 6819 5973 50  0000 R CNN
 F 1 "WHITE" V 6728 5973 50  0000 R CNN
-F 2 "Diode_SMD:D_SOD-323_HandSoldering" H 6780 6090 50  0001 C CNN
+F 2 "LED_SMD:LED_1206_3216Metric_Pad1.42x1.75mm_HandSolder" H 6780 6090 50  0001 C CNN
 F 3 "~" H 6780 6090 50  0001 C CNN
 	1    6780 6090

Commit message: Change oscillator caps to 27pF
There aren't actually any 26pF caps on Digikey and we've been using 25
and 27pF instead. Changed in all schematics.
Parts:
- C11, C12: value 26pF -> 27pF
Changed lines of the file:
@@
 EESchema Schematic File Version 4
 LIBS:gps_2-cache
-EELAYER 30 0
+EELAYER 26 0
 EELAYER END
 $Descr A4 11693 8268
@@
 P 5610 1130
 F 0 "C11" V 5358 1130 50  0000 C CNN
-F 1 "26pF" V 5449 1130 50  0000 C CNN
+F 1 "27pF" V 5449 1130 50  0000 C CNN
 F 2 "Capacitor_SMD:C_0805_2012Metric_Pad1.15x1.40mm_HandSolder" H 5648 980 50  0001 C CNN
 F 3 "~" H 5610 1130 50  0001 C CNN
@@
 P 5610 1790
 F 0 "C12" V 5358 1790 50  0000 C CNN
-F 1 "26pF" V 5449 1790 50  0000 C CNN
+F 1 "27pF" V 5449 1790 50  0000 C CNN
 F 2 "Capacitor_SMD:C_0805_2012Metric_Pad1.15x1.40mm_HandSolder" H 5648 1640 50  0001 C CNN
 F 3 "~" H 5610 1790 50  0001 C CNN
