File: vent_2/vent_2.sch (KiCad schematic (older format))
At the start: 0 parts

Commit message: Finish rev 1 of vent_2
Changed lines of the file:
@@
 Wire Wire Line
 	4400 2950 4850 2950
+Text HLabel 7400 2800 0    50   Output ~ 0
+VALVE_CONTROL
+Text HLabel 7950 2800 2    50   Output ~ 0
+VALVE_CONTROL
+Wire Wire Line
+	7400 2800 7950 2800
 $EndSCHEMATC
