File: vent_2/valvectrl.sch (KiCad schematic (older format))
At the start: 0 parts

Commit message: Finish rev 1 of vent_2
Parts:
- added D1: BAS16WJ, symbol Device:D
- added J4: Valve Connection, symbol Connector:Conn_01x02_Female
- added Q1: AOD417, symbol Device:Q_NMOS_GDS
- added R10: 10K, symbol Device:R_US
- added R8: 270R, symbol Device:R_US
- added R9: 15K, symbol Device:R_US
Connections:
- new net: Q1.1 (G), R10.1, R8.1, R9.2
- new net +BATT: D1.1 (K), Q1.2 (D), R9.1
- new net CLOSE: D1.2 (A), Q1.3 (S)
- new net GND: J4.2 (Pin_2), R10.2
- new net Open: J4.1 (Pin_1)
- new net VALVE_CONTROL: R8.2
Changed lines of the file:
@@
 $Descr A4 11693 8268
 encoding utf-8
-Sheet 1 4
+Sheet 4 4
 Title ""
 Date ""
@@
 Comment4 ""
 $EndDescr
+Text HLabel 2800 5250 0    50   Input ~ 0
+VALVE_CONTROL
+$Comp
+L Device:R_US R10
+U 1 1 5DCDA7D7
+P 3500 5550
+F 0 "R10" H 3568 5596 50  0000 L CNN
+F 1 "10K" H 3568 5505 50  0000 L CNN
+F 2 "" V 3540 5540 50  0001 C CNN
+F 3 "~" H 3500 5550 50  0001 C CNN
+	1    3500 5550
+	1    0    0    -1
+$EndComp
+$Comp
+L Device:R_US R8
+U 1 1 5DCDB461
+P 3150 5250
+F 0 "R8" V 2945 5250 50  0000 C CNN
+F 1 "270R" V 3036 5250 50  0000 C CNN
+F 2 "" V 3190 5240 50  0001 C CNN
+F 3 "~" H 3150 5250 50  0001 C CNN
+	1    3150 5250
+	0    1    1    0
+$EndComp
+$Comp
+L Device:Q_NMOS_GDS Q1
+U 1 1 5DCDCBAB
+P 4050 5250
+F 0 "Q1" H 4256 5296 50  0000 L CNN
+F 1 "AOD417" H 4256 5205 50  0000 L CNN
+F 2 "" H 4250 5350 50  0001 C CNN
+F 3 "~" H 4050 5250 50  0001 C CNN
+	1    4050 5250
+	1    0    0    -1
+$EndComp
+$Comp
+L Device:D D1
+U 1 1 5DCDDCA7
+P 4700 5200
+F 0 "D1" V 4654 5279 50  0000 L CNN
+F 1 "BAS16WJ" V 4745 5279 50  0000 L CNN
+F 2 "" H 4700 5200 50  0001 C CNN
+F 3 "~" H 4700 5200 50  0001 C CNN
+	1    4700 5200
+	0    1    1    0
+$EndComp
+Wire Wire Line
+	2800 5250 3000 5250
+Wire Wire Line
+	3300 5250 3500 5250
+Wire Wire Line
+	3500 5400 3500 5250
+Connection ~ 3500 5250
+Wire Wire Line
+	3500 5250 3750 5250
+$Comp
+L power:GND #PWR?
+U 1 1 5DCDE6BA
+P 3500 5700
+F 0 "#PWR?" H 3500 5450 50  0001 C CNN
+F 1 "GND" H 3505 5527 50  0000 C CNN
+F 2 "" H 3500 5700 50  0001 C CNN
+F 3 "" H 3500 5700 50  0001 C CNN
+	1    3500 5700
+	1    0    0    -1
+$EndComp
+Text Label 4850 5600 0    50   ~ 0
+CLOSE
+Wire Wire Line
+	4150 5450 4150 5600
+$Comp
+L Connector:Conn_01x02_Female J4
+U 1 1 5DCDEFC3
+P 3650 3450
+F 0 "J4" H 3678 3426 50  0000 L CNN
+F 1 "Valve Connection" H 3678 3335 50  0000 L CNN
+F 2 "" H 3650 3450 50  0001 C CNN
+F 3 "~" H 3650 3450 50  0001 C CNN
+	1    3650 3450
+	1    0    0    -1
+$EndComp
+Wire Wire Line
+	4150 5600 4700 5600
+Wire Wire Line
+	4700 5350 4700 5600
+Connection ~ 4700 5600
+Wire Wire Line
+	4700 5600 4850 5600
+$Comp
+L power:+BATT #PWR?
+U 1 1 5DCE091A
+P 4400 4450
+F 0 "#PWR?" H 4400 4300 50  0001 C CNN
+F 1 "+BATT" H 4415 4623 50  0000 C CNN
+F 2 "" H 4400 4450 50  0001 C CNN
+F 3 "" H 4400 4450 50  0001 C CNN
+	1    4400 4450
+	1    0    0    -1
+$EndComp
+Wire Wire Line
+	4700 5050 4700 4600
+Wire Wire Line
+	4150 4600 4150 5050
+Wire Wire Line
+	4150 4600 4400 4600
+Wire Wire Line
+	4400 4450 4400 4600
+Connection ~ 4400 4600
+Wire Wire Line
+	4400 4600 4700 4600
+$Comp
+L Device:R_US R9
+U 1 1 5DCE17D1
+P 3750 4850
+F 0 "R9" H 3818 4896 50  0000 L CNN
+F 1 "15K" H 3818 4805 50  0000 L CNN
+F 2 "" V 3790 4840 50  0001 C CNN
+F 3 "~" H 3750 4850 50  0001 C CNN
+	1    3750 4850
+	1    0    0    -1
+$EndComp
+Wire Wire Line
+	4150 4600 3750 4600
+Wire Wire Line
+	3750 4600 3750 4700
+Connection ~ 4150 4600
+Wire Wire Line
+	3750 5000 3750 5250
+Connection ~ 3750 5250
+Wire Wire Line
+	3750 5250 3850 5250
+Text Label 3150 3450 2    50   ~ 0
+Open
+$Comp
+L power:GND #PWR?
+U 1 1 5DCE229A
+P 3200 3550
+F 0 "#PWR?" H 3200 3300 50  0001 C CNN
+F 1 "GND" H 3205 3377 50  0000 C CNN
+F 2 "" H 3200 3550 50  0001 C CNN
+F 3 "" H 3200 3550 50  0001 C CNN
+	1    3200 3550
+	1    0    0    -1
+$EndComp
+Wire Wire Line
+	3450 3450 3150 3450
+Wire Wire Line
+	3450 3550 3200 3550
 $EndSCHEMATC

Commit message: Fix typo
Connections:
- net Open is gone; now on net CLOSE: J4.1 (Pin_1)
Changed lines of the file:
@@
 	3750 5250 3850 5250
 Text Label 3150 3450 2    50   ~ 0
-Open
+CLOSE
 $Comp
 L power:GND #PWR?

Commit message: Attempt 2 for the mosfets
Parts:
- removed R10: 10K, symbol Device:R_US
- removed R9: 15K, symbol Device:R_US
- D1: value BAS16WJ -> BAS16GWJ
- Q1: value AOD417 -> Q_NMOS_GDS
Connections:
- net GND: now also Q1.3 (S); no longer J4.2 (Pin_2)
- net +BATT renamed +12V
- net +12V: now also J4.1 (Pin_1); no longer Q1.2 (D)
- removed net CLOSE: D1.2 (A), J4.1 (Pin_1), Q1.3 (S)
- new net RELAY-: D1.2 (A), J4.2 (Pin_2), Q1.2 (D)
Changed lines of the file:
@@
 VALVE_CONTROL
-$Comp
-L Device:R_US R10
-U 1 1 5DCDA7D7
-P 3500 5550
-F 0 "R10" H 3568 5596 50  0000 L CNN
-F 1 "10K" H 3568 5505 50  0000 L CNN
-F 2 "" V 3540 5540 50  0001 C CNN
-F 3 "~" H 3500 5550 50  0001 C CNN
-	1    3500 5550
-	1    0    0    -1
-$EndComp
 $Comp
 L Device:R_US R8
@@
 	0    1    1    0
 $EndComp
-$Comp
-L Device:Q_NMOS_GDS Q1
-U 1 1 5DCDCBAB
-P 4050 5250
-F 0 "Q1" H 4256 5296 50  0000 L CNN
-F 1 "AOD417" H 4256 5205 50  0000 L CNN
-F 2 "" H 4250 5350 50  0001 C CNN
-F 3 "~" H 4050 5250 50  0001 C CNN
-	1    4050 5250
-	1    0    0    -1
-$EndComp
-$Comp
-L Device:D D1
-U 1 1 5DCDDCA7
-P 4700 5200
-F 0 "D1" V 4654 5279 50  0000 L CNN
-F 1 "BAS16WJ" V 4745 5279 50  0000 L CNN
-F 2 "" H 4700 5200 50  0001 C CNN
-F 3 "~" H 4700 5200 50  0001 C CNN
-	1    4700 5200
-	0    1    1    0
-$EndComp
 Wire Wire Line
 	2800 5250 3000 5250
-Wire Wire Line
-	3300 5250 3500 5250
-Wire Wire Line
-	3500 5400 3500 5250
-Connection ~ 3500 5250
-Wire Wire Line
-	3500 5250 3750 5250
-$Comp
-L power:GND #PWR?
-U 1 1 5DCDE6BA
-P 3500 5700
-F 0 "#PWR?" H 3500 5450 50  0001 C CNN
-F 1 "GND" H 3505 5527 50  0000 C CNN
-F 2 "" H 3500 5700 50  0001 C CNN
-F 3 "" H 3500 5700 50  0001 C CNN
-	1    3500 5700
-	1    0    0    -1
-$EndComp
-Text Label 4850 5600 0    50   ~ 0
-CLOSE
-Wire Wire Line
-	4150 5450 4150 5600
 $Comp
 L Connector:Conn_01x02_Female J4
@@
 	1    0    0    -1
 $EndComp
+Text Label 3200 3550 2    50   ~ 0
+RELAY-
 Wire Wire Line
-	4150 5600 4700 5600
-Wire Wire Line
-	4700 5350 4700 5600
-Connection ~ 4700 5600
-Wire Wire Line
-	4700 5600 4850 5600
+	3450 3550 3200 3550
 $Comp
-L power:+BATT #PWR?
-U 1 1 5DCE091A
-P 4400 4450
-F 0 "#PWR?" H 4400 4300 50  0001 C CNN
-F 1 "+BATT" H 4415 4623 50  0000 C CNN
-F 2 "" H 4400 4450 50  0001 C CNN
-F 3 "" H 4400 4450 50  0001 C CNN
-	1    4400 4450
+L Device:Q_NMOS_GDS Q1
+U 1 1 5DCE1675
+P 3650 5250
+F 0 "Q1" H 3856 5296 50  0000 L CNN
+F 1 "Q_NMOS_GDS" H 3856 5205 50  0000 L CNN
+F 2 "" H 3850 5350 50  0001 C CNN
+F 3 "~" H 3650 5250 50  0001 C CNN
+	1    3650 5250
 	1    0    0    -1
 $EndComp
 Wire Wire Line
-	4700 5050 4700 4600
-Wire Wire Line
-	4150 4600 4150 5050
-Wire Wire Line
-	4150 4600 4400 4600
-Wire Wire Line
-	4400 4450 4400 4600
-Connection ~ 4400 4600
-Wire Wire Line
-	4400 4600 4700 4600
+	3300 5250 3450 5250
 $Comp
-L Device:R_US R9
-U 1 1 5DCE17D1
-P 3750 4850
-F 0 "R9" H 3818 4896 50  0000 L CNN
-F 1 "15K" H 3818 4805 50  0000 L CNN
-F 2 "" V 3790 4840 50  0001 C CNN
-F 3 "~" H 3750 4850 50  0001 C CNN
-	1    3750 4850
+L power:GND #PWR?
+U 1 1 5DCE259E
+P 3750 5700
+F 0 "#PWR?" H 3750 5450 50  0001 C CNN
+F 1 "GND" H 3755 5527 50  0000 C CNN
+F 2 "" H 3750 5700 50  0001 C CNN
+F 3 "" H 3750 5700 50  0001 C CNN
+	1    3750 5700
 	1    0    0    -1
 $EndComp
 Wire Wire Line
-	4150 4600 3750 4600
+	3750 5450 3750 5700
+Text Label 3750 4800 0    50   ~ 0
+RELAY-
 Wire Wire Line
-	3750 4600 3750 4700
-Connection ~ 4150 4600
+	3750 4800 3750 4900
+Text Label 3850 4300 0    50   ~ 0
+RELAY+
+Text Label 3200 3450 2    50   ~ 0
+RELAY+
 Wire Wire Line
-	3750 5000 3750 5250
-Connection ~ 3750 5250
-Wire Wire Line
-	3750 5250 3850 5250
-Text Label 3150 3450 2    50   ~ 0
-CLOSE
+	3200 3450 3450 3450
 $Comp
-L power:GND #PWR?
-U 1 1 5DCE229A
-P 3200 3550
-F 0 "#PWR?" H 3200 3300 50  0001 C CNN
-F 1 "GND" H 3205 3377 50  0000 C CNN
-F 2 "" H 3200 3550 50  0001 C CNN
-F 3 "" H 3200 3550 50  0001 C CNN
-	1    3200 3550
+L power:+12V #PWR?
+U 1 1 5DCE3D3C
+P 3750 4100
+F 0 "#PWR?" H 3750 3950 50  0001 C CNN
+F 1 "+12V" H 3765 4273 50  0000 C CNN
+F 2 "" H 3750 4100 50  0001 C CNN
+F 3 "" H 3750 4100 50  0001 C CNN
+	1    3750 4100
 	1    0    0    -1
 $EndComp
 Wire Wire Line
-	3450 3450 3150 3450
+	3750 4100 3750 4200
+$Comp
+L Device:D D1
+U 1 1 5DCE4645
+P 3500 4550
+F 0 "D1" V 3454 4629 50  0000 L CNN
+F 1 "BAS16GWJ" V 3545 4629 50  0000 L CNN
+F 2 "" H 3500 4550 50  0001 C CNN
+F 3 "~" H 3500 4550 50  0001 C CNN
+	1    3500 4550
+	0    1    1    0
+$EndComp
 Wire Wire Line
-	3450 3550 3200 3550
+	3500 4700 3500 4900
+Wire Wire Line
+	3500 4900 3750 4900
+Connection ~ 3750 4900
+Wire Wire Line
+	3750 4900 3750 5050
+Wire Wire Line
+	3500 4400 3500 4200
+Wire Wire Line
+	3500 4200 3750 4200
+Connection ~ 3750 4200
+Wire Wire Line
+	3750 4200 3750 4300
+Wire Wire Line
+	3850 4300 3750 4300
 $EndSCHEMATC
