File: recovery/_autosave-recovery_CAN.kicad_pcb (KiCad board)
At the start: 2 copper layers, 54 parts, among them J1 Conn_01x05_Female, J4 Conn_01x05_Female, Q1 DMG2302UK, Q2 DMG2302UK, Q3 AOD417, Q4 AOD417, Q5 BSS138, U1 MCP2562, U2 PIC18F26K83, U3 L78L05AC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

Commit message: Redesined scematic to reflect change to conectors for altimeter wiring, added more solder jumpers for increased board flexibility, created PCB file.
Parts:
- moved J4 37.6 mm to (193.0, 64.8)
Changed lines of the file:
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@@
   )
   (module canhw_footprints:connector_Harwin_M80-5000642 (layer F.Cu)
-    (at 203.655001 28.745001)
+    (at 193.04 64.77)
     (fp_text reference J4 (at 0 0.5) (layer F.SilkS)
       (effects (font (size 1 1) (thickness 0.15)))
