File: rocketlog/rocketlog_2/logger_power.sch (KiCad schematic (older format))
At the start: 8 parts, among them J4 BUS CONN, U3 AP2114H-3.3, U4 INA180

Commit message: Add first pass of traces
Also
- make LEDs run on 3v3 instead of 5V
- change footprints for CAN connector and crystal
Parts:
- J4: footprint canhw_footprints:connector_Harwin_M80-5420642 -> canhw_footprints:connector_Harwin_M80-5000642
Changed lines of the file:
@@
 $Descr A4 11693 8268
 encoding utf-8
-Sheet 4 3
+Sheet 3 3
 Title ""
 Date ""
@@
 F 0 "J4" H 2644 2725 50  0000 C CNN
 F 1 "BUS CONN" H 2644 2816 50  0000 C CNN
-F 2 "canhw_footprints:connector_Harwin_M80-5420642" H 2750 3150 50  0001 C CNN
+F 2 "canhw_footprints:connector_Harwin_M80-5000642" H 2750 3150 50  0001 C CNN
 F 3 "~" H 2750 3150 50  0001 C CNN
 	1    2750 3150
