File: live_telemetry/telemetry_transmitter/telemetry_transmitter.sch (KiCad schematic (older format))
At the start: 15 parts, among them J1 Programming Header, U1 PIC18F26K83, U2 MCP2562, Y1 Crystal

Commit message: Add pull downs to the RESET lines
Parts:
- added R17: 10k, symbol Device:R_US
Connections:
- net GND: now also R17.2
- net radio/RESET: now also R17.1
Changed lines of the file:
@@
 $EndSheet
 Wire Wire Line
-	6550 4000 7400 4000
+	6550 4000 7050 4000
+$Comp
+L Device:R_US R17
+U 1 1 5E2883A8
+P 7050 4200
+F 0 "R17" H 7118 4246 50  0000 L CNN
+F 1 "10k" H 7118 4155 50  0000 L CNN
+F 2 "" V 7090 4190 50  0001 C CNN
+F 3 "~" H 7050 4200 50  0001 C CNN
+	1    7050 4200
+	1    0    0    -1
+$EndComp
+$Comp
+L power:GND #PWR052
+U 1 1 5E288D4E
+P 7050 4350
+F 0 "#PWR052" H 7050 4100 50  0001 C CNN
+F 1 "GND" H 7055 4177 50  0000 C CNN
+F 2 "" H 7050 4350 50  0001 C CNN
+F 3 "" H 7050 4350 50  0001 C CNN
+	1    7050 4350
+	1    0    0    -1
+$EndComp
+Wire Wire Line
+	7050 4050 7050 4000
+Connection ~ 7050 4000
+Wire Wire Line
+	7050 4000 7400 4000
 $EndSCHEMATC

Commit message: Add initial PCB layouts
Parts:
- C1, C2, C3, C4: footprint (none) -> Capacitor_SMD:C_0805_2012Metric_Pad1.15x1.40mm_HandSolder
- D1, D2, D3: footprint (none) -> LED_SMD:LED_1206_3216Metric_Pad1.42x1.75mm_HandSolder
- J1: footprint (none) -> Connector_PinSocket_2.54mm:PinSocket_1x05_P2.54mm_Horizontal
- R1, R17, R2, R3, R4: footprint (none) -> Resistor_SMD:R_0805_2012Metric_Pad1.15x1.40mm_HandSolder
- U1: footprint (none) -> Package_SO:SOIC-28W_7.5x18.7mm_P1.27mm
- U2: footprint (none) -> Package_SO:SOIC-8_3.9x4.9mm_P1.27mm
- Y1: footprint (none) -> Crystal:Crystal_HC49-U_Vertical
Changed lines of the file:
@@
 F 0 "U1" H 5825 4565 50  0000 C CNN
 F 1 "PIC18F26K83" H 5825 4474 50  0000 C CNN
-F 2 "" H 6300 3650 50  0001 C CNN
+F 2 "Package_SO:SOIC-28W_7.5x18.7mm_P1.27mm" H 6300 3650 50  0001 C CNN
 F 3 "http://ww1.microchip.com/downloads/en/DeviceDoc/40001943A.pdf" H 6300 3650 50  0001 C CNN
 	1    5850 3650
@@
 F 0 "C3" V 7002 2800 50  0000 C CNN
 F 1 "0.1u" V 6911 2800 50  0000 C CNN
-F 2 "" H 6788 2650 50  0001 C CNN
+F 2 "Capacitor_SMD:C_0805_2012Metric_Pad1.15x1.40mm_HandSolder" H 6788 2650 50  0001 C CNN
 F 3 "~" H 6750 2800 50  0001 C CNN
 	1    6750 2800
@@
 F 0 "R4" H 4632 2754 50  0000 R CNN
 F 1 "10K" H 4632 2845 50  0000 R CNN
-F 2 "" V 4740 2790 50  0001 C CNN
+F 2 "Resistor_SMD:R_0805_2012Metric_Pad1.15x1.40mm_HandSolder" V 4740 2790 50  0001 C CNN
 F 3 "~" H 4700 2800 50  0001 C CNN
 	1    4700 2800
@@
 F 0 "C4" H 8715 5196 50  0000 L CNN
 F 1 "10u" H 8715 5105 50  0000 L CNN
-F 2 "" H 8638 5000 50  0001 C CNN
+F 2 "Capacitor_SMD:C_0805_2012Metric_Pad1.15x1.40mm_HandSolder" H 8638 5000 50  0001 C CNN
 F 3 "~" H 8600 5150 50  0001 C CNN
 	1    8600 5150
@@
 F 0 "Y1" V 3204 5781 50  0000 L CNN
 F 1 "Crystal" V 3295 5781 50  0000 L CNN
-F 2 "" H 3250 5650 50  0001 C CNN
+F 2 "Crystal:Crystal_HC49-U_Vertical" H 3250 5650 50  0001 C CNN
 F 3 "~" H 3250 5650 50  0001 C CNN
 	1    3250 5650
@@
 F 0 "C1" V 2498 5400 50  0000 C CNN
 F 1 "26p" V 2589 5400 50  0000 C CNN
-F 2 "" H 2788 5250 50  0001 C CNN
+F 2 "Capacitor_SMD:C_0805_2012Metric_Pad1.15x1.40mm_HandSolder" H 2788 5250 50  0001 C CNN
 F 3 "~" H 2750 5400 50  0001 C CNN
 	1    2750 5400
@@
 F 0 "C2" V 2498 5900 50  0000 C CNN
 F 1 "26p" V 2589 5900 50  0000 C CNN
-F 2 "" H 2788 5750 50  0001 C CNN
+F 2 "Capacitor_SMD:C_0805_2012Metric_Pad1.15x1.40mm_HandSolder" H 2788 5750 50  0001 C CNN
 F 3 "~" H 2750 5900 50  0001 C CNN
 	1    2750 5900
@@
 F 0 "J1" H 1742 1725 50  0000 C CNN
 F 1 "Programming Header" H 1742 1816 50  0000 C CNN
-F 2 "" H 1850 2150 50  0001 C CNN
+F 2 "Connector_PinSocket_2.54mm:PinSocket_1x05_P2.54mm_Horizontal" H 1850 2150 50  0001 C CNN
 F 3 "~" H 1850 2150 50  0001 C CNN
 	1    1850 2150
@@
 F 0 "U2" H 9375 4915 50  0000 C CNN
 F 1 "MCP2562" H 9375 4824 50  0000 C CNN
-F 2 "" H 9400 4650 50  0001 C CNN
+F 2 "Package_SO:SOIC-8_3.9x4.9mm_P1.27mm" H 9400 4650 50  0001 C CNN
 F 3 "http://hades.mech.northwestern.edu/images/5/5e/MCP2562.pdf" H 9400 4650 50  0001 C CNN
 	1    9400 4650
@@
 F 0 "R1" H 2068 3896 50  0000 L CNN
 F 1 "130" H 2068 3805 50  0000 L CNN
-F 2 "" V 2040 3840 50  0001 C CNN
+F 2 "Resistor_SMD:R_0805_2012Metric_Pad1.15x1.40mm_HandSolder" V 2040 3840 50  0001 C CNN
 F 3 "~" H 2000 3850 50  0001 C CNN
 	1    2000 3850
@@
 F 0 "R2" H 2418 3896 50  0000 L CNN
 F 1 "130" H 2418 3805 50  0000 L CNN
-F 2 "" V 2390 3840 50  0001 C CNN
+F 2 "Resistor_SMD:R_0805_2012Metric_Pad1.15x1.40mm_HandSolder" V 2390 3840 50  0001 C CNN
 F 3 "~" H 2350 3850 50  0001 C CNN
 	1    2350 3850
@@
 F 0 "R3" H 2768 3896 50  0000 L CNN
 F 1 "130" H 2768 3805 50  0000 L CNN
-F 2 "" V 2740 3840 50  0001 C CNN
+F 2 "Resistor_SMD:R_0805_2012Metric_Pad1.15x1.40mm_HandSolder" V 2740 3840 50  0001 C CNN
 F 3 "~" H 2700 3850 50  0001 C CNN
 	1    2700 3850
@@
 F 0 "D1" V 2039 3433 50  0000 R CNN
 F 1 "LED" V 1948 3433 50  0000 R CNN
-F 2 "" H 2000 3550 50  0001 C CNN
+F 2 "LED_SMD:LED_1206_3216Metric_Pad1.42x1.75mm_HandSolder" H 2000 3550 50  0001 C CNN
 F 3 "~" H 2000 3550 50  0001 C CNN
 	1    2000 3550
@@
 F 0 "D2" V 2389 3433 50  0000 R CNN
 F 1 "LED" V 2298 3433 50  0000 R CNN
-F 2 "" H 2350 3550 50  0001 C CNN
+F 2 "LED_SMD:LED_1206_3216Metric_Pad1.42x1.75mm_HandSolder" H 2350 3550 50  0001 C CNN
 F 3 "~" H 2350 3550 50  0001 C CNN
 	1    2350 3550
@@
 F 0 "D3" V 2739 3433 50  0000 R CNN
 F 1 "LED" V 2648 3433 50  0000 R CNN
-F 2 "" H 2700 3550 50  0001 C CNN
+F 2 "LED_SMD:LED_1206_3216Metric_Pad1.42x1.75mm_HandSolder" H 2700 3550 50  0001 C CNN
 F 3 "~" H 2700 3550 50  0001 C CNN
 	1    2700 3550
@@
 F 0 "R17" H 7118 4246 50  0000 L CNN
 F 1 "10k" H 7118 4155 50  0000 L CNN
-F 2 "" V 7090 4190 50  0001 C CNN
+F 2 "Resistor_SMD:R_0805_2012Metric_Pad1.15x1.40mm_HandSolder" V 7090 4190 50  0001 C CNN
 F 3 "~" H 7050 4200 50  0001 C CNN
 	1    7050 4200

Commit message: Change oscillator caps to 27pF
There aren't actually any 26pF caps on Digikey and we've been using 25
and 27pF instead. Changed in all schematics.
Parts:
- C1, C2: value 26p -> 27pF
Changed lines of the file:
@@
 EESchema Schematic File Version 4
-LIBS:telemetry_transmitter-cache
-EELAYER 29 0
+EELAYER 26 0
 EELAYER END
 $Descr A4 11693 8268
@@
 P 2750 5400
 F 0 "C1" V 2498 5400 50  0000 C CNN
-F 1 "26p" V 2589 5400 50  0000 C CNN
+F 1 "27pF" V 2589 5400 50  0000 C CNN
 F 2 "Capacitor_SMD:C_0805_2012Metric_Pad1.15x1.40mm_HandSolder" H 2788 5250 50  0001 C CNN
 F 3 "~" H 2750 5400 50  0001 C CNN
@@
 P 2750 5900
 F 0 "C2" V 2498 5900 50  0000 C CNN
-F 1 "26p" V 2589 5900 50  0000 C CNN
+F 1 "27pF" V 2589 5900 50  0000 C CNN
 F 2 "Capacitor_SMD:C_0805_2012Metric_Pad1.15x1.40mm_HandSolder" H 2788 5750 50  0001 C CNN
 F 3 "~" H 2750 5900 50  0001 C CNN
