File: sensor_mini/power.sch (KiCad schematic (older format))
At the start: 10 parts, among them J1 Conn_01x05_Female, U4 INA180, U8 MIC5365-1.8

Commit message: Sensor mini: Add analog stuff
Adds one thermistor and the tank pressure sensor to sensor_mini.
Required making the board a quarter inch wider. This commit updates the
PCB and the schematic.

Note that while all the traces are there (DRC mostly passes (IMU is too
small for 6mil DRC), and everything is connected), it isn't done. The
traces are not great, much improvement possible. Also, it's likely that
we'll be swapping the integrated IMU and gyro for just a discrete gyro,
since it was a bitch to work with on the big sensor board.
Parts:
- added C3: 0.1uF, Capacitor_SMD:C_0805_2012Metric_Pad1.15x1.40mm_HandSolder, symbol Device:C
- added C4: 4.7uF, Capacitor_SMD:C_0805_2012Metric_Pad1.15x1.40mm_HandSolder, symbol Device:C
- added F1: Polyfuse, Fuse:Fuse_1206_3216Metric_Pad1.42x1.75mm_HandSolder, symbol Device:Polyfuse
- added R1: ?, Resistor_SMD:R_1206_3216Metric_Pad1.42x1.75mm_HandSolder, symbol Device:R_US
- added TP1, TP2: TestPoint, TestPoint:TestPoint_THTPad_D1.0mm_Drill0.5mm, symbol Connector:TestPoint
- added U3: INA180, Package_TO_SOT_SMD:SOT-23-5_HandSoldering, symbol sensors-rescue:INA180-canhw
- added U5: SPU01M-15, flight_instr:SIP6_Housing, symbol flight_instr:SPU01M-15
Connections:
- net labels added: +12V, +15V, CURR_AMP_12V
- wire segments 32 -> 64
- no-connect marks 1 -> 0
Other:
- moved on the sheet: F2

Commit message: Add magnetometer to schematic and move to SPI
Parts:
- U3, U4: symbol sensors-rescue:INA180-canhw -> sensors-rescue:INA180-canhw-sensors-rescue
- U8: symbol sensors-rescue:MIC5365-1.8-canhw -> sensors-rescue:MIC5365-1.8-canhw-sensors-rescue
Changed lines of the file:
@@
 	3600 4000 3700 4000
 $Comp
-L sensors-rescue:INA180-canhw U?
+L sensors-rescue:INA180-canhw-sensors-rescue U?
 U 1 1 5BB12B37
 P 4350 5000
@@
 	9200 5350 9600 5350
 $Comp
-L sensors-rescue:MIC5365-1.8-canhw U8
+L sensors-rescue:MIC5365-1.8-canhw-sensors-rescue U8
 U 1 1 5BD847E8
 P 8400 5350
@@
 	3700 1600 3800 1600
 $Comp
-L sensors-rescue:INA180-canhw U?
+L sensors-rescue:INA180-canhw-sensors-rescue U?
 U 1 1 5C960D34
 P 4450 2600

Commit message: New sensor mini layout + routing
This does not include cosmetic things like silkscreen
Parts:
- removed TP1, TP2, TP3, TP4: TestPoint, TestPoint:TestPoint_THTPad_D1.0mm_Drill0.5mm, symbol Connector:TestPoint
Connections:
- wire segments 64 -> 56
Changed lines of the file:
@@
 	0    1    1    0
 $EndComp
-Wire Wire Line
-	2450 4000 2350 4000
 Connection ~ 3200 4000
 $Comp
@@
 	1    0    0    -1
 $EndComp
-$Comp
-L Connector:TestPoint TP4
-U 1 1 5BDCB8C1
-P 2900 3650
-F 0 "TP4" H 2958 3770 50  0000 L CNN
-F 1 "TestPoint" H 2958 3679 50  0000 L CNN
-F 2 "TestPoint:TestPoint_THTPad_D1.0mm_Drill0.5mm" H 3100 3650 50  0001 C CNN
-F 3 "~" H 3100 3650 50  0001 C CNN
-	1    2900 3650
-	1    0    0    -1
-$EndComp
-Wire Wire Line
-	2900 3650 2900 4000
-Wire Wire Line
-	2750 4000 2900 4000
-Connection ~ 2900 4000
-Wire Wire Line
-	2900 4000 3200 4000
-$Comp
-L Connector:TestPoint TP3
-U 1 1 5BDCD140
-P 2350 3650
-F 0 "TP3" H 2408 3770 50  0000 L CNN
-F 1 "TestPoint" H 2408 3679 50  0000 L CNN
-F 2 "TestPoint:TestPoint_THTPad_D1.0mm_Drill0.5mm" H 2550 3650 50  0001 C CNN
-F 3 "~" H 2550 3650 50  0001 C CNN
-	1    2350 3650
-	1    0    0    -1
-$EndComp
-Wire Wire Line
-	2350 3650 2350 4000
-Connection ~ 2350 4000
-Wire Wire Line
-	2350 4000 1850 4000
 Wire Wire Line
 	4200 1600 4200 1500
@@
 	0    1    1    0
 $EndComp
-$Comp
-L Connector:TestPoint TP2
-U 1 1 5C961755
-P 2900 1200
-F 0 "TP2" H 2958 1320 50  0000 L CNN
-F 1 "TestPoint" H 2958 1229 50  0000 L CNN
-F 2 "TestPoint:TestPoint_THTPad_D1.0mm_Drill0.5mm" H 3100 1200 50  0001 C CNN
-F 3 "~" H 3100 1200 50  0001 C CNN
-	1    2900 1200
-	1    0    0    -1
-$EndComp
-$Comp
-L Connector:TestPoint TP1
-U 1 1 5C9617CF
-P 2350 1200
-F 0 "TP1" H 2408 1320 50  0000 L CNN
-F 1 "TestPoint" H 2408 1229 50  0000 L CNN
-F 2 "TestPoint:TestPoint_THTPad_D1.0mm_Drill0.5mm" H 2550 1200 50  0001 C CNN
-F 3 "~" H 2550 1200 50  0001 C CNN
-	1    2350 1200
-	1    0    0    -1
-$EndComp
 Wire Wire Line
 	1850 3900 2200 3900
 Wire Wire Line
 	2200 3900 2200 1600
-Wire Wire Line
-	2200 1600 2350 1600
-Wire Wire Line
-	2350 1200 2350 1600
-Connection ~ 2350 1600
-Wire Wire Line
-	2350 1600 2450 1600
-Wire Wire Line
-	2750 1600 2900 1600
-Wire Wire Line
-	2900 1600 2900 1200
-Wire Wire Line
-	2900 1600 3300 1600
-Connection ~ 2900 1600
 $Comp
 L power:+12V #PWR01
@@
 Wire Wire Line
 	9350 4450 9350 4500
+Wire Wire Line
+	2200 1600 2450 1600
+Wire Wire Line
+	2750 1600 3300 1600
+Wire Wire Line
+	2750 4000 3200 4000
+Wire Wire Line
+	1850 4000 2450 4000
 $EndSCHEMATC

Commit message: Address Aidan's schematic comments
- Add sense resistor values
- Add comments for IMU functionality
Parts:
- R1, R2: value ? -> 200mR
Changed lines of the file:
@@
 AR Path="/5BB129A7/5BB12B86" Ref="R2"  Part="1"
 F 0 "R2" V 3245 4000 50  0000 C CNN
-F 1 "?" V 3336 4000 50  0000 C CNN
+F 1 "200mR" V 3336 4000 50  0000 C CNN
 F 2 "Resistor_SMD:R_1206_3216Metric_Pad1.42x1.75mm_HandSolder" V 3490 3990 50  0001 C CNN
 F 3 "~" H 3450 4000 50  0001 C CNN
@@
 AR Path="/5BB129A7/5C960D64" Ref="R1"  Part="1"
 F 0 "R1" V 3345 1600 50  0000 C CNN
-F 1 "?" V 3436 1600 50  0000 C CNN
+F 1 "200mR" V 3436 1600 50  0000 C CNN
 F 2 "Resistor_SMD:R_1206_3216Metric_Pad1.42x1.75mm_HandSolder" V 3590 1590 50  0001 C CNN
 F 3 "~" H 3550 1600 50  0001 C CNN

Commit message: Switch minisensor to run off 3v3, not 1v8
We weren't able to program the microcontroller on minisensor when it was
running on 1v8 VDD, so we swapped the voltage regulator for a 3v3
regulator and it all worked fine. The original reason for 1v8 was that
there was a digital sensor we wanted to use that couldn't run on 3 volts
(the ICM-20948). This sensor got removed in the move from macrosensor to
minisensor, so there's no reason not to use 3v3 on minisensor. The three
digital sensors on the latter all work at 3v3, datasheets below:

- https://www.te.com/commerce/DocumentDelivery/DDEController?Action=srchrtrv&DocNm=MS5607-02BA03&DocType=Data+Sheet&DocLang=English
- https://www.st.com/content/ccc/resource/technical/document/datasheet/group0/38/96/79/af/ab/62/42/c3/DM00229854/files/DM00229854.pdf/jcr:content/translations/en.DM00229854.pdf
- https://www.st.com/content/ccc/resource/technical/document/datasheet/74/c4/19/54/62/c5/46/13/DM00177685.pdf/files/DM00177685.pdf/jcr:content/translations/en.DM00177685.pdf
Parts:
- U3, U4: symbol sensors-rescue:INA180-canhw-sensors-rescue -> sensors-rescue:INA180-canhw-sensors-rescue-sensors-rescue
- U8: value MIC5365-1.8 -> MIC5365-3.3; symbol sensors-rescue:MIC5365-1.8-canhw-sensors-rescue -> sensors-rescue:MIC5365-1.8-canhw-sensors-rescue-sensors-rescue
Connections:
- net labels added: +3V3
- net labels removed: +1V8
Changed lines of the file:
@@
 EESchema Schematic File Version 4
-LIBS:sensors-cache
-EELAYER 26 0
+EELAYER 30 0
 EELAYER END
 $Descr A4 11693 8268
@@
 	3600 4000 3700 4000
 $Comp
-L sensors-rescue:INA180-canhw-sensors-rescue U?
+L sensors-rescue:INA180-canhw-sensors-rescue-sensors-rescue U?
 U 1 1 5BB12B37
 P 4350 5000
 AR Path="/5BB11D6C/5BB12B37" Ref="U?"  Part="1"
 AR Path="/5BB129A7/5BB12B37" Ref="U4"  Part="1"
+AR Path="/5BB12B37" Ref="U4"  Part="1"
 F 0 "U4" H 4300 4528 50  0000 C CNN
 F 1 "INA180" H 4300 4437 50  0000 C CNN
@@
 	9200 5350 9600 5350
 $Comp
-L sensors-rescue:MIC5365-1.8-canhw-sensors-rescue U8
+L sensors-rescue:MIC5365-1.8-canhw-sensors-rescue-sensors-rescue U8
 U 1 1 5BD847E8
 P 8400 5350
 F 0 "U8" H 8375 5575 50  0000 C CNN
-F 1 "MIC5365-1.8" H 8375 5484 50  0000 C CNN
+F 1 "MIC5365-3.3" H 8375 5484 50  0000 C CNN
 F 2 "Package_TO_SOT_SMD:SOT-23-5_HandSoldering" H 8450 5350 50  0001 C CNN
 F 3 "" H 8450 5350 50  0001 C CNN
@@
 	1    0    0    -1
 $EndComp
-$Comp
-L power:+1V8 #PWR043
-U 1 1 5BD849F7
-P 9600 5250
-F 0 "#PWR043" H 9600 5100 50  0001 C CNN
-F 1 "+1V8" H 9615 5423 50  0000 C CNN
-F 2 "" H 9600 5250 50  0001 C CNN
-F 3 "" H 9600 5250 50  0001 C CNN
-	1    9600 5250
-	1    0    0    -1
-$EndComp
 Wire Wire Line
 	4200 1600 4200 1500
@@
 	3700 1600 3800 1600
 $Comp
-L sensors-rescue:INA180-canhw-sensors-rescue U?
+L sensors-rescue:INA180-canhw-sensors-rescue-sensors-rescue U?
 U 1 1 5C960D34
 P 4450 2600
 AR Path="/5BB11D6C/5C960D34" Ref="U?"  Part="1"
 AR Path="/5BB129A7/5C960D34" Ref="U3"  Part="1"
+AR Path="/5C960D34" Ref="U3"  Part="1"
 F 0 "U3" H 4400 2128 50  0000 C CNN
 F 1 "INA180" H 4400 2037 50  0000 C CNN
@@
 Wire Wire Line
 	1850 4000 2450 4000
+$Comp
+L power:+3V3 #PWR?
+U 1 1 5EAC76AF
+P 9600 5250
+F 0 "#PWR?" H 9600 5100 50  0001 C CNN
+F 1 "+3V3" H 9615 5423 50  0000 C CNN
+F 2 "" H 9600 5250 50  0001 C CNN
+F 3 "" H 9600 5250 50  0001 C CNN
+	1    9600 5250
+	1    0    0    -1
+$EndComp
 $EndSCHEMATC

Commit message: Updated MiniSensor PCB
Added testpoints for SCL, SDA, INT_IMU, INT_MAG, THERM_0 and TANK_PREASURE Lines
Switched IMU to MPU-6050
Changed most of the 6 mil tracks on previous design to 8 tracks
Parts:
- J1: symbol Connector:Conn_01x05_Female -> sensors-rescue:Conn_01x05_Female-Connector
- U1: renamed from U4; symbol sensors-rescue:INA180-canhw-sensors-rescue-sensors-rescue -> sensors-rescue:INA180-canhw-sensors-rescue-sensors-rescue-sensors-rescue
- U2: renamed from U3; symbol sensors-rescue:INA180-canhw-sensors-rescue-sensors-rescue -> sensors-rescue:INA180-canhw-sensors-rescue-sensors-rescue-sensors-rescue
- U4: renamed from U8; symbol sensors-rescue:MIC5365-1.8-canhw-sensors-rescue-sensors-rescue -> sensors-rescue:MIC5365-1.8-canhw-sensors-rescue-sensors-rescue-sensors-rescue
- renumbered C6 to C1, C3 to C2, C15 to C3, C16 to C4, C4 to C5, R2 to R1, R1 to R2, U5 to U3
Changed lines of the file:
@@
 P 2250 4500
 AR Path="/5BB11D6C/5BB12B29" Ref="#PWR?"  Part="1"
-AR Path="/5BB129A7/5BB12B29" Ref="#PWR018"  Part="1"
-F 0 "#PWR018" H 2250 4250 50  0001 C CNN
+AR Path="/5BB129A7/5BB12B29" Ref="#PWR01"  Part="1"
+F 0 "#PWR01" H 2250 4250 50  0001 C CNN
 F 1 "GND" H 2255 4327 50  0000 C CNN
 F 2 "" H 2250 4500 50  0001 C CNN
@@
 	3600 4000 3700 4000
 $Comp
-L sensors-rescue:INA180-canhw-sensors-rescue-sensors-rescue U?
+L sensors-rescue:INA180-canhw-sensors-rescue-sensors-rescue-sensors-rescue U?
 U 1 1 5BB12B37
 P 4350 5000
 AR Path="/5BB11D6C/5BB12B37" Ref="U?"  Part="1"
-AR Path="/5BB129A7/5BB12B37" Ref="U4"  Part="1"
-AR Path="/5BB12B37" Ref="U4"  Part="1"
-F 0 "U4" H 4300 4528 50  0000 C CNN
+AR Path="/5BB129A7/5BB12B37" Ref="U1"  Part="1"
+AR Path="/5BB12B37" Ref="U?"  Part="1"
+F 0 "U1" H 4300 4528 50  0000 C CNN
 F 1 "INA180" H 4300 4437 50  0000 C CNN
 F 2 "Package_TO_SOT_SMD:SOT-23-5_HandSoldering" H 4350 5000 50  0001 C CNN
@@
 P 4200 4350
 AR Path="/5BB11D6C/5BB12B3E" Ref="#PWR?"  Part="1"
-AR Path="/5BB129A7/5BB12B3E" Ref="#PWR017"  Part="1"
-F 0 "#PWR017" H 4200 4200 50  0001 C CNN
+AR Path="/5BB129A7/5BB12B3E" Ref="#PWR06"  Part="1"
+F 0 "#PWR06" H 4200 4200 50  0001 C CNN
 F 1 "+5V" H 4215 4523 50  0000 C CNN
 F 2 "" H 4200 4350 50  0001 C CNN
@@
 P 3850 5200
 AR Path="/5BB11D6C/5BB12B44" Ref="#PWR?"  Part="1"
-AR Path="/5BB129A7/5BB12B44" Ref="#PWR020"  Part="1"
-F 0 "#PWR020" H 3850 4950 50  0001 C CNN
+AR Path="/5BB129A7/5BB12B44" Ref="#PWR02"  Part="1"
+F 0 "#PWR02" H 3850 4950 50  0001 C CNN
 F 1 "GND" H 3855 5027 50  0000 C CNN
 F 2 "" H 3850 5200 50  0001 C CNN
@@
 P 4500 4500
 AR Path="/5BB11D6C/5BB12B55" Ref="C?"  Part="1"
-AR Path="/5BB129A7/5BB12B55" Ref="C6"  Part="1"
-F 0 "C6" V 4248 4500 50  0000 C CNN
+AR Path="/5BB129A7/5BB12B55" Ref="C1"  Part="1"
+F 0 "C1" V 4248 4500 50  0000 C CNN
 F 1 "0.1uF" V 4339 4500 50  0000 C CNN
 F 2 "Capacitor_SMD:C_0805_2012Metric_Pad1.15x1.40mm_HandSolder" H 4538 4350 50  0001 C CNN
@@
 P 4750 4550
 AR Path="/5BB11D6C/5BB12B5C" Ref="#PWR?"  Part="1"
-AR Path="/5BB129A7/5BB12B5C" Ref="#PWR019"  Part="1"
-F 0 "#PWR019" H 4750 4300 50  0001 C CNN
+AR Path="/5BB129A7/5BB12B5C" Ref="#PWR08"  Part="1"
+F 0 "#PWR08" H 4750 4300 50  0001 C CNN
 F 1 "GND" H 4755 4377 50  0000 C CNN
 F 2 "" H 4750 4550 50  0001 C CNN
@@
 	4200 4500 4200 4550
 $Comp
-L Connector:Conn_01x05_Female J?
+L sensors-rescue:Conn_01x05_Female-Connector J?
 U 1 1 5BB12B67
 P 1650 4100
@@
 P 4100 3900
 AR Path="/5BB11D6C/5BB12B6E" Ref="#PWR?"  Part="1"
-AR Path="/5BB129A7/5BB12B6E" Ref="#PWR012"  Part="1"
-F 0 "#PWR012" H 4100 3750 50  0001 C CNN
+AR Path="/5BB129A7/5BB12B6E" Ref="#PWR04"  Part="1"
+F 0 "#PWR04" H 4100 3750 50  0001 C CNN
 F 1 "+5V" H 4115 4073 50  0000 C CNN
 F 2 "" H 4100 3900 50  0001 C CNN
@@
 P 3450 4000
 AR Path="/5BB11D6C/5BB12B86" Ref="R?"  Part="1"
-AR Path="/5BB129A7/5BB12B86" Ref="R2"  Part="1"
-F 0 "R2" V 3245 4000 50  0000 C CNN
+AR Path="/5BB129A7/5BB12B86" Ref="R1"  Part="1"
+F 0 "R1" V 3245 4000 50  0000 C CNN
 F 1 "200mR" V 3336 4000 50  0000 C CNN
 F 2 "Resistor_SMD:R_1206_3216Metric_Pad1.42x1.75mm_HandSolder" V 3490 3990 50  0001 C CNN
@@
 $EndComp
 $Comp
-L power:GND #PWR044
+L power:GND #PWR014
 U 1 1 5BD83591
 P 8800 5550
-F 0 "#PWR044" H 8800 5300 50  0001 C CNN
+F 0 "#PWR014" H 8800 5300 50  0001 C CNN
 F 1 "GND" H 8805 5377 50  0000 C CNN
 F 2 "" H 8800 5550 50  0001 C CNN
@@
 	9600 5250 9600 5350
 $Comp
-L Device:C C16
+L Device:C C4
 U 1 1 5BD8359E
 P 9200 5500
-F 0 "C16" H 9315 5546 50  0000 L CNN
+F 0 "C4" H 9315 5546 50  0000 L CNN
 F 1 "1uF" H 9315 5455 50  0000 L CNN
 F 2 "Capacitor_SMD:C_0805_2012Metric_Pad1.15x1.40mm_HandSolder" H 9238 5350 50  0001 C CNN
@@
 $EndComp
 $Comp
-L power:GND #PWR047
+L power:GND #PWR017
 U 1 1 5BD835A5
 P 9200 5650
-F 0 "#PWR047" H 9200 5400 50  0001 C CNN
+F 0 "#PWR017" H 9200 5400 50  0001 C CNN
 F 1 "GND" H 9205 5477 50  0000 C CNN
 F 2 "" H 9200 5650 50  0001 C CNN
@@
 $EndComp
 $Comp
-L power:+5V #PWR042
+L power:+5V #PWR010
 U 1 1 5BD835AB
 P 7200 5250
-F 0 "#PWR042" H 7200 5100 50  0001 C CNN
+F 0 "#PWR010" H 7200 5100 50  0001 C CNN
 F 1 "+5V" H 7215 5423 50  0000 C CNN
 F 2 "" H 7200 5250 50  0001 C CNN
@@
 	7850 5350 7950 5350
 $Comp
-L Device:C C15
+L Device:C C3
 U 1 1 5BD835B6
 P 7500 5500
-F 0 "C15" H 7615 5546 50  0000 L CNN
+F 0 "C3" H 7615 5546 50  0000 L CNN
 F 1 "1uF" H 7615 5455 50  0000 L CNN
 F 2 "Capacitor_SMD:C_0805_2012Metric_Pad1.15x1.40mm_HandSolder" H 7538 5350 50  0001 C CNN
@@
 $EndComp
 $Comp
-L power:GND #PWR046
+L power:GND #PWR011
 U 1 1 5BD835BD
 P 7500 5650
-F 0 "#PWR046" H 7500 5400 50  0001 C CNN
+F 0 "#PWR011" H 7500 5400 50  0001 C CNN
 F 1 "GND" H 7505 5477 50  0000 C CNN
 F 2 "" H 7500 5650 50  0001 C CNN
@@
 	9200 5350 9600 5350
 $Comp
-L sensors-rescue:MIC5365-1.8-canhw-sensors-rescue-sensors-rescue U8
+L sensors-rescue:MIC5365-1.8-canhw-sensors-rescue-sensors-rescue-sensors-rescue U4
 U 1 1 5BD847E8
 P 8400 5350
-F 0 "U8" H 8375 5575 50  0000 C CNN
+F 0 "U4" H 8375 5575 50  0000 C CNN
 F 1 "MIC5365-3.3" H 8375 5484 50  0000 C CNN
 F 2 "Package_TO_SOT_SMD:SOT-23-5_HandSoldering" H 8450 5350 50  0001 C CNN
@@
 	3700 1600 3800 1600
 $Comp
-L sensors-rescue:INA180-canhw-sensors-rescue-sensors-rescue U?
+L sensors-rescue:INA180-canhw-sensors-rescue-sensors-rescue-sensors-rescue U?
 U 1 1 5C960D34
 P 4450 2600
 AR Path="/5BB11D6C/5C960D34" Ref="U?"  Part="1"
-AR Path="/5BB129A7/5C960D34" Ref="U3"  Part="1"
-AR Path="/5C960D34" Ref="U3"  Part="1"
-F 0 "U3" H 4400 2128 50  0000 C CNN
+AR Path="/5BB129A7/5C960D34" Ref="U2"  Part="1"
+AR Path="/5C960D34" Ref="U?"  Part="1"
+F 0 "U2" H 4400 2128 50  0000 C CNN
 F 1 "INA180" H 4400 2037 50  0000 C CNN
 F 2 "Package_TO_SOT_SMD:SOT-23-5_HandSoldering" H 4450 2600 50  0001 C CNN
@@
 P 4300 1950
 AR Path="/5BB11D6C/5C960D3B" Ref="#PWR?"  Part="1"
-AR Path="/5BB129A7/5C960D3B" Ref="#PWR02"  Part="1"
-F 0 "#PWR02" H 4300 1800 50  0001 C CNN
+AR Path="/5BB129A7/5C960D3B" Ref="#PWR07"  Part="1"
+F 0 "#PWR07" H 4300 1800 50  0001 C CNN
 F 1 "+5V" H 4315 2123 50  0000 C CNN
 F 2 "" H 4300 1950 50  0001 C CNN
@@
 P 3950 2800
 AR Path="/5BB11D6C/5C960D41" Ref="#PWR?"  Part="1"
-AR Path="/5BB129A7/5C960D41" Ref="#PWR04"  Part="1"
-F 0 "#PWR04" H 3950 2550 50  0001 C CNN
+AR Path="/5BB129A7/5C960D41" Ref="#PWR03"  Part="1"
+F 0 "#PWR03" H 3950 2550 50  0001 C CNN
 F 1 "GND" H 3955 2627 50  0000 C CNN
 F 2 "" H 3950 2800 50  0001 C CNN
@@
 P 4600 2100
 AR Path="/5BB11D6C/5C960D51" Ref="C?"  Part="1"
-AR Path="/5BB129A7/5C960D51" Ref="C3"  Part="1"
-F 0 "C3" V 4348 2100 50  0000 C CNN
+AR Path="/5BB129A7/5C960D51" Ref="C2"  Part="1"
+F 0 "C2" V 4348 2100 50  0000 C CNN
 F 1 "0.1uF" V 4439 2100 50  0000 C CNN
 F 2 "Capacitor_SMD:C_0805_2012Metric_Pad1.15x1.40mm_HandSolder" H 4638 1950 50  0001 C CNN
@@
 P 4850 2150
 AR Path="/5BB11D6C/5C960D58" Ref="#PWR?"  Part="1"
-AR Path="/5BB129A7/5C960D58" Ref="#PWR03"  Part="1"
-F 0 "#PWR03" H 4850 1900 50  0001 C CNN
+AR Path="/5BB129A7/5C960D58" Ref="#PWR09"  Part="1"
+F 0 "#PWR09" H 4850 1900 50  0001 C CNN
 F 1 "GND" H 4855 1977 50  0000 C CNN
 F 2 "" H 4850 2150 50  0001 C CNN
@@
 P 3550 1600
 AR Path="/5BB11D6C/5C960D64" Ref="R?"  Part="1"
-AR Path="/5BB129A7/5C960D64" Ref="R1"  Part="1"
-F 0 "R1" V 3345 1600 50  0000 C CNN
+AR Path="/5BB129A7/5C960D64" Ref="R2"  Part="1"
+F 0 "R2" V 3345 1600 50  0000 C CNN
 F 1 "200mR" V 3436 1600 50  0000 C CNN
 F 2 "Resistor_SMD:R_1206_3216Metric_Pad1.42x1.75mm_HandSolder" V 3590 1590 50  0001 C CNN
@@
 	2200 3900 2200 1600
 $Comp
-L power:+12V #PWR01
+L power:+12V #PWR05
 U 1 1 5C9647FF
 P 4200 1500
-F 0 "#PWR01" H 4200 1350 50  0001 C CNN
+F 0 "#PWR05" H 4200 1350 50  0001 C CNN
 F 1 "+12V" H 4215 1673 50  0000 C CNN
 F 2 "" H 4200 1500 50  0001 C CNN
@@
 $EndComp
 $Comp
-L flight_instr:SPU01M-15 U5
+L flight_instr:SPU01M-15 U3
 U 1 1 5C96497A
 P 8250 4100
-F 0 "U5" H 8325 4387 60  0000 C CNN
+F 0 "U3" H 8325 4387 60  0000 C CNN
 F 1 "SPU01M-15" H 8325 4281 60  0000 C CNN
 F 2 "flight_instr:SIP6_Housing" H 8250 4100 60  0001 C CNN
@@
 $EndComp
 $Comp
-L power:GND #PWR09
+L power:GND #PWR013
 U 1 1 5C964B78
 P 7650 4550
-F 0 "#PWR09" H 7650 4300 50  0001 C CNN
+F 0 "#PWR013" H 7650 4300 50  0001 C CNN
 F 1 "GND" H 7655 4377 50  0000 C CNN
 F 2 "" H 7650 4550 50  0001 C CNN
@@
 $EndComp
 $Comp
-L power:GND #PWR07
+L power:GND #PWR016
 U 1 1 5C964BAC
 P 9050 4500
-F 0 "#PWR07" H 9050 4250 50  0001 C CNN
+F 0 "#PWR016" H 9050 4250 50  0001 C CNN
 F 1 "GND" H 9055 4327 50  0000 C CNN
 F 2 "" H 9050 4500 50  0001 C CNN
@@
 	7650 4300 7800 4300
 $Comp
-L power:+12V #PWR05
+L power:+12V #PWR012
 U 1 1 5C966749
 P 7650 3900
-F 0 "#PWR05" H 7650 3750 50  0001 C CNN
+F 0 "#PWR012" H 7650 3750 50  0001 C CNN
 F 1 "+12V" H 7665 4073 50  0000 C CNN
 F 2 "" H 7650 3900 50  0001 C CNN
@@
 	7650 4100 7650 3900
 $Comp
-L power:+15V #PWR06
+L power:+15V #PWR015
 U 1 1 5C968615
 P 9050 3900
-F 0 "#PWR06" H 9050 3750 50  0001 C CNN
+F 0 "#PWR015" H 9050 3750 50  0001 C CNN
 F 1 "+15V" H 9065 4073 50  0000 C CNN
 F 2 "" H 9050 3900 50  0001 C CNN
@@
 	9050 4100 9050 3900
 $Comp
-L Device:C C4
+L Device:C C5
 U 1 1 5C9695EF
 P 9350 4300
-F 0 "C4" H 9465 4346 50  0000 L CNN
+F 0 "C5" H 9465 4346 50  0000 L CNN
 F 1 "4.7uF" H 9465 4255 50  0000 L CNN
 F 2 "Capacitor_SMD:C_0805_2012Metric_Pad1.15x1.40mm_HandSolder" H 9388 4150 50  0001 C CNN
@@
 Connection ~ 9050 4100
 $Comp
-L power:GND #PWR08
+L power:GND #PWR018
 U 1 1 5C96A6D6
 P 9350 4500
-F 0 "#PWR08" H 9350 4250 50  0001 C CNN
+F 0 "#PWR018" H 9350 4250 50  0001 C CNN
 F 1 "GND" H 9355 4327 50  0000 C CNN
 F 2 "" H 9350 4500 50  0001 C CNN
@@
 	1850 4000 2450 4000
 $Comp
-L power:+3V3 #PWR?
+L power:+3V3 #PWR019
 U 1 1 5EAC76AF
 P 9600 5250
-F 0 "#PWR?" H 9600 5100 50  0001 C CNN
+F 0 "#PWR019" H 9600 5100 50  0001 C CNN
 F 1 "+3V3" H 9615 5423 50  0000 C CNN
 F 2 "" H 9600 5250 50  0001 C CNN
