File: CanardBoard/flash.kicad_sch (KiCad schematic)
At the start: 4 parts, among them U3 GD5F1GM7UEYIGR

Commit message: more schematic
Parts:
- U3: footprint SON127P800X600X80-9N-D -> canardboard:GD5F1GM7UEYIGR
Changed lines of the file:
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@@
 			)
 		)
-		(property "Footprint" "SON127P800X600X80-9N-D"
+		(property "Footprint" "canardboard:GD5F1GM7UEYIGR"
 			(at 213.36 196.52 0)
 			(effects

Commit message: more schematic work
Parts:
- removed U3: GD5F1GM7UEYIGR, canardboard:GD5F1GM7UEYIGR, symbol canardboard:GD5F1GM7UEYIGR
- added U3: MX25L25645GM2I-08G, SOIC127P790X216-8N, symbol canardboard:MX25L25645GM2I-08G
Connections:
- net +3V3: now also U3.8 (VCC)
- net FLASH_CLK: now also U3.6 (SCLK)
- net FLASH_IO0: now also U3.5 (SI/SIO0)
- net FLASH_IO1: now also U3.2 (SO/SIO1)
- net FLASH_IO2: now also U3.3 (WP#/SIO2)
- net FLASH_IO3: now also U3.7 (RESET#/SIO3)
- net FLASH_NCS: now also U3.1 (CS#)
- net GND: now also U3.4 (GND)
- no-connect marks 1 -> 0
Other:
- moved on the sheet: R17

Commit message: mag
Parts:
- U3: footprint SOIC127P790X216-8N -> (none)
Changed lines of the file:
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@@
 			)
 		)
-		(property "Footprint" "SOIC127P790X216-8N"
+		(property "Footprint" ""
 			(at 191.77 191.44 0)
 			(effects

Commit message: AD Breakout interface
Parts:
- U3: footprint (none) -> SOIC127P790X216-8N
Changed lines of the file:
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@@
 			)
 		)
-		(property "Footprint" ""
+		(property "Footprint" "SOIC127P790X216-8N"
 			(at 191.77 191.44 0)
 			(effects

Commit message: work
Parts:
- C7, C8: footprint Capacitor_SMD:C_0805_2012Metric_Pad1.18x1.45mm_HandSolder -> Capacitor_SMD:C_0402_1005Metric
- R17: footprint Resistor_SMD:R_0805_2012Metric_Pad1.20x1.40mm_HandSolder -> Resistor_SMD:R_0402_1005Metric
- U3: footprint SOIC127P790X216-8N -> canardboard:MX25L25645GM2I-08G
Changed lines of the file:
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@@
 			)
 		)
-		(property "Footprint" "SOIC127P790X216-8N"
+		(property "Footprint" "canardboard:MX25L25645GM2I-08G"
 			(at 191.77 191.44 0)
 			(effects
@@
 			)
 		)
-		(property "Footprint" "Capacitor_SMD:C_0805_2012Metric_Pad1.18x1.45mm_HandSolder"
+		(property "Footprint" "Capacitor_SMD:C_0402_1005Metric"
 			(at 92.71 99.06 0)
 			(effects
@@
 			)
 		)
-		(property "Footprint" "Capacitor_SMD:C_0805_2012Metric_Pad1.18x1.45mm_HandSolder"
+		(property "Footprint" "Capacitor_SMD:C_0402_1005Metric"
 			(at 104.14 99.06 0)
 			(effects
@@
 			)
 		)
-		(property "Footprint" "Resistor_SMD:R_0805_2012Metric_Pad1.20x1.40mm_HandSolder"
+		(property "Footprint" "Resistor_SMD:R_0402_1005Metric"
 			(at 139.7 93.98 0)
 			(effects

Commit message: done
Parts:
- C45: renamed from C8; symbol Device_Custom:C_Small -> Device:C_Small
- C46: renamed from C7; symbol Device_Custom:C_Small -> Device:C_Small
- R37: renamed from R17; value 10kΩ -> 10k; symbol Device_Custom:R_Small_US -> Device:R_Small_US
- renumbered U3 to U10
Changed lines of the file:
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@@
 		(dnp no)
 		(fields_autoplaced yes)
-		(property "Reference" "#PWR050"
+		(property "Reference" "#PWR098"
 			(at 104.14 95.25 0)
 			(effects
@@
 			(project "CanardBoard"
 				(path "/605ab838-6b02-4cf5-a6b5-94a0cdb1b998/3bf63de2-f072-4034-9f3c-b5559a05babe"
-					(reference "#PWR050")
+					(reference "#PWR098")
 					(unit 1)
 				)
@@
 		(dnp no)
 		(fields_autoplaced yes)
-		(property "Reference" "U3"
+		(property "Reference" "U10"
 			(at 170.18 88.9 0)
 			(effects
@@
 			(project ""
 				(path "/605ab838-6b02-4cf5-a6b5-94a0cdb1b998/3bf63de2-f072-4034-9f3c-b5559a05babe"
-					(reference "U3")
+					(reference "U10")
 					(unit 1)
 				)
@@
 		(dnp no)
 		(fields_autoplaced yes)
-		(property "Reference" "#PWR047"
+		(property "Reference" "#PWR099"
 			(at 104.14 114.3 0)
 			(effects
@@
 			(project "CanardBoard"
 				(path "/605ab838-6b02-4cf5-a6b5-94a0cdb1b998/3bf63de2-f072-4034-9f3c-b5559a05babe"
-					(reference "#PWR047")
+					(reference "#PWR099")
 					(unit 1)
 				)
@@
 	)
 	(symbol
-		(lib_id "Device_Custom:C_Small")
+		(lib_id "Device:C_Small")
 		(at 92.71 99.06 0)
 		(mirror y)
@@
 		(dnp no)
 		(fields_autoplaced yes)
-		(property "Reference" "C8"
+		(property "Reference" "C45"
 			(at 95.25 97.7962 0)
 			(effects
@@
 			(project "CanardBoard"
 				(path "/605ab838-6b02-4cf5-a6b5-94a0cdb1b998/3bf63de2-f072-4034-9f3c-b5559a05babe"
-					(reference "C8")
+					(reference "C45")
 					(unit 1)
 				)
@@
 	)
 	(symbol
-		(lib_id "Device_Custom:C_Small")
+		(lib_id "Device:C_Small")
 		(at 104.14 99.06 0)
 		(mirror y)
@@
 		(dnp no)
 		(fields_autoplaced yes)
-		(property "Reference" "C7"
+		(property "Reference" "C46"
 			(at 106.68 97.7962 0)
 			(effects
@@
 			(project "CanardBoard"
 				(path "/605ab838-6b02-4cf5-a6b5-94a0cdb1b998/3bf63de2-f072-4034-9f3c-b5559a05babe"
-					(reference "C7")
+					(reference "C46")
 					(unit 1)
 				)
@@
 	)
 	(symbol
-		(lib_id "Device_Custom:R_Small_US")
+		(lib_id "Device:R_Small_US")
 		(at 139.7 93.98 0)
 		(unit 1)
@@
 		(on_board yes)
 		(dnp no)
-		(property "Reference" "R17"
+		(property "Reference" "R37"
 			(at 137.16 93.98 90)
 			(effects
@@
 			)
 		)
-		(property "Value" "10kΩ"
+		(property "Value" "10k"
 			(at 142.24 93.98 90)
 			(effects
@@
 			(project "CanardBoard"
 				(path "/605ab838-6b02-4cf5-a6b5-94a0cdb1b998/3bf63de2-f072-4034-9f3c-b5559a05babe"
-					(reference "R17")
+					(reference "R37")
 					(unit 1)
 				)
@@
 		(dnp no)
 		(fields_autoplaced yes)
-		(property "Reference" "#PWR0102"
+		(property "Reference" "#PWR0100"
 			(at 148.59 92.71 0)
 			(effects
@@
 			(project "CanardBoard"
 				(path "/605ab838-6b02-4cf5-a6b5-94a0cdb1b998/3bf63de2-f072-4034-9f3c-b5559a05babe"
-					(reference "#PWR0102")
-					(unit 1)
-				)
+					(reference "#PWR0100")
+					(unit 1)
+				)

Commit message: changes
Parts:
- renumbered R37 to R36
Changed lines of the file:
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@@
 		(dnp no)
 		(fields_autoplaced yes)
-		(property "Reference" "#PWR098"
+		(property "Reference" "#PWR099"
 			(at 104.14 95.25 0)
 			(effects
@@
 			(project "CanardBoard"
 				(path "/605ab838-6b02-4cf5-a6b5-94a0cdb1b998/3bf63de2-f072-4034-9f3c-b5559a05babe"
-					(reference "#PWR098")
+					(reference "#PWR099")
 					(unit 1)
 				)
@@
 		(dnp no)
 		(fields_autoplaced yes)
-		(property "Reference" "#PWR099"
+		(property "Reference" "#PWR0100"
 			(at 104.14 114.3 0)
 			(effects
@@
 			(project "CanardBoard"
 				(path "/605ab838-6b02-4cf5-a6b5-94a0cdb1b998/3bf63de2-f072-4034-9f3c-b5559a05babe"
-					(reference "#PWR099")
+					(reference "#PWR0100")
 					(unit 1)
 				)
@@
 		(dnp no)
 		(fields_autoplaced yes)
-		(property "Reference" "#PWR0101"
+		(property "Reference" "#PWR0102"
 			(at 148.59 118.11 0)
 			(effects
@@
 			(project "CanardBoard"
 				(path "/605ab838-6b02-4cf5-a6b5-94a0cdb1b998/3bf63de2-f072-4034-9f3c-b5559a05babe"
-					(reference "#PWR0101")
+					(reference "#PWR0102")
 					(unit 1)
 				)
@@
 		(on_board yes)
 		(dnp no)
-		(property "Reference" "R37"
+		(property "Reference" "R36"
 			(at 137.16 93.98 90)
 			(effects
@@
 			(project "CanardBoard"
 				(path "/605ab838-6b02-4cf5-a6b5-94a0cdb1b998/3bf63de2-f072-4034-9f3c-b5559a05babe"
-					(reference "R37")
+					(reference "R36")
 					(unit 1)
 				)
@@
 		(dnp no)
 		(fields_autoplaced yes)
-		(property "Reference" "#PWR0100"
+		(property "Reference" "#PWR0101"
 			(at 148.59 92.71 0)
 			(effects
@@
 			(project "CanardBoard"
 				(path "/605ab838-6b02-4cf5-a6b5-94a0cdb1b998/3bf63de2-f072-4034-9f3c-b5559a05babe"
-					(reference "#PWR0100")
-					(unit 1)
-				)
+					(reference "#PWR0101")
+					(unit 1)
+				)

Commit message: some changes
Parts:
- added R52, R67: 10k, Resistor_SMD:R_0402_1005Metric, symbol Device:R_Small_US
Connections:
- net +3V3: now also R52.1, R67.1
- net FLASH_IO2: now also R52.2
- net FLASH_IO3: now also R67.2
