File: CanardBoard/SD_Card.kicad_sch (KiCad schematic)
At the start: 9 parts, among them J1 Conn_ST_STDC14, J2 Micro_SD_Card, J4 USB_C_Receptacle_USB2.0_16P

Commit message: schematic work
Parts:
- removed J1: Conn_ST_STDC14, Connector_PinHeader_1.27mm:PinHeader_2x07_P1.27mm_Vertical, symbol Connector:Conn_ST_STDC14
- removed J4: USB_C_Receptacle_USB2.0_16P, Connector_USB:USB_C_Receptacle_GCT_USB4105-xx-A_16P_TopMnt_Horizontal, symbol Connector:USB_C_Receptacle_USB2.0_16P
- added C4: 4.7uF, Capacitor_SMD:C_0805_2012Metric_Pad1.18x1.45mm_HandSolder, symbol Device_Custom:C_Small
- added U1: EMIF06-HSD03F3, EMIF06HSD03F3, symbol canhw:EMIF06-HSD03F3
Connections:
- net +3V3: now also C4.1, U1.B2 (VCC)
- net GND: now also C4.2, U1.D2 (GND_1), U1.F2 (GND_2), U1.H2 (GND_3)
- net SD_CLK: now also R3.2, U1.G1 (O4); no longer J2.5 (CLK), R4.2
- net SD_CMD: now also R4.2, U1.E1 (O3); no longer J2.3 (CMD), R3.2
- net SD_D0: now also R2.2, U1.I1 (O5); no longer J2.7 (DAT0), R5.2
- net SD_D1: now also R1.2, U1.K1 (O6); no longer J2.8 (DAT1), R6.2
- net SD_D2: now also R6.2, U1.A1 (O1); no longer J2.1 (DAT2), R1.2
- net SD_D3: now also R5.2, U1.C1 (O2); no longer J2.2 (DAT3/CD), R2.2
- new net: J2.1 (DAT2), U1.A3 (I1)
- new net: J2.2 (DAT3/CD), U1.C3 (I2)
- new net: J2.3 (CMD), U1.E3 (I3)
- new net: J2.5 (CLK), U1.G3 (I4)
- new net: J2.7 (DAT0), U1.I3 (I5)
- new net: J2.8 (DAT1), U1.K3 (I6)
- no-connect marks 4 -> 1
Other:
- note added: "EMI Filtering and TVS Protection"
- note removed: "Debug header"
- moved on the sheet: J2, R1, R2, R3, R4, R5, R6

Commit message: make project symbols and footprints
Parts:
- U1: symbol canhw:EMIF06-HSD03F3 -> canardboard:EMIF06-HSD03F3
Changed lines of the file:
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@@
 	)
 	(symbol
-		(lib_id "canhw:EMIF06-HSD03F3")
+		(lib_id "canardboard:EMIF06-HSD03F3")
 		(at 165.1 87.63 0)
 		(unit 1)

Commit message: work
Parts:
- C4: footprint Capacitor_SMD:C_0805_2012Metric_Pad1.18x1.45mm_HandSolder -> Capacitor_SMD:C_0402_1005Metric
- R1, R2, R3, R4, R5, R6: footprint Resistor_SMD:R_0201_0603Metric -> Resistor_SMD:R_0402_1005Metric
- U1: footprint EMIF06HSD03F3 -> canardboard:EMIF06HSD03F3
Changed lines of the file:
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@@
 			)
 		)
-		(property "Footprint" "Capacitor_SMD:C_0805_2012Metric_Pad1.18x1.45mm_HandSolder"
+		(property "Footprint" "Capacitor_SMD:C_0402_1005Metric"
 			(at 52.07 88.9 0)
 			(effects
@@
 			)
 		)
-		(property "Footprint" "Resistor_SMD:R_0201_0603Metric"
+		(property "Footprint" "Resistor_SMD:R_0402_1005Metric"
 			(at 92.71 80.01 0)
 			(effects
@@
 			)
 		)
-		(property "Footprint" "Resistor_SMD:R_0201_0603Metric"
+		(property "Footprint" "Resistor_SMD:R_0402_1005Metric"
 			(at 139.7 80.01 0)
 			(effects
@@
 			)
 		)
-		(property "Footprint" "Resistor_SMD:R_0201_0603Metric"
+		(property "Footprint" "Resistor_SMD:R_0402_1005Metric"
 			(at 128.27 80.01 0)
 			(effects
@@
 			)
 		)
-		(property "Footprint" "EMIF06HSD03F3"
+		(property "Footprint" "canardboard:EMIF06HSD03F3"
 			(at 191.77 182.55 0)
 			(effects
@@
 			)
 		)
-		(property "Footprint" "Resistor_SMD:R_0201_0603Metric"
+		(property "Footprint" "Resistor_SMD:R_0402_1005Metric"
 			(at 104.14 80.01 0)
 			(effects
@@
 			)
 		)
-		(property "Footprint" "Resistor_SMD:R_0201_0603Metric"
+		(property "Footprint" "Resistor_SMD:R_0402_1005Metric"
 			(at 151.13 80.01 0)
 			(effects
@@
 			)
 		)
-		(property "Footprint" "Resistor_SMD:R_0201_0603Metric"
+		(property "Footprint" "Resistor_SMD:R_0402_1005Metric"
 			(at 116.84 80.01 0)
 			(effects

Commit message: done
Parts:
- C17: renamed from C4; symbol Device_Custom:C_Small -> Device:C_Small
- R10: renamed from R3; value 10kR -> 10k; symbol Device:R_Small -> Device:R_Small_US
- R11: renamed from R4; value 10kR -> 10k; symbol Device:R_Small -> Device:R_Small_US
- R12: renamed from R5; value 10kR -> 10k; symbol Device:R_Small -> Device:R_Small_US
- R13: renamed from R6; value 10kR -> 10k; symbol Device:R_Small -> Device:R_Small_US
- R8: renamed from R1; value 10kR -> 10k; symbol Device:R_Small -> Device:R_Small_US
- R9: renamed from R2; value 10kR -> 10k; symbol Device:R_Small -> Device:R_Small_US
- renumbered U1 to U3
Changed lines of the file:
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@@
 	)
 	(symbol
-		(lib_id "Device_Custom:C_Small")
+		(lib_id "Device:C_Small")
 		(at 52.07 88.9 0)
 		(mirror y)
@@
 		(dnp no)
 		(fields_autoplaced yes)
-		(property "Reference" "C4"
+		(property "Reference" "C17"
 			(at 54.61 87.6362 0)
 			(effects
@@
 			(project "CanardBoard"
 				(path "/605ab838-6b02-4cf5-a6b5-94a0cdb1b998/78243af2-5eea-48f5-811a-91865538cf4e"
-					(reference "C4")
-					(unit 1)
-				)
-			)
-		)
-	)
-	(symbol
-		(lib_id "Device:R_Small")
+					(reference "C17")
+					(unit 1)
+				)
+			)
+		)
+	)
+	(symbol
+		(lib_id "Device:R_Small_US")
 		(at 92.71 80.01 0)
 		(unit 1)
@@
 		(on_board yes)
 		(dnp no)
-		(property "Reference" "R1"
+		(property "Reference" "R8"
 			(at 93.98 78.74 0)
 			(effects
@@
 			)
 		)
-		(property "Value" "10kR"
+		(property "Value" "10k"
 			(at 93.98 81.28 0)
 			(effects
@@
 			)
 		)
-		(property "Description" "Resistor, small symbol"
+		(property "Description" "Resistor, small US symbol"
 			(at 92.71 80.01 0)
 			(effects
@@
 			(project "CanardBoard"
 				(path "/605ab838-6b02-4cf5-a6b5-94a0cdb1b998/78243af2-5eea-48f5-811a-91865538cf4e"
-					(reference "R1")
-					(unit 1)
-				)
-			)
-		)
-	)
-	(symbol
-		(lib_id "Device:R_Small")
+					(reference "R8")
+					(unit 1)
+				)
+			)
+		)
+	)
+	(symbol
+		(lib_id "Device:R_Small_US")
 		(at 139.7 80.01 0)
 		(unit 1)
@@
 		(on_board yes)
 		(dnp no)
-		(property "Reference" "R5"
+		(property "Reference" "R12"
 			(at 140.97 78.74 0)
 			(effects
@@
 			)
 		)
-		(property "Value" "10kR"
+		(property "Value" "10k"
 			(at 140.97 81.28 0)
 			(effects
@@
 			)
 		)
-		(property "Description" "Resistor, small symbol"
+		(property "Description" "Resistor, small US symbol"
 			(at 139.7 80.01 0)
 			(effects
@@
 			(project "CanardBoard"
 				(path "/605ab838-6b02-4cf5-a6b5-94a0cdb1b998/78243af2-5eea-48f5-811a-91865538cf4e"
-					(reference "R5")
+					(reference "R12")
 					(unit 1)
 				)
@@
 		(dnp no)
 		(fields_autoplaced yes)
-		(property "Reference" "#PWR04"
+		(property "Reference" "#PWR028"
 			(at 52.07 71.12 0)
 			(effects
@@
 			(project "CanardBoard"
 				(path "/605ab838-6b02-4cf5-a6b5-94a0cdb1b998/78243af2-5eea-48f5-811a-91865538cf4e"
-					(reference "#PWR04")
+					(reference "#PWR028")
 					(unit 1)
 				)
@@
 		(dnp no)
 		(fields_autoplaced yes)
-		(property "Reference" "#PWR07"
+		(property "Reference" "#PWR032"
 			(at 162.56 123.19 0)
 			(effects
@@
 			(project "CanardBoard"
 				(path "/605ab838-6b02-4cf5-a6b5-94a0cdb1b998/78243af2-5eea-48f5-811a-91865538cf4e"
-					(reference "#PWR07")
-					(unit 1)
-				)
-			)
-		)
-	)
-	(symbol
-		(lib_id "Device:R_Small")
+					(reference "#PWR032")
+					(unit 1)
+				)
+			)
+		)
+	)
+	(symbol
+		(lib_id "Device:R_Small_US")
 		(at 128.27 80.01 0)
 		(unit 1)
@@
 		(on_board yes)
 		(dnp no)
-		(property "Reference" "R4"
+		(property "Reference" "R11"
 			(at 129.54 78.74 0)
 			(effects
@@
 			)
 		)
-		(property "Value" "10kR"
+		(property "Value" "10k"
 			(at 129.54 81.28 0)
 			(effects
@@
 			)
 		)
-		(property "Description" "Resistor, small symbol"
+		(property "Description" "Resistor, small US symbol"
 			(at 128.27 80.01 0)
 			(effects
@@
 			(project "CanardBoard"
 				(path "/605ab838-6b02-4cf5-a6b5-94a0cdb1b998/78243af2-5eea-48f5-811a-91865538cf4e"
-					(reference "R4")
+					(reference "R11")
 					(unit 1)
 				)
@@
 		(dnp no)
 		(fields_autoplaced yes)
-		(property "Reference" "#PWR013"
+		(property "Reference" "#PWR036"
 			(at 256.54 121.92 0)
 			(effects
@@
 			(project "CanardBoard"
 				(path "/605ab838-6b02-4cf5-a6b5-94a0cdb1b998/78243af2-5eea-48f5-811a-91865538cf4e"
-					(reference "#PWR013")
+					(reference "#PWR036")
 					(unit 1)
 				)
@@
 		(dnp no)
 		(fields_autoplaced yes)
-		(property "Reference" "#PWR015"
+		(property "Reference" "#PWR034"
 			(at 209.55 82.55 0)
 			(effects
@@
 			(project "CanardBoard"
 				(path "/605ab838-6b02-4cf5-a6b5-94a0cdb1b998/78243af2-5eea-48f5-811a-91865538cf4e"
-					(reference "#PWR015")
+					(reference "#PWR034")
 					(unit 1)
 				)
@@
 		(dnp no)
 		(fields_autoplaced yes)
-		(property "Reference" "U1"
+		(property "Reference" "U3"
 			(at 180.34 80.01 0)
 			(effects
@@
 			(project ""
 				(path "/605ab838-6b02-4cf5-a6b5-94a0cdb1b998/78243af2-5eea-48f5-811a-91865538cf4e"
-					(reference "U1")
-					(unit 1)
-				)
-			)
-		)
-	)
-	(symbol
-		(lib_id "Device:R_Small")
+					(reference "U3")
+					(unit 1)
+				)
+			)
+		)
+	)
+	(symbol
+		(lib_id "Device:R_Small_US")
 		(at 104.14 80.01 0)
 		(unit 1)
@@
 		(on_board yes)
 		(dnp no)
-		(property "Reference" "R2"
+		(property "Reference" "R9"
 			(at 105.41 78.74 0)
 			(effects
@@
 			)
 		)
-		(property "Value" "10kR"
+		(property "Value" "10k"
 			(at 105.41 81.28 0)
 			(effects
@@
 			)
 		)
-		(property "Description" "Resistor, small symbol"
+		(property "Description" "Resistor, small US symbol"
 			(at 104.14 80.01 0)
 			(effects
@@
 			(project "CanardBoard"
 				(path "/605ab838-6b02-4cf5-a6b5-94a0cdb1b998/78243af2-5eea-48f5-811a-91865538cf4e"
-					(reference "R2")
-					(unit 1)
-				)
-			)
-		)
-	)
-	(symbol
-		(lib_id "Device:R_Small")
+					(reference "R9")
+					(unit 1)
+				)
+			)
+		)
+	)
+	(symbol
+		(lib_id "Device:R_Small_US")
 		(at 151.13 80.01 0)
 		(unit 1)
@@
 		(on_board yes)
 		(dnp no)
-		(property "Reference" "R6"
+		(property "Reference" "R13"
 			(at 152.4 78.74 0)
 			(effects
@@
 			)
 		)
-		(property "Value" "10kR"
+		(property "Value" "10k"
 			(at 152.4 81.28 0)
 			(effects
@@
 			)
 		)
-		(property "Description" "Resistor, small symbol"
+		(property "Description" "Resistor, small US symbol"
 			(at 151.13 80.01 0)
 			(effects
@@
 			(project "CanardBoard"
 				(path "/605ab838-6b02-4cf5-a6b5-94a0cdb1b998/78243af2-5eea-48f5-811a-91865538cf4e"
-					(reference "R6")
+					(reference "R13")
 					(unit 1)
 				)
@@
 		(dnp no)
 		(fields_autoplaced yes)
-		(property "Reference" "#PWR017"
+		(property "Reference" "#PWR030"
 			(at 92.71 72.39 0)
 			(effects
@@
 			(project "CanardBoard"
 				(path "/605ab838-6b02-4cf5-a6b5-94a0cdb1b998/78243af2-5eea-48f5-811a-91865538cf4e"
-					(reference "#PWR017")
-					(unit 1)
-				)
-			)
-		)
-	)
-	(symbol
-		(lib_id "Device:R_Small")
+					(reference "#PWR030")
+					(unit 1)
+				)
+			)
+		)
+	)
+	(symbol
+		(lib_id "Device:R_Small_US")
 		(at 116.84 80.01 0)
 		(unit 1)
@@
 		(on_board yes)
 		(dnp no)
-		(property "Reference" "R3"
+		(property "Reference" "R10"
 			(at 118.11 78.74 0)
 			(effects
@@
 			)
 		)
-		(property "Value" "10kR"
+		(property "Value" "10k"
 			(at 118.11 81.28 0)
 			(effects
@@
 			)
 		)
-		(property "Description" "Resistor, small symbol"
+		(property "Description" "Resistor, small US symbol"
 			(at 116.84 80.01 0)
 			(effects
@@
 			(project "CanardBoard"
 				(path "/605ab838-6b02-4cf5-a6b5-94a0cdb1b998/78243af2-5eea-48f5-811a-91865538cf4e"
-					(reference "R3")
+					(reference "R10")
 					(unit 1)
 				)
@@
 		(dnp no)
 		(fields_autoplaced yes)
-		(property "Reference" "#PWR05"
+		(property "Reference" "#PWR033"
 			(at 198.12 123.19 0)
 			(effects
@@
 			(project "CanardBoard"
 				(path "/605ab838-6b02-4cf5-a6b5-94a0cdb1b998/78243af2-5eea-48f5-811a-91865538cf4e"
-					(reference "#PWR05")
+					(reference "#PWR033")
 					(unit 1)
 				)
@@
 		(dnp no)
 		(fields_autoplaced yes)
-		(property "Reference" "#PWR014"
+		(property "Reference" "#PWR035"
 			(at 209.55 123.19 0)
 			(effects
@@
 			(project "CanardBoard"
 				(path "/605ab838-6b02-4cf5-a6b5-94a0cdb1b998/78243af2-5eea-48f5-811a-91865538cf4e"
-					(reference "#PWR014")
+					(reference "#PWR035")
 					(unit 1)
 				)
@@
 		(dnp no)
 		(fields_autoplaced yes)
-		(property "Reference" "#PWR06"
+		(property "Reference" "#PWR031"
 			(at 162.56 83.82 0)
 			(effects
@@
 			(project "CanardBoard"
 				(path "/605ab838-6b02-4cf5-a6b5-94a0cdb1b998/78243af2-5eea-48f5-811a-91865538cf4e"
-					(reference "#PWR06")
+					(reference "#PWR031")
 					(unit 1)
 				)
@@
 		(dnp no)
 		(fields_autoplaced yes)
-		(property "Reference" "#PWR03"
+		(property "Reference" "#PWR029"
 			(at 52.07 111.76 0)
 			(effects
@@
 			(project "CanardBoard"
 				(path "/605ab838-6b02-4cf5-a6b5-94a0cdb1b998/78243af2-5eea-48f5-811a-91865538cf4e"
-					(reference "#PWR03")
-					(unit 1)
-				)
+					(reference "#PWR029")
+					(unit 1)
+				)

Commit message: changes
Parts:
- removed R10: 10k, Resistor_SMD:R_0402_1005Metric, symbol Device:R_Small_US
- renumbered R11 to R10, R12 to R11, R13 to R12
Changed lines of the file:
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@@
-	)
-	(junction
-		(at 116.84 97.79)
-		(diameter 0)
-		(color 0 0 0 0)
 	)
 	(junction
@@
 	)
 	(junction
-		(at 116.84 71.12)
-		(diameter 0)
-		(color 0 0 0 0)
-	)
-	(junction
 		(at 92.71 102.87)
 		(diameter 0)
@@
 	(wire
 		(pts
-			(xy 115.57 97.79) (xy 116.84 97.79)
-		)
-		(stroke
-			(width 0)
-			(type default)
-		)
-	)
-	(wire
-		(pts
 			(xy 209.55 116.84) (xy 209.55 102.87)
 		)
@@
 	(wire
 		(pts
-			(xy 116.84 97.79) (xy 165.1 97.79)
+			(xy 115.57 97.79) (xy 165.1 97.79)
 		)
 		(stroke
@@
 	(wire
 		(pts
-			(xy 116.84 71.12) (xy 116.84 77.47)
-		)
-		(stroke
-			(width 0)
-			(type default)
-		)
-	)
-	(wire
-		(pts
 			(xy 91.44 102.87) (xy 92.71 102.87)
 		)
@@
 	(wire
 		(pts
-			(xy 116.84 71.12) (xy 128.27 71.12)
+			(xy 104.14 71.12) (xy 128.27 71.12)
 		)
 		(stroke
@@
 	(wire
 		(pts
-			(xy 104.14 71.12) (xy 116.84 71.12)
-		)
-		(stroke
-			(width 0)
-			(type default)
-		)
-	)
-	(wire
-		(pts
 			(xy 195.58 95.25) (xy 213.36 95.25)
 		)
@@
 		(pts
 			(xy 198.12 105.41) (xy 198.12 107.95)
-		)
-		(stroke
-			(width 0)
-			(type default)
-		)
-	)
-	(wire
-		(pts
-			(xy 116.84 82.55) (xy 116.84 97.79)
 		)
 		(stroke
@@
 		(on_board yes)
 		(dnp no)
-		(property "Reference" "R12"
+		(property "Reference" "R11"
 			(at 140.97 78.74 0)
 			(effects
@@
 			(project "CanardBoard"
 				(path "/605ab838-6b02-4cf5-a6b5-94a0cdb1b998/78243af2-5eea-48f5-811a-91865538cf4e"
-					(reference "R12")
+					(reference "R11")
 					(unit 1)
 				)
@@
 		(on_board yes)
 		(dnp no)
-		(property "Reference" "R11"
+		(property "Reference" "R10"
 			(at 129.54 78.74 0)
 			(effects
@@
 			(project "CanardBoard"
 				(path "/605ab838-6b02-4cf5-a6b5-94a0cdb1b998/78243af2-5eea-48f5-811a-91865538cf4e"
-					(reference "R11")
+					(reference "R10")
 					(unit 1)
 				)
@@
 		(on_board yes)
 		(dnp no)
-		(property "Reference" "R13"
+		(property "Reference" "R12"
 			(at 152.4 78.74 0)
 			(effects
@@
 			(project "CanardBoard"
 				(path "/605ab838-6b02-4cf5-a6b5-94a0cdb1b998/78243af2-5eea-48f5-811a-91865538cf4e"
-					(reference "R13")
+					(reference "R12")
 					(unit 1)
 				)
@@
 					(unit 1)
 				)
-			)
-		)
-	)
-	(symbol
-		(lib_id "Device:R_Small_US")
-		(at 116.84 80.01 0)
-		(unit 1)
-		(exclude_from_sim no)
-		(in_bom yes)
-		(on_board yes)
-		(dnp no)
-		(property "Reference" "R10"
-			(at 118.11 78.74 0)
-			(effects
-				(font
-					(size 1.016 1.016)
-				)
-				(justify left)
-			)
-		)
-		(property "Value" "10k"
-			(at 118.11 81.28 0)
-			(effects
-				(font
-					(size 1.27 1.27)
-				)
-				(justify left)
-			)
-		)
-		(property "Footprint" "Resistor_SMD:R_0402_1005Metric"
-			(at 116.84 80.01 0)
-			(effects
-				(font
-					(size 1.27 1.27)
-				)
-				(hide yes)
-			)
-		)
-		(property "Datasheet" "~"
-			(at 116.84 80.01 0)
-			(effects
-				(font
-					(size 1.27 1.27)
-				)
-				(hide yes)
-			)
-		)
-		(property "Description" "Resistor, small US symbol"
-			(at 116.84 80.01 0)
-			(effects
-				(font
-					(size 1.27 1.27)
-				)
-				(hide yes)
-			)
-		)
-		(pin "1"
-		)
-		(pin "2"
-		)
-		(instances
-			(project "CanardBoard"
-				(path "/605ab838-6b02-4cf5-a6b5-94a0cdb1b998/78243af2-5eea-48f5-811a-91865538cf4e"
-					(reference "R10")
-					(unit 1)
-				)

Commit message: work
Parts:
- added C84: 0.1uF, Capacitor_SMD:C_0402_1005Metric, symbol Device:C_Small
- C17: value 4.7uF -> 2.2uF
Connections:
- net +3V3: now also C84.1
- net GND: now also C84.2
Changed lines of the file:
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@@
+	)
+	(junction
+		(at 52.07 99.06)
+		(diameter 0)
+		(color 0 0 0 0)
 	)
 	(junction
@@
 	)
 	(junction
+		(at 52.07 77.47)
+		(diameter 0)
+		(color 0 0 0 0)
+	)
+	(junction
 		(at 128.27 95.25)
 		(diameter 0)
@@
 	(wire
 		(pts
+			(xy 63.5 86.36) (xy 63.5 77.47)
+		)
+		(stroke
+			(width 0)
+			(type default)
+		)
+	)
+	(wire
+		(pts
 			(xy 128.27 71.12) (xy 139.7 71.12)
 		)
@@
 	(wire
 		(pts
-			(xy 52.07 67.31) (xy 52.07 86.36)
+			(xy 52.07 67.31) (xy 52.07 77.47)
 		)
 		(stroke
@@
 	(wire
 		(pts
+			(xy 63.5 91.44) (xy 63.5 99.06)
+		)
+		(stroke
+			(width 0)
+			(type default)
+		)
+	)
+	(wire
+		(pts
 			(xy 209.55 116.84) (xy 209.55 102.87)
 		)
@@
 	(wire
 		(pts
+			(xy 52.07 99.06) (xy 52.07 105.41)
+		)
+		(stroke
+			(width 0)
+			(type default)
+		)
+	)
+	(wire
+		(pts
 			(xy 165.1 106.68) (xy 162.56 106.68)
 		)
@@
 	(wire
 		(pts
+			(xy 63.5 99.06) (xy 52.07 99.06)
+		)
+		(stroke
+			(width 0)
+			(type default)
+		)
+	)
+	(wire
+		(pts
 			(xy 138.43 92.71) (xy 139.7 92.71)
 		)
@@
 	(wire
 		(pts
-			(xy 52.07 91.44) (xy 52.07 105.41)
+			(xy 52.07 91.44) (xy 52.07 99.06)
 		)
 		(stroke
@@
 	(wire
 		(pts
+			(xy 52.07 77.47) (xy 52.07 86.36)
+		)
+		(stroke
+			(width 0)
+			(type default)
+		)
+	)
+	(wire
+		(pts
 			(xy 198.12 105.41) (xy 198.12 107.95)
+		)
+		(stroke
+			(width 0)
+			(type default)
+		)
+	)
+	(wire
+		(pts
+			(xy 63.5 77.47) (xy 52.07 77.47)
 		)
 		(stroke
@@
 			)
 		)
-		(property "Value" "4.7uF"
+		(property "Value" "2.2uF"
 			(at 54.61 90.1762 0)
 			(effects
@@
 					(unit 1)
 				)
+			)
+		)
+	)
+	(symbol
+		(lib_id "Device:C_Small")
+		(at 63.5 88.9 0)
+		(mirror y)
+		(unit 1)
+		(exclude_from_sim no)
+		(in_bom yes)
+		(on_board yes)
+		(dnp no)
+		(fields_autoplaced yes)
+		(property "Reference" "C84"
+			(at 66.04 87.6362 0)
+			(effects
+				(font
+					(size 1.27 1.27)
+				)
+				(justify right)
+			)
+		)
+		(property "Value" "0.1uF"
+			(at 66.04 90.1762 0)
+			(effects
+				(font
+					(size 1.27 1.27)
+				)
+				(justify right)
+			)
+		)
+		(property "Footprint" "Capacitor_SMD:C_0402_1005Metric"
+			(at 63.5 88.9 0)
+			(effects
+				(font
+					(size 1.27 1.27)
+				)
+				(hide yes)
+			)
+		)
+		(property "Datasheet" "~"
+			(at 63.5 88.9 0)
+			(effects
+				(font
+					(size 1.27 1.27)
+				)
+				(hide yes)
+			)
+		)
+		(property "Description" "Unpolarized capacitor, small symbol"
+			(at 63.5 88.9 0)
+			(effects
+				(font
+					(size 1.27 1.27)
+				)
+				(hide yes)
+			)
+		)
+		(property "LCSC Part #" "C49678"
+			(at 63.5 88.9 0)
+			(effects
+				(font
+					(size 1.27 1.27)
+				)
+				(hide yes)
+			)
+		)
+		(pin "1"
+		)
+		(pin "2"
+		)
+		(instances
+			(project "CanardBoard"
+				(path "/605ab838-6b02-4cf5-a6b5-94a0cdb1b998/78243af2-5eea-48f5-811a-91865538cf4e"
+					(reference "C84")
+					(unit 1)
+				)

Commit message: stuff
Parts:
- J2: footprint Connector_Card:microSD_HC_Molex_47219-2001 -> canardboard:microSD_HC_Molex_47219-2001
- renumbered C84 to C18
Changed lines of the file:
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@@
 		(dnp no)
 		(fields_autoplaced yes)
-		(property "Reference" "#PWR027"
+		(property "Reference" "#PWR029"
 			(at 52.07 71.12 0)
 			(effects
@@
 			(project "CanardBoard"
 				(path "/605ab838-6b02-4cf5-a6b5-94a0cdb1b998/78243af2-5eea-48f5-811a-91865538cf4e"
-					(reference "#PWR027")
+					(reference "#PWR029")
 					(unit 1)
 				)
@@
 		(dnp no)
 		(fields_autoplaced yes)
-		(property "Reference" "#PWR031"
+		(property "Reference" "#PWR033"
 			(at 162.56 123.19 0)
 			(effects
@@
 			(project "CanardBoard"
 				(path "/605ab838-6b02-4cf5-a6b5-94a0cdb1b998/78243af2-5eea-48f5-811a-91865538cf4e"
-					(reference "#PWR031")
+					(reference "#PWR033")
 					(unit 1)
 				)
@@
 		(dnp no)
 		(fields_autoplaced yes)
-		(property "Reference" "#PWR035"
+		(property "Reference" "#PWR037"
 			(at 256.54 121.92 0)
 			(effects
@@
 			(project "CanardBoard"
 				(path "/605ab838-6b02-4cf5-a6b5-94a0cdb1b998/78243af2-5eea-48f5-811a-91865538cf4e"
-					(reference "#PWR035")
+					(reference "#PWR037")
 					(unit 1)
 				)
@@
 		(dnp no)
 		(fields_autoplaced yes)
-		(property "Reference" "#PWR033"
+		(property "Reference" "#PWR035"
 			(at 209.55 82.55 0)
 			(effects
@@
 			(project "CanardBoard"
 				(path "/605ab838-6b02-4cf5-a6b5-94a0cdb1b998/78243af2-5eea-48f5-811a-91865538cf4e"
-					(reference "#PWR033")
+					(reference "#PWR035")
 					(unit 1)
 				)
@@
 		(dnp no)
 		(fields_autoplaced yes)
-		(property "Reference" "#PWR029"
+		(property "Reference" "#PWR031"
 			(at 92.71 72.39 0)
 			(effects
@@
 			(project "CanardBoard"
 				(path "/605ab838-6b02-4cf5-a6b5-94a0cdb1b998/78243af2-5eea-48f5-811a-91865538cf4e"
-					(reference "#PWR029")
+					(reference "#PWR031")
 					(unit 1)
 				)
@@
 		(dnp no)
 		(fields_autoplaced yes)
-		(property "Reference" "C84"
+		(property "Reference" "C18"
 			(at 66.04 87.6362 0)
 			(effects
@@
 			(project "CanardBoard"
 				(path "/605ab838-6b02-4cf5-a6b5-94a0cdb1b998/78243af2-5eea-48f5-811a-91865538cf4e"
-					(reference "C84")
+					(reference "C18")
 					(unit 1)
 				)
@@
 		(dnp no)
 		(fields_autoplaced yes)
-		(property "Reference" "#PWR032"
+		(property "Reference" "#PWR034"
 			(at 198.12 123.19 0)
 			(effects
@@
 			(project "CanardBoard"
 				(path "/605ab838-6b02-4cf5-a6b5-94a0cdb1b998/78243af2-5eea-48f5-811a-91865538cf4e"
-					(reference "#PWR032")
+					(reference "#PWR034")
 					(unit 1)
 				)
@@
 		(dnp no)
 		(fields_autoplaced yes)
-		(property "Reference" "#PWR034"
+		(property "Reference" "#PWR036"
 			(at 209.55 123.19 0)
 			(effects
@@
 			(project "CanardBoard"
 				(path "/605ab838-6b02-4cf5-a6b5-94a0cdb1b998/78243af2-5eea-48f5-811a-91865538cf4e"
-					(reference "#PWR034")
+					(reference "#PWR036")
 					(unit 1)
 				)
@@
 			)
 		)
-		(property "Footprint" "Connector_Card:microSD_HC_Molex_47219-2001"
+		(property "Footprint" "canardboard:microSD_HC_Molex_47219-2001"
 			(at 265.43 90.17 0)
 			(effects
@@
 		(dnp no)
 		(fields_autoplaced yes)
-		(property "Reference" "#PWR030"
+		(property "Reference" "#PWR032"
 			(at 162.56 83.82 0)
 			(effects
@@
 			(project "CanardBoard"
 				(path "/605ab838-6b02-4cf5-a6b5-94a0cdb1b998/78243af2-5eea-48f5-811a-91865538cf4e"
-					(reference "#PWR030")
+					(reference "#PWR032")
 					(unit 1)
 				)
@@
 		(dnp no)
 		(fields_autoplaced yes)
-		(property "Reference" "#PWR028"
+		(property "Reference" "#PWR030"
 			(at 52.07 111.76 0)
 			(effects
@@
 			(project "CanardBoard"
 				(path "/605ab838-6b02-4cf5-a6b5-94a0cdb1b998/78243af2-5eea-48f5-811a-91865538cf4e"
-					(reference "#PWR028")
-					(unit 1)
-				)
+					(reference "#PWR030")
+					(unit 1)
+				)
