File: live_telemetry/LTT/power-splitter.kicad_pcb (KiCad board)
At the start: 2 copper layers, 29 x 16.6 mm, 7 parts, among them J1 Conn_Coaxial_Small, J2 Conn_Coaxial_Small, J3 Conn_Coaxial_Small, U1 PD0810J5050S2HF

Commit message: use via'd mounting hole and add silkscreen
Parts:
- added G***: LOGO, Team_Logo:Logo_SilkScreen_5mm, F.Cu at (151.2, 100.5)
- H1, H2: footprint MountingHole:MountingHole_3.2mm_M3_DIN965_Pad_TopBottom -> MountingHole:MountingHole_3.2mm_M3_Pad_Via
Other:
- board text added: "Wilkinson Divider 800MHz - 1000MHz Rio Liu"
