File: CAN_relay/CAN_relay.kicad_sch (KiCad schematic)
At the start: 0 parts

Commit message: relay
Parts:
- added H1, H2, H3, H4: MountingHole_Pad, MountingHole:MountingHole_3.2mm_M3_Pad, symbol Mechanical:MountingHole_Pad
Connections:
- no-connect marks 0 -> 4
Other:
- added sheet Buck (buck.kicad_sch)
- added sheet CAN (can.kicad_sch)
- sheet MCU ports: added CAN0_RX, CAN0_TX, CAN1_RX, CAN1_TX; removed none
- company: (none) -> Waterloo Rocketry
- title: (none) -> CAN Repeater
